Commit message: added battery and COM is still ok, battery is fine at the back. Still need to play around with SDF values for physics engine accuracy (e.g component friction)

File: plen_ros/urdf/plen.gazebo.xacro (robot description, xacro)
@@ -3,161 +3,166 @@
 <gazebo reference="torso">
     <material>Gazebo/Gray</material>
-    <mu1>0.8</mu1> <!-- static -->
-    <mu2>0.8</mu2> <!-- dynamic -->
+    <mu1>100</mu1> <!-- static -->
+    <mu2>100</mu2> <!-- dynamic -->
+</gazebo>
+<gazebo reference="battery">
+    <material>Gazebo/Orange</material>
+    <mu1>100</mu1> <!-- static -->
+    <mu2>100</mu2> <!-- dynamic -->
 </gazebo>
 <gazebo reference="head">
     <material>Gazebo/Gray</material>
-    <mu1>0.8</mu1> <!-- static -->
-    <mu2>0.8</mu2> <!-- dynamic -->
+    <mu1>100</mu1> <!-- static -->
+    <mu2>100</mu2> <!-- dynamic -->
 </gazebo>
 <gazebo reference="rt_servo">
     <material>Gazebo/Orange</material>
-    <mu1>0.8</mu1> <!-- static -->
-    <mu2>0.8</mu2> <!-- dynamic -->
+    <mu1>100</mu1> <!-- static -->
+    <mu2>100</mu2> <!-- dynamic -->
 </gazebo>
 <gazebo reference="lt_servo">
     <material>Gazebo/Orange</material>
-    <mu1>0.8</mu1> <!-- static -->
-    <mu2>0.8</mu2> <!-- dynamic -->
+    <mu1>100</mu1> <!-- static -->
+    <mu2>100</mu2> <!-- dynamic -->
 </gazebo>
 <gazebo reference="rb_servo">
     <material>Gazebo/Orange</material>
-    <mu1>0.8</mu1> <!-- static -->
-    <mu2>0.8</mu2> <!-- dynamic -->
+    <mu1>100</mu1> <!-- static -->
+    <mu2>100</mu2> <!-- dynamic -->
 </gazebo>
 <gazebo reference="lb_servo">
     <material>Gazebo/Orange</material>
-    <mu1>0.8</mu1> <!-- static -->
-    <mu2>0.8</mu2> <!-- dynamic -->
+    <mu1>100</mu1> <!-- static -->
+    <mu2>100</mu2> <!-- dynamic -->
 </gazebo>
 <gazebo reference="r_shoulder">
     <material>Gazebo/Gray</material>
-    <mu1>0.8</mu1> <!-- static -->
-    <mu2>0.8</mu2> <!-- dynamic -->
+    <mu1>100</mu1> <!-- static -->
+    <mu2>100</mu2> <!-- dynamic -->
 </gazebo>
 <gazebo reference="rs_servo">
     <material>Gazebo/Orange</material>
-    <mu1>0.8</mu1> <!-- static -->
-    <mu2>0.8</mu2> <!-- dynamic -->
+    <mu1>100</mu1> <!-- static -->
+    <mu2>100</mu2> <!-- dynamic -->
 </gazebo>
 <gazebo reference="r_arm">
     <material>Gazebo/Gray</material>
-    <mu1>0.8</mu1> <!-- static -->
-    <mu2>0.8</mu2> <!-- dynamic -->
+    <mu1>100</mu1> <!-- static -->
+    <mu2>100</mu2> <!-- dynamic -->
 </gazebo>
 <gazebo reference="re_servo">
     <material>Gazebo/Orange</material>
-    <mu1>0.8</mu1> <!-- static -->
-    <mu2>0.8</mu2> <!-- dynamic -->
+    <mu1>100</mu1> <!-- static -->
+    <mu2>100</mu2> <!-- dynamic -->
 </gazebo>
 <gazebo reference="r_elbow">
     <material>Gazebo/Gray</material>
-    <mu1>0.8</mu1> <!-- static -->
-    <mu2>0.8</mu2> <!-- dynamic -->
+    <mu1>100</mu1> <!-- static -->
+    <mu2>100</mu2> <!-- dynamic -->
 </gazebo>
 <gazebo reference="r_hand">
     <material>Gazebo/Gray</material>
-    <mu1>0.8</mu1> <!-- static -->
-    <mu2>0.8</mu2> <!-- dynamic -->
+    <mu1>100</mu1> <!-- static -->
+    <mu2>100</mu2> <!-- dynamic -->
 </gazebo>
 <gazebo reference="l_shoulder">
     <material>Gazebo/Gray</material>
-    <mu1>0.8</mu1> <!-- static -->
-    <mu2>0.8</mu2> <!-- dynamic -->
+    <mu1>100</mu1> <!-- static -->
+    <mu2>100</mu2> <!-- dynamic -->
 </gazebo>
 <gazebo reference="ls_servo">
     <material>Gazebo/Orange</material>
-    <mu1>0.8</mu1> <!-- static -->
-    <mu2>0.8</mu2> <!-- dynamic -->
+    <mu1>100</mu1> <!-- static -->
+    <mu2>100</mu2> <!-- dynamic -->
 </gazebo>
 <gazebo reference="l_arm">
     <material>Gazebo/Gray</material>
-    <mu1>0.8</mu1> <!-- static -->
-    <mu2>0.8</mu2> <!-- dynamic -->
+    <mu1>100</mu1> <!-- static -->
+    <mu2>100</mu2> <!-- dynamic -->
 </gazebo>
 <gazebo reference="le_servo">
     <material>Gazebo/Orange</material>
-    <mu1>0.8</mu1> <!-- static -->
-    <mu2>0.8</mu2> <!-- dynamic -->
+    <mu1>100</mu1> <!-- static -->
+    <mu2>100</mu2> <!-- dynamic -->
 </gazebo>
 <gazebo reference="l_elbow">
     <material>Gazebo/Gray</material>
-    <mu1>0.8</mu1> <!-- static -->
-    <mu2>0.8</mu2> <!-- dynamic -->
+    <mu1>100</mu1> <!-- static -->
+    <mu2>100</mu2> <!-- dynamic -->
 </gazebo>
 <gazebo reference="l_hand">
     <material>Gazebo/Gray</material>
-    <mu1>0.8</mu1> <!-- static -->
-    <mu2>0.8</mu2> <!-- dynamic -->
+    <mu1>100</mu1> <!-- static -->
+    <mu2>100</mu2> <!-- dynamic -->
 </gazebo>
 <gazebo reference="r_hip">
     <material>Gazebo/Gray</material>
-    <mu1>0.8</mu1> <!-- static -->
-    <mu2>0.8</mu2> <!-- dynamic -->
+    <mu1>100</mu1> <!-- static -->
+    <mu2>100</mu2> <!-- dynamic -->
 </gazebo>
 <gazebo reference="r_thigh">
     <material>Gazebo/Orange</material>
-    <mu1>0.8</mu1> <!-- static -->
-    <mu2>0.8</mu2> <!-- dynamic -->
+    <mu1>100</mu1> <!-- static -->
+    <mu2>100</mu2> <!-- dynamic -->
 </gazebo>
 <gazebo reference="r_knee">
     <material>Gazebo/Gray</material>
-    <mu1>0.8</mu1> <!-- static -->
-    <mu2>0.8</mu2> <!-- dynamic -->
+    <mu1>100</mu1> <!-- static -->
+    <mu2>100</mu2> <!-- dynamic -->
 </gazebo>
 <gazebo reference="r_knee_servo">
     <material>Gazebo/Orange</material>
-    <mu1>0.8</mu1> <!-- static -->
-    <mu2>0.8</mu2> <!-- dynamic -->
+    <mu1>100</mu1> <!-- static -->
+    <mu2>100</mu2> <!-- dynamic -->
 </gazebo>
 <gazebo reference="r_shin">
     <material>Gazebo/Gray</material>
-    <mu1>0.8</mu1> <!-- static -->
-    <mu2>0.8</mu2> <!-- dynamic -->
+    <mu1>100</mu1> <!-- static -->
+    <mu2>100</mu2> <!-- dynamic -->
 </gazebo>
 <gazebo reference="r_ankle">
     <material>Gazebo/Orange</material>
-    <mu1>0.8</mu1> <!-- static -->
-    <mu2>0.8</mu2> <!-- dynamic -->
+    <mu1>100</mu1> <!-- static -->
+    <mu2>100</mu2> <!-- dynamic -->
 </gazebo>
 <gazebo reference="r_foot">
     <material>Gazebo/Gray</material>
-    <mu1>0.8</mu1> <!-- static -->
-    <mu2>0.8</mu2> <!-- dynamic -->
+    <mu1>100</mu1> <!-- static -->
+    <mu2>100</mu2> <!-- dynamic -->
 </gazebo>
 <gazebo reference="l_hip">
     <material>Gazebo/Gray</material>
-    <mu1>0.8</mu1> <!-- static -->
-    <mu2>0.8</mu2> <!-- dynamic -->
+    <mu1>100</mu1> <!-- static -->
+    <mu2>100</mu2> <!-- dynamic -->
 </gazebo>
 <gazebo reference="l_thigh">
     <material>Gazebo/Orange</material>
-    <mu1>0.8</mu1> <!-- static -->
-    <mu2>0.8</mu2> <!-- dynamic -->
+    <mu1>100</mu1> <!-- static -->
+    <mu2>100</mu2> <!-- dynamic -->
 </gazebo>
 <gazebo reference="l_knee">
     <material>Gazebo/Gray</material>
-    <mu1>0.8</mu1> <!-- static -->
-    <mu2>0.8</mu2> <!-- dynamic -->
+    <mu1>100</mu1> <!-- static -->
+    <mu2>100</mu2> <!-- dynamic -->
 </gazebo>
 <gazebo reference="l_knee_servo">
     <material>Gazebo/Orange</material>
-    <mu1>0.8</mu1> <!-- static -->
-    <mu2>0.8</mu2> <!-- dynamic -->
+    <mu1>100</mu1> <!-- static -->
+    <mu2>100</mu2> <!-- dynamic -->
 </gazebo>
 <gazebo reference="l_shin">
     <material>Gazebo/Gray</material>
-    <mu1>0.8</mu1> <!-- static -->
-    <mu2>0.8</mu2> <!-- dynamic -->
+    <mu1>100</mu1> <!-- static -->
+    <mu2>100</mu2> <!-- dynamic -->
 </gazebo>
 <gazebo reference="l_ankle">
     <material>Gazebo/Orange</material>
-    <mu1>0.8</mu1> <!-- static -->
-    <mu2>0.8</mu2> <!-- dynamic -->
+    <mu1>100</mu1> <!-- static -->
+    <mu2>100</mu2> <!-- dynamic -->
 </gazebo>
 <gazebo reference="l_foot">
     <material>Gazebo/Gray</material>
-    <mu1>0.8</mu1> <!-- static -->
-    <mu2>0.8</mu2> <!-- dynamic -->
+    <mu1>100</mu1> <!-- static -->
+    <mu2>100</mu2> <!-- dynamic -->
 </gazebo>
 </robot>

File: plen_ros/urdf/plen.urdf.xacro (robot description, xacro)
@@ -22,4 +22,17 @@
               meshfile="package://plen_ros/meshes/torso.stl"
               meshscale="0.001 0.001 0.001" /> <!-- m to mm -->
+  <mesh_link name="battery"
+              origin_rpy="0 0 0" origin_xyz="0 0 0"
+              i_rpy="0 0 0" i_xyz="${15/2000} ${0} ${46/4000}"
+              mass="${64/1000}"
+              ixx="${64*(11*11+46*46)/(12*1000000000)}" ixy="${0}" ixz="${0}"
+              iyy="${64*(11*11+46*46)/(12*1000000000)}" iyz="${0}"
+              izz="${64*(11*11+51*51)/(12*1000000000)}"
+              c_xyz="${15/2000} ${0} ${46/4000}"
+              size="${11/1000} ${51/1000} ${46/1000}"
+              matname="green_mat"
+              rgba="0 1 0 1"
+              meshfile="package://plen_ros/meshes/battery.stl"
+              meshscale="0.001 0.001 0.001" />
   <mesh_link name="head"
               origin_rpy="0 0 0" origin_xyz="0 0 0"
@@ -431,4 +444,7 @@
                     origin_rpy="0 0 0" origin_xyz="0 0 0"
                     parent="base_footprint" child="torso"/>
+  <frame_joint name="torso_batter" type="fixed"
+                    origin_rpy="0 0 0" origin_xyz="${-36/1000} 0 ${-12/1000}"
+                    parent="torso" child="battery"/>
   <frame_joint name="torso_head" type="fixed"
                     origin_rpy="0 0 0" origin_xyz="${-6.5/1000} 0 ${56/1000}"
