Commit message: added joint controllers for gazebo. No errors but breaks model

File: plen_ros/urdf/plen.gazebo.xacro (robot description, xacro)
@@ -1,4 +1,11 @@
 <?xml version="1.0"?>
 <robot name="plen" xmlns:xacro="http://www.ros.org/wiki/xacro">
+<!-- ros_control plugin -->
+<gazebo>
+<plugin name="gazebo_ros_control" filename="libgazebo_ros_control.so">
+  <robotNamespace>/plen</robotNamespace>
+  <robotSimType>gazebo_ros_control/DefaultRobotHWSim</robotSimType>
+</plugin>
+</gazebo>
 <gazebo reference="torso">
     <material>Gazebo/Gray</material>

File: plen_ros/urdf/plen.urdf.xacro (robot description, xacro)
@@ -9,5 +9,5 @@
   <link name="base_footprint"/>
   <!-- TORSO -->
-  <mesh_link name="torso"
+  <xacro:mesh_link name="torso"
               origin_rpy="0 0 0" origin_xyz="0 0 0"
               i_rpy="0 0 0" i_xyz="${0/8000} ${0} ${0/2000}"
@@ -22,5 +22,5 @@
               meshfile="package://plen_ros/meshes/torso.stl"
               meshscale="0.001 0.001 0.001" /> <!-- m to mm -->
-  <mesh_link name="battery"
+  <xacro:mesh_link name="battery"
               origin_rpy="0 0 0" origin_xyz="0 0 0"
               i_rpy="0 0 0" i_xyz="${15/2000} ${0} ${46/4000}"
@@ -35,5 +35,5 @@
               meshfile="package://plen_ros/meshes/battery.stl"
               meshscale="0.001 0.001 0.001" />
-  <mesh_link name="head"
+  <xacro:mesh_link name="head"
               origin_rpy="0 0 0" origin_xyz="0 0 0"
               i_rpy="0 0 0" i_xyz="${0/8000} ${0} ${0/2000}"
@@ -48,57 +48,57 @@
               meshfile="package://plen_ros/meshes/head.stl"
               meshscale="0.001 0.001 0.001" />
-  <mesh_link name="rt_servo"
-              origin_rpy="0 0 ${pi}" origin_xyz="0 0 0"
-              i_rpy="0 0 0" i_xyz="${0} ${25/4000} ${0/2000}"
-              mass="${12/1000}"
-              ixx="${12*(12*12+25*25)/(12*1000000000)}" ixy="${0}" ixz="${0}"
-              iyy="${12*(12*12+25*25)/(12*1000000000)}" iyz="${0}"
-              izz="${12*(12*12+25*25)/(12*1000000000)}"
-              c_xyz="${0} ${25/4000} ${0/2000}"
-              size="${12/1000} ${25/1000} ${25/1000}"
-              matname="blue_mat"
-              rgba="0 0 1 1"
-              meshfile="package://plen_ros/meshes/servo.stl"
-              meshscale="0.001 0.001 0.001" />
-  <mesh_link name="lt_servo"
-              origin_rpy="0 0 ${pi}" origin_xyz="0 0 0"
-              i_rpy="0 0 0" i_xyz="${0} ${25/4000} ${0/2000}"
-              mass="${12/1000}"
-              ixx="${12*(12*12+25*25)/(12*1000000000)}" ixy="${0}" ixz="${0}"
-              iyy="${12*(12*12+25*25)/(12*1000000000)}" iyz="${0}"
-              izz="${12*(12*12+25*25)/(12*1000000000)}"
-              c_xyz="${0} ${25/4000} ${0/2000}"
-              size="${12/1000} ${25/1000} ${25/1000}"
-              matname="blue_mat"
-              rgba="0 0 1 1"
-              meshfile="package://plen_ros/meshes/servo.stl"
-              meshscale="0.001 0.001 0.001" />
-  <mesh_link name="rb_servo"
-              origin_rpy="0 0 ${pi}" origin_xyz="0 0 0"
-              i_rpy="0 0 0" i_xyz="${0} ${25/4000} ${0/2000}"
-              mass="${12/1000}"
-              ixx="${12*(12*12+25*25)/(12*1000000000)}" ixy="${0}" ixz="${0}"
-              iyy="${12*(12*12+25*25)/(12*1000000000)}" iyz="${0}"
-              izz="${12*(12*12+25*25)/(12*1000000000)}"
-              c_xyz="${0} ${25/4000} ${0/2000}"
-              size="${12/1000} ${25/1000} ${25/1000}"
-              matname="blue_mat"
-              rgba="0 0 1 1"
-              meshfile="package://plen_ros/meshes/servo.stl"
-              meshscale="0.001 0.001 0.001" />
-  <mesh_link name="lb_servo"
-              origin_rpy="0 0 ${pi}" origin_xyz="0 0 0"
-              i_rpy="0 0 0" i_xyz="${0} ${25/4000} ${0/2000}"
-              mass="${12/1000}"
-              ixx="${12*(12*12+25*25)/(12*1000000000)}" ixy="${0}" ixz="${0}"
-              iyy="${12*(12*12+25*25)/(12*1000000000)}" iyz="${0}"
-              izz="${12*(12*12+25*25)/(12*1000000000)}"
-              c_xyz="${0} ${25/4000} ${0/2000}"
-              size="${12/1000} ${25/1000} ${25/1000}"
-              matname="blue_mat"
-              rgba="0 0 1 1"
-              meshfile="package://plen_ros/meshes/servo.stl"
-              meshscale="0.001 0.001 0.001" />
-  <mesh_link name="r_shoulder"
+  <xacro:mesh_link name="rt_servo"
+              origin_rpy="0 0 ${pi}" origin_xyz="0 0 0"
+              i_rpy="0 0 0" i_xyz="${0} ${25/4000} ${0/2000}"
+              mass="${12/1000}"
+              ixx="${12*(12*12+25*25)/(12*1000000000)}" ixy="${0}" ixz="${0}"
+              iyy="${12*(12*12+25*25)/(12*1000000000)}" iyz="${0}"
+              izz="${12*(12*12+25*25)/(12*1000000000)}"
+              c_xyz="${0} ${25/4000} ${0/2000}"
+              size="${12/1000} ${25/1000} ${25/1000}"
+              matname="blue_mat"
+              rgba="0 0 1 1"
+              meshfile="package://plen_ros/meshes/servo.stl"
+              meshscale="0.001 0.001 0.001" />
+  <xacro:mesh_link name="lt_servo"
+              origin_rpy="0 0 ${pi}" origin_xyz="0 0 0"
+              i_rpy="0 0 0" i_xyz="${0} ${25/4000} ${0/2000}"
+              mass="${12/1000}"
+              ixx="${12*(12*12+25*25)/(12*1000000000)}" ixy="${0}" ixz="${0}"
+              iyy="${12*(12*12+25*25)/(12*1000000000)}" iyz="${0}"
+              izz="${12*(12*12+25*25)/(12*1000000000)}"
+              c_xyz="${0} ${25/4000} ${0/2000}"
+              size="${12/1000} ${25/1000} ${25/1000}"
+              matname="blue_mat"
+              rgba="0 0 1 1"
+              meshfile="package://plen_ros/meshes/servo.stl"
+              meshscale="0.001 0.001 0.001" />
+  <xacro:mesh_link name="rb_servo"
+              origin_rpy="0 0 ${pi}" origin_xyz="0 0 0"
+              i_rpy="0 0 0" i_xyz="${0} ${25/4000} ${0/2000}"
+              mass="${12/1000}"
+              ixx="${12*(12*12+25*25)/(12*1000000000)}" ixy="${0}" ixz="${0}"
+              iyy="${12*(12*12+25*25)/(12*1000000000)}" iyz="${0}"
+              izz="${12*(12*12+25*25)/(12*1000000000)}"
+              c_xyz="${0} ${25/4000} ${0/2000}"
+              size="${12/1000} ${25/1000} ${25/1000}"
+              matname="blue_mat"
+              rgba="0 0 1 1"
+              meshfile="package://plen_ros/meshes/servo.stl"
+              meshscale="0.001 0.001 0.001" />
+  <xacro:mesh_link name="lb_servo"
+              origin_rpy="0 0 ${pi}" origin_xyz="0 0 0"
+              i_rpy="0 0 0" i_xyz="${0} ${25/4000} ${0/2000}"
+              mass="${12/1000}"
+              ixx="${12*(12*12+25*25)/(12*1000000000)}" ixy="${0}" ixz="${0}"
+              iyy="${12*(12*12+25*25)/(12*1000000000)}" iyz="${0}"
+              izz="${12*(12*12+25*25)/(12*1000000000)}"
+              c_xyz="${0} ${25/4000} ${0/2000}"
+              size="${12/1000} ${25/1000} ${25/1000}"
+              matname="blue_mat"
+              rgba="0 0 1 1"
+              meshfile="package://plen_ros/meshes/servo.stl"
+              meshscale="0.001 0.001 0.001" />
+  <xacro:mesh_link name="r_shoulder"
               origin_rpy="0 0 ${0}" origin_xyz="0 0 0"
               i_rpy="0 0 0" i_xyz="${0} ${0} ${25/2000}"
@@ -113,18 +113,18 @@
               meshfile="package://plen_ros/meshes/shoulder.stl"
               meshscale="0.001 0.001 0.001" />
-  <mesh_link name="rs_servo"
-              origin_rpy="0 0 ${pi}" origin_xyz="0 0 0"
-              i_rpy="0 0 0" i_xyz="${0} ${25/4000} ${0/2000}"
-              mass="${12/1000}"
-              ixx="${12*(12*12+25*25)/(12*1000000000)}" ixy="${0}" ixz="${0}"
-              iyy="${12*(12*12+25*25)/(12*1000000000)}" iyz="${0}"
-              izz="${12*(12*12+25*25)/(12*1000000000)}"
-              c_xyz="${0} ${25/4000} ${0/2000}"
-              size="${12/1000} ${25/1000} ${25/1000}"
-              matname="blue_mat"
-              rgba="0 0 1 1"
-              meshfile="package://plen_ros/meshes/servo.stl"
-              meshscale="0.001 0.001 0.001" />
-  <mesh_link name="r_arm"
+  <xacro:mesh_link name="rs_servo"
+              origin_rpy="0 0 ${pi}" origin_xyz="0 0 0"
+              i_rpy="0 0 0" i_xyz="${0} ${25/4000} ${0/2000}"
+              mass="${12/1000}"
+              ixx="${12*(12*12+25*25)/(12*1000000000)}" ixy="${0}" ixz="${0}"
+              iyy="${12*(12*12+25*25)/(12*1000000000)}" iyz="${0}"
+              izz="${12*(12*12+25*25)/(12*1000000000)}"
+              c_xyz="${0} ${25/4000} ${0/2000}"
+              size="${12/1000} ${25/1000} ${25/1000}"
+              matname="blue_mat"
+              rgba="0 0 1 1"
+              meshfile="package://plen_ros/meshes/servo.stl"
+              meshscale="0.001 0.001 0.001" />
+  <xacro:mesh_link name="r_arm"
               origin_rpy="0 0 ${0}" origin_xyz="0 0 0"
               i_rpy="0 0 0" i_xyz="${0} ${0} ${0/2000}"
@@ -139,18 +139,18 @@
               meshfile="package://plen_ros/meshes/arm.stl"
               meshscale="0.001 0.001 0.001" />
-  <mesh_link name="re_servo"
-              origin_rpy="0 0 ${pi}" origin_xyz="0 0 0"
-              i_rpy="0 0 0" i_xyz="${0} ${25/4000} ${0/2000}"
-              mass="${12/1000}"
-              ixx="${12*(12*12+25*25)/(12*1000000000)}" ixy="${0}" ixz="${0}"
-              iyy="${12*(12*12+25*25)/(12*1000000000)}" iyz="${0}"
-              izz="${12*(12*12+25*25)/(12*1000000000)}"
-              c_xyz="${0} ${25/4000} ${0/2000}"
-              size="${12/1000} ${25/1000} ${25/1000}"
-              matname="blue_mat"
-              rgba="0 0 1 1"
-              meshfile="package://plen_ros/meshes/servo.stl"
-              meshscale="0.001 0.001 0.001" />
-  <mesh_link name="r_elbow"
+  <xacro:mesh_link name="re_servo"
+              origin_rpy="0 0 ${pi}" origin_xyz="0 0 0"
+              i_rpy="0 0 0" i_xyz="${0} ${25/4000} ${0/2000}"
+              mass="${12/1000}"
+              ixx="${12*(12*12+25*25)/(12*1000000000)}" ixy="${0}" ixz="${0}"
+              iyy="${12*(12*12+25*25)/(12*1000000000)}" iyz="${0}"
+              izz="${12*(12*12+25*25)/(12*1000000000)}"
+              c_xyz="${0} ${25/4000} ${0/2000}"
+              size="${12/1000} ${25/1000} ${25/1000}"
+              matname="blue_mat"
+              rgba="0 0 1 1"
+              meshfile="package://plen_ros/meshes/servo.stl"
+              meshscale="0.001 0.001 0.001" />
+  <xacro:mesh_link name="r_elbow"
               origin_rpy="0 0 ${0}" origin_xyz="${-13.5/1000} 0 0"
               i_rpy="0 0 0" i_xyz="${-27/4000} ${0} ${0/2000}"
@@ -165,5 +165,5 @@
               meshfile="package://plen_ros/meshes/elbow.stl"
               meshscale="0.001 0.001 0.001" />
-  <mesh_link name="r_hand"
+  <xacro:mesh_link name="r_hand"
               origin_rpy="0 0 ${0}" origin_xyz="${0/1000} 0 0"
               i_rpy="0 0 0" i_xyz="${0} ${0} ${0/2000}"
@@ -178,5 +178,5 @@
               meshfile="package://plen_ros/meshes/hand.stl"
               meshscale="0.001 0.001 0.001" />
-  <mesh_link name="l_shoulder"
+  <xacro:mesh_link name="l_shoulder"
               origin_rpy="0 0 ${0}" origin_xyz="0 0 0"
               i_rpy="0 0 0" i_xyz="${0} ${0} ${25/2000}"
@@ -191,18 +191,18 @@
               meshfile="package://plen_ros/meshes/shoulder.stl"
               meshscale="0.001 0.001 0.001" />
-  <mesh_link name="ls_servo"
-              origin_rpy="0 0 ${pi}" origin_xyz="0 0 0"
-              i_rpy="0 0 0" i_xyz="${0} ${25/4000} ${0/2000}"
-              mass="${12/1000}"
-              ixx="${12*(12*12+25*25)/(12*1000000000)}" ixy="${0}" ixz="${0}"
-              iyy="${12*(12*12+25*25)/(12*1000000000)}" iyz="${0}"
-              izz="${12*(12*12+25*25)/(12*1000000000)}"
-              c_xyz="${0} ${25/4000} ${0/2000}"
-              size="${12/1000} ${25/1000} ${25/1000}"
-              matname="blue_mat"
-              rgba="0 0 1 1"
-              meshfile="package://plen_ros/meshes/servo.stl"
-              meshscale="0.001 0.001 0.001" />
-  <mesh_link name="l_arm"
+  <xacro:mesh_link name="ls_servo"
+              origin_rpy="0 0 ${pi}" origin_xyz="0 0 0"
+              i_rpy="0 0 0" i_xyz="${0} ${25/4000} ${0/2000}"
+              mass="${12/1000}"
+              ixx="${12*(12*12+25*25)/(12*1000000000)}" ixy="${0}" ixz="${0}"
+              iyy="${12*(12*12+25*25)/(12*1000000000)}" iyz="${0}"
+              izz="${12*(12*12+25*25)/(12*1000000000)}"
+              c_xyz="${0} ${25/4000} ${0/2000}"
+              size="${12/1000} ${25/1000} ${25/1000}"
+              matname="blue_mat"
+              rgba="0 0 1 1"
+              meshfile="package://plen_ros/meshes/servo.stl"
+              meshscale="0.001 0.001 0.001" />
+  <xacro:mesh_link name="l_arm"
               origin_rpy="0 0 ${0}" origin_xyz="0 0 0"
               i_rpy="0 0 0" i_xyz="${0} ${0} ${0/2000}"
@@ -217,18 +217,18 @@
               meshfile="package://plen_ros/meshes/arm.stl"
               meshscale="0.001 0.001 0.001" />
-  <mesh_link name="le_servo"
-              origin_rpy="0 0 ${pi}" origin_xyz="0 0 0"
-              i_rpy="0 0 0" i_xyz="${0} ${25/4000} ${0/2000}"
-              mass="${12/1000}"
-              ixx="${12*(12*12+25*25)/(12*1000000000)}" ixy="${0}" ixz="${0}"
-              iyy="${12*(12*12+25*25)/(12*1000000000)}" iyz="${0}"
-              izz="${12*(12*12+25*25)/(12*1000000000)}"
-              c_xyz="${0} ${25/4000} ${0/2000}"
-              size="${12/1000} ${25/1000} ${25/1000}"
-              matname="blue_mat"
-              rgba="0 0 1 1"
-              meshfile="package://plen_ros/meshes/servo.stl"
-              meshscale="0.001 0.001 0.001" />
-  <mesh_link name="l_elbow"
+  <xacro:mesh_link name="le_servo"
+              origin_rpy="0 0 ${pi}" origin_xyz="0 0 0"
+              i_rpy="0 0 0" i_xyz="${0} ${25/4000} ${0/2000}"
+              mass="${12/1000}"
+              ixx="${12*(12*12+25*25)/(12*1000000000)}" ixy="${0}" ixz="${0}"
+              iyy="${12*(12*12+25*25)/(12*1000000000)}" iyz="${0}"
+              izz="${12*(12*12+25*25)/(12*1000000000)}"
+              c_xyz="${0} ${25/4000} ${0/2000}"
+              size="${12/1000} ${25/1000} ${25/1000}"
+              matname="blue_mat"
+              rgba="0 0 1 1"
+              meshfile="package://plen_ros/meshes/servo.stl"
+              meshscale="0.001 0.001 0.001" />
+  <xacro:mesh_link name="l_elbow"
               origin_rpy="0 0 ${0}" origin_xyz="${-13.5/1000} 0 0"
               i_rpy="0 0 0" i_xyz="${-27/4000} ${0} ${0/2000}"
@@ -243,5 +243,5 @@
               meshfile="package://plen_ros/meshes/elbow.stl"
               meshscale="0.001 0.001 0.001" />
-  <mesh_link name="l_hand"
+  <xacro:mesh_link name="l_hand"
               origin_rpy="0 0 ${0}" origin_xyz="${0/1000} 0 0"
               i_rpy="0 0 0" i_xyz="${0} ${0} ${0/2000}"
@@ -256,5 +256,5 @@
               meshfile="package://plen_ros/meshes/hand.stl"
               meshscale="0.001 0.001 0.001" />
-  <mesh_link name="r_hip"
+  <xacro:mesh_link name="r_hip"
               origin_rpy="${pi} ${0} ${pi}" origin_xyz="${0/1000} ${0/1000} ${0/1000}"
               i_rpy="0 0 0" i_xyz="${0} ${0} ${-18/2000}"
@@ -269,5 +269,5 @@
               meshfile="package://plen_ros/meshes/rhip.stl"
               meshscale="0.001 0.001 0.001" />
-  <mesh_link name="r_thigh"
+  <xacro:mesh_link name="r_thigh"
               origin_rpy="${0} ${0} ${0}" origin_xyz="${-7.5/1000} ${0} ${-7.5/1000}"
               i_rpy="0 0 0" i_xyz="${-14/2000} ${0} ${14/2000}"
@@ -283,5 +283,5 @@
               meshscale="0.001 0.001 0.001" />
               <!-- og mass: 21.617-->
-  <mesh_link name="r_knee"
+  <xacro:mesh_link name="r_knee"
               origin_rpy="${0} ${0} ${0}" origin_xyz="${0/1000} ${0/1000} ${0/1000}"
               i_rpy="0 0 0" i_xyz="${35/2000} ${-30/2000} ${0/2000}"
@@ -296,18 +296,18 @@
               meshfile="package://plen_ros/meshes/rknee.stl"
               meshscale="0.001 0.001 0.001" />
-  <mesh_link name="r_knee_servo"
-              origin_rpy="0 0 ${pi}" origin_xyz="0 0 0"
-              i_rpy="0 0 0" i_xyz="${0} ${25/4000} ${0/2000}"
-              mass="${12/1000}"
-              ixx="${12*(12*12+25*25)/(12*1000000000)}" ixy="${0}" ixz="${0}"
-              iyy="${12*(12*12+25*25)/(12*1000000000)}" iyz="${0}"
-              izz="${12*(12*12+25*25)/(12*1000000000)}"
-              c_xyz="${0} ${25/4000} ${0/2000}"
-              size="${12/1000} ${25/1000} ${25/1000}"
-              matname="blue_mat"
-              rgba="0 0 1 1"
-              meshfile="package://plen_ros/meshes/servo.stl"
-              meshscale="0.001 0.001 0.001" />
-  <mesh_link name="r_shin"
+  <xacro:mesh_link name="r_knee_servo"
+              origin_rpy="0 0 ${pi}" origin_xyz="0 0 0"
+              i_rpy="0 0 0" i_xyz="${0} ${25/4000} ${0/2000}"
+              mass="${12/1000}"
+              ixx="${12*(12*12+25*25)/(12*1000000000)}" ixy="${0}" ixz="${0}"
+              iyy="${12*(12*12+25*25)/(12*1000000000)}" iyz="${0}"
+              izz="${12*(12*12+25*25)/(12*1000000000)}"
+              c_xyz="${0} ${25/4000} ${0/2000}"
+              size="${12/1000} ${25/1000} ${25/1000}"
+              matname="blue_mat"
+              rgba="0 0 1 1"
+              meshfile="package://plen_ros/meshes/servo.stl"
+              meshscale="0.001 0.001 0.001" />
+  <xacro:mesh_link name="r_shin"
               origin_rpy="0 ${0} ${0}" origin_xyz="${16.8/1000} ${0} ${-9.1/1000}"
               i_rpy="0 0 0" i_xyz="${36/2000} ${0} ${8/2000}"
@@ -322,5 +322,5 @@
               meshfile="package://plen_ros/meshes/rshin.stl"
               meshscale="0.001 0.001 0.001" />
-  <mesh_link name="r_ankle"
+  <xacro:mesh_link name="r_ankle"
               origin_rpy="${0} ${0} ${0}" origin_xyz="${0/1000} ${0/1000} ${0/1000}"
               i_rpy="0 0 0" i_xyz="${14/2000} ${-14/2000} ${-28/2000}"
@@ -335,5 +335,5 @@
               meshfile="package://plen_ros/meshes/rankle.stl"
               meshscale="0.001 0.001 0.001" />
-  <mesh_link name="r_foot"
+  <xacro:mesh_link name="r_foot"
               origin_rpy="0 0 ${0}" origin_xyz="${-8.5/1000} 0 ${-19.8/1000}"
               i_rpy="0 0 0" i_xyz="${-37/4000} ${0} ${-9/1000}"
@@ -348,5 +348,5 @@
               meshfile="package://plen_ros/meshes/rfoot.stl"
               meshscale="0.001 0.001 0.001" />
-  <mesh_link name="l_hip"
+  <xacro:mesh_link name="l_hip"
               origin_rpy="${0} ${0} ${pi}" origin_xyz="${0/1000} ${0/1000} ${1/1000}"
               i_rpy="0 0 0" i_xyz="${0} ${0} ${-18/2000}"
@@ -361,5 +361,5 @@
               meshfile="package://plen_ros/meshes/lhip.stl"
               meshscale="0.001 0.001 0.001" />
-  <mesh_link name="l_thigh"
+  <xacro:mesh_link name="l_thigh"
               origin_rpy="${0} ${pi/2} ${0}" origin_xyz="${0/1000} ${0} ${0/1000}"
               i_rpy="0 0 0" i_xyz="${-28/2000} ${-14/2000} ${-14/2000}"
@@ -374,5 +374,5 @@
               meshfile="package://plen_ros/meshes/rankle.stl"
               meshscale="0.001 0.001 0.001" />
-  <mesh_link name="l_knee"
+  <xacro:mesh_link name="l_knee"
               origin_rpy="${0} ${0} ${0}" origin_xyz="${0/1000} ${0/1000} ${0/1000}"
               i_rpy="0 0 0" i_xyz="${35/2000} ${-2/2000} ${0/2000}"
@@ -387,18 +387,18 @@
               meshfile="package://plen_ros/meshes/lknee.stl"
               meshscale="0.001 0.001 0.001" />
-  <mesh_link name="l_knee_servo"
-              origin_rpy="0 0 ${pi}" origin_xyz="0 0 0"
-              i_rpy="0 0 0" i_xyz="${0} ${25/4000} ${0/2000}"
-              mass="${12/1000}"
-              ixx="${12*(12*12+25*25)/(12*1000000000)}" ixy="${0}" ixz="${0}"
-              iyy="${12*(12*12+25*25)/(12*1000000000)}" iyz="${0}"
-              izz="${12*(12*12+25*25)/(12*1000000000)}"
-              c_xyz="${0} ${25/4000} ${0/2000}"
-              size="${12/1000} ${25/1000} ${25/1000}"
-              matname="blue_mat"
-              rgba="0 0 1 1"
-              meshfile="package://plen_ros/meshes/servo.stl"
-              meshscale="0.001 0.001 0.001" />
-  <mesh_link name="l_shin"
+  <xacro:mesh_link name="l_knee_servo"
+              origin_rpy="0 0 ${pi}" origin_xyz="0 0 0"
+              i_rpy="0 0 0" i_xyz="${0} ${25/4000} ${0/2000}"
+              mass="${12/1000}"
+              ixx="${12*(12*12+25*25)/(12*1000000000)}" ixy="${0}" ixz="${0}"
+              iyy="${12*(12*12+25*25)/(12*1000000000)}" iyz="${0}"
+              izz="${12*(12*12+25*25)/(12*1000000000)}"
+              c_xyz="${0} ${25/4000} ${0/2000}"
+              size="${12/1000} ${25/1000} ${25/1000}"
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
File: plen_ros/urdf/plen_macro.xacro (robot description, xacro)
@@ -1,5 +1,5 @@
 <?xml version="1.0" ?>
 <robot xmlns:xacro="http://www.ros.org/wiki/xacro">
-  <xacro:macro name="rev_joint" params="name type axis_xyz origin_rpy origin_xyz parent child effort velocity damping friction">
+  <xacro:macro name="rev_joint" params="name number type axis_xyz origin_rpy origin_xyz parent child effort velocity damping friction">
     <joint name="${name}" type="${type}">
       <axis xyz="${axis_xyz}" />
@@ -10,4 +10,14 @@
       <joint_properties damping="${damping}" friction="${friction}" />
     </joint>
+    <transmission name="tran${number}">
+    <type>transmission_interface/SimpleTransmission</type>
+    <joint name="${name}">
+      <hardwareInterface>hardware_interface/EffortJointInterface</hardwareInterface>
+    </joint>
+    <actuator name="motor${number}">
+      <hardwareInterface>hardware_interface/EffortJointInterface</hardwareInterface>
+      <mechanicalReduction>1</mechanicalReduction>
+    </actuator>
+    </transmission>
   </xacro:macro>
   <xacro:macro name="frame_joint" params="name type origin_rpy origin_xyz parent child">
