Commit message: stable standing with gazebo ros control! can still improve steady state error and overshoot, but settling time is ok!

File: plen_ros/urdf/plen.gazebo.xacro (robot description, xacro)
@@ -5,5 +5,4 @@
 <plugin name="gazebo_ros_control" filename="libgazebo_ros_control.so">
   <robotNamespace>/plen</robotNamespace>
-  <robotSimType>gazebo_ros_control/DefaultRobotHWSim</robotSimType>
 </plugin>
 </gazebo>
@@ -16,5 +15,5 @@
     <kd>1.0</kd> <!-- rigidity (damping) -->
     <minDepth>0.001</minDepth>
-    <fdir1>1 0 0</fdir1> <!-- friction direction -->
+    <fdir1>1 1 0</fdir1> <!-- friction direction -->
 </gazebo>
 <gazebo reference="battery">
@@ -26,5 +25,5 @@
     <kd>1.0</kd> <!-- rigidity (damping) -->
     <minDepth>0.001</minDepth>
-    <fdir1>1 0 0</fdir1> <!-- friction direction -->
+    <fdir1>1 1 0</fdir1> <!-- friction direction -->
 </gazebo>
 <gazebo reference="head">
@@ -36,5 +35,5 @@
     <kd>1.0</kd> <!-- rigidity (damping) -->
     <minDepth>0.001</minDepth>
-    <fdir1>1 0 0</fdir1> <!-- friction direction -->
+    <fdir1>1 1 0</fdir1> <!-- friction direction -->
 </gazebo>
 <gazebo reference="rt_servo">
@@ -46,5 +45,5 @@
     <kd>1.0</kd> <!-- rigidity (damping) -->
     <minDepth>0.001</minDepth>
-    <fdir1>1 0 0</fdir1> <!-- friction direction -->
+    <fdir1>1 1 0</fdir1> <!-- friction direction -->
 </gazebo>
 <gazebo reference="lt_servo">
@@ -56,5 +55,5 @@
     <kd>1.0</kd> <!-- rigidity (damping) -->
     <minDepth>0.001</minDepth>
-    <fdir1>1 0 0</fdir1> <!-- friction direction -->
+    <fdir1>1 1 0</fdir1> <!-- friction direction -->
 </gazebo>
 <gazebo reference="rb_servo">
@@ -66,5 +65,5 @@
     <kd>1.0</kd> <!-- rigidity (damping) -->
     <minDepth>0.001</minDepth>
-    <fdir1>1 0 0</fdir1> <!-- friction direction -->
+    <fdir1>1 1 0</fdir1> <!-- friction direction -->
 </gazebo>
 <gazebo reference="lb_servo">
@@ -76,5 +75,5 @@
     <kd>1.0</kd> <!-- rigidity (damping) -->
     <minDepth>0.001</minDepth>
-    <fdir1>1 0 0</fdir1> <!-- friction direction -->
+    <fdir1>1 1 0</fdir1> <!-- friction direction -->
 </gazebo>
 <gazebo reference="r_shoulder">
@@ -86,5 +85,5 @@
     <kd>1.0</kd> <!-- rigidity (damping) -->
     <minDepth>0.001</minDepth>
-    <fdir1>1 0 0</fdir1> <!-- friction direction -->
+    <fdir1>1 1 0</fdir1> <!-- friction direction -->
 </gazebo>
 <gazebo reference="rs_servo">
@@ -96,5 +95,5 @@
     <kd>1.0</kd> <!-- rigidity (damping) -->
     <minDepth>0.001</minDepth>
-    <fdir1>1 0 0</fdir1> <!-- friction direction -->
+    <fdir1>1 1 0</fdir1> <!-- friction direction -->
 </gazebo>
 <gazebo reference="r_arm">
@@ -106,5 +105,5 @@
     <kd>1.0</kd> <!-- rigidity (damping) -->
     <minDepth>0.001</minDepth>
-    <fdir1>1 0 0</fdir1> <!-- friction direction -->
+    <fdir1>1 1 0</fdir1> <!-- friction direction -->
 </gazebo>
 <gazebo reference="re_servo">
@@ -116,5 +115,5 @@
     <kd>1.0</kd> <!-- rigidity (damping) -->
     <minDepth>0.001</minDepth>
-    <fdir1>1 0 0</fdir1> <!-- friction direction -->
+    <fdir1>1 1 0</fdir1> <!-- friction direction -->
 </gazebo>
 <gazebo reference="r_elbow">
@@ -126,5 +125,5 @@
     <kd>1.0</kd> <!-- rigidity (damping) -->
     <minDepth>0.001</minDepth>
-    <fdir1>1 0 0</fdir1> <!-- friction direction -->
+    <fdir1>1 1 0</fdir1> <!-- friction direction -->
 </gazebo>
 <gazebo reference="r_hand">
@@ -136,5 +135,5 @@
     <kd>1.0</kd> <!-- rigidity (damping) -->
     <minDepth>0.001</minDepth>
-    <fdir1>1 0 0</fdir1> <!-- friction direction -->
+    <fdir1>1 1 0</fdir1> <!-- friction direction -->
 </gazebo>
 <gazebo reference="l_shoulder">
@@ -146,5 +145,5 @@
     <kd>1.0</kd> <!-- rigidity (damping) -->
     <minDepth>0.001</minDepth>
-    <fdir1>1 0 0</fdir1> <!-- friction direction -->
+    <fdir1>1 1 0</fdir1> <!-- friction direction -->
 </gazebo>
 <gazebo reference="ls_servo">
@@ -156,5 +155,5 @@
     <kd>1.0</kd> <!-- rigidity (damping) -->
     <minDepth>0.001</minDepth>
-    <fdir1>1 0 0</fdir1> <!-- friction direction -->
+    <fdir1>1 1 0</fdir1> <!-- friction direction -->
 </gazebo>
 <gazebo reference="l_arm">
@@ -166,5 +165,5 @@
     <kd>1.0</kd> <!-- rigidity (damping) -->
     <minDepth>0.001</minDepth>
-    <fdir1>1 0 0</fdir1> <!-- friction direction -->
+    <fdir1>1 1 0</fdir1> <!-- friction direction -->
 </gazebo>
 <gazebo reference="le_servo">
@@ -176,5 +175,5 @@
     <kd>1.0</kd> <!-- rigidity (damping) -->
     <minDepth>0.001</minDepth>
-    <fdir1>1 0 0</fdir1> <!-- friction direction -->
+    <fdir1>1 1 0</fdir1> <!-- friction direction -->
 </gazebo>
 <gazebo reference="l_elbow">
@@ -186,5 +185,5 @@
     <kd>1.0</kd> <!-- rigidity (damping) -->
     <minDepth>0.001</minDepth>
-    <fdir1>1 0 0</fdir1> <!-- friction direction -->
+    <fdir1>1 1 0</fdir1> <!-- friction direction -->
 </gazebo>
 <gazebo reference="l_hand">
@@ -196,5 +195,5 @@
     <kd>1.0</kd> <!-- rigidity (damping) -->
     <minDepth>0.001</minDepth>
-    <fdir1>1 0 0</fdir1> <!-- friction direction -->
+    <fdir1>1 1 0</fdir1> <!-- friction direction -->
 </gazebo>
 <gazebo reference="r_hip">
@@ -206,5 +205,5 @@
     <kd>1.0</kd> <!-- rigidity (damping) -->
     <minDepth>0.001</minDepth>
-    <fdir1>1 0 0</fdir1> <!-- friction direction -->
+    <fdir1>1 1 0</fdir1> <!-- friction direction -->
 </gazebo>
 <gazebo reference="r_thigh">
@@ -216,5 +215,5 @@
     <kd>1.0</kd> <!-- rigidity (damping) -->
     <minDepth>0.001</minDepth>
-    <fdir1>1 0 0</fdir1> <!-- friction direction -->
+    <fdir1>1 1 0</fdir1> <!-- friction direction -->
 </gazebo>
 <gazebo reference="r_knee">
@@ -226,5 +225,5 @@
     <kd>1.0</kd> <!-- rigidity (damping) -->
     <minDepth>0.001</minDepth>
-    <fdir1>1 0 0</fdir1> <!-- friction direction -->
+    <fdir1>1 1 0</fdir1> <!-- friction direction -->
 </gazebo>
 <gazebo reference="r_knee_servo">
@@ -236,5 +235,5 @@
     <kd>1.0</kd> <!-- rigidity (damping) -->
     <minDepth>0.001</minDepth>
-    <fdir1>1 0 0</fdir1> <!-- friction direction -->
+    <fdir1>1 1 0</fdir1> <!-- friction direction -->
 </gazebo>
 <gazebo reference="r_shin">
@@ -246,5 +245,5 @@
     <kd>1.0</kd> <!-- rigidity (damping) -->
     <minDepth>0.001</minDepth>
-    <fdir1>1 0 0</fdir1> <!-- friction direction -->
+    <fdir1>1 1 0</fdir1> <!-- friction direction -->
 </gazebo>
 <gazebo reference="r_ankle">
@@ -256,5 +255,5 @@
     <kd>1.0</kd> <!-- rigidity (damping) -->
     <minDepth>0.001</minDepth>
-    <fdir1>1 0 0</fdir1> <!-- friction direction -->
+    <fdir1>1 1 0</fdir1> <!-- friction direction -->
 </gazebo>
 <gazebo reference="r_foot">
@@ -266,5 +265,5 @@
     <kd>1.0</kd> <!-- rigidity (damping) -->
     <minDepth>0.001</minDepth>
-    <fdir1>1 0 0</fdir1> <!-- friction direction -->
+    <fdir1>1 1 0</fdir1> <!-- friction direction -->
 </gazebo>
 <gazebo reference="l_hip">
@@ -276,5 +275,5 @@
     <kd>1.0</kd> <!-- rigidity (damping) -->
     <minDepth>0.001</minDepth>
-    <fdir1>1 0 0</fdir1> <!-- friction direction -->
+    <fdir1>1 1 0</fdir1> <!-- friction direction -->
 </gazebo>
 <gazebo reference="l_thigh">
@@ -286,5 +285,5 @@
     <kd>1.0</kd> <!-- rigidity (damping) -->
     <minDepth>0.001</minDepth>
-    <fdir1>1 0 0</fdir1> <!-- friction direction -->
+    <fdir1>1 1 0</fdir1> <!-- friction direction -->
 </gazebo>
 <gazebo reference="l_knee">
@@ -296,5 +295,5 @@
     <kd>1.0</kd> <!-- rigidity (damping) -->
     <minDepth>0.001</minDepth>
-    <fdir1>1 0 0</fdir1> <!-- friction direction -->
+    <fdir1>1 1 0</fdir1> <!-- friction direction -->
 </gazebo>
 <gazebo reference="l_knee_servo">
@@ -306,5 +305,5 @@
     <kd>1.0</kd> <!-- rigidity (damping) -->
     <minDepth>0.001</minDepth>
-    <fdir1>1 0 0</fdir1> <!-- friction direction -->
+    <fdir1>1 1 0</fdir1> <!-- friction direction -->
 </gazebo>
 <gazebo reference="l_shin">
@@ -316,5 +315,5 @@
     <kd>1.0</kd> <!-- rigidity (damping) -->
     <minDepth>0.001</minDepth>
-    <fdir1>1 0 0</fdir1> <!-- friction direction -->
+    <fdir1>1 1 0</fdir1> <!-- friction direction -->
 </gazebo>
 <gazebo reference="l_ankle">
@@ -326,5 +325,5 @@
     <kd>1.0</kd> <!-- rigidity (damping) -->
     <minDepth>0.001</minDepth>
-    <fdir1>1 0 0</fdir1> <!-- friction direction -->
+    <fdir1>1 1 0</fdir1> <!-- friction direction -->
 </gazebo>
 <gazebo reference="l_foot">
@@ -336,5 +335,5 @@
     <kd>1.0</kd> <!-- rigidity (damping) -->
     <minDepth>0.001</minDepth>
-    <fdir1>1 0 0</fdir1> <!-- friction direction -->
+    <fdir1>1 1 0</fdir1> <!-- friction direction -->
 </gazebo>
 </robot>

File: plen_ros/urdf/plen.urdf.xacro (robot description, xacro)
@@ -467,6 +467,5 @@
                     origin_rpy="${pi/2} ${-pi/2} 0" origin_xyz="${-6.6/1000} ${-38/1000} ${30.8/1000}"
                     parent="torso" child="r_shoulder"
-                    effort="100"
-                    velocity="100"
+                    effort="3" velocity="1"
                     damping="1"
                     friction="1"/>
@@ -475,6 +474,5 @@
                     origin_rpy="${-pi/2} ${pi/2} ${0}" origin_xyz="${-5.35/1000} ${0.6/1000} ${12.65/1000}"
                     parent="r_shoulder" child="rs_servo"
-                    effort="100"
-                    velocity="100"
+                    effort="3" velocity="1"
                     damping="1"
                     friction="1"/>
@@ -489,6 +487,5 @@
                     origin_rpy="${-pi/2} ${0} ${pi/2}" origin_xyz="${0/1000} ${0/1000} ${-1.5/1000}"
                     parent="re_servo" child="r_elbow"
-                    effort="100"
-                    velocity="100"
+                    effort="3" velocity="1"
                     damping="1"
                     friction="1"/>
@@ -501,6 +498,5 @@
                     origin_rpy="${-pi/2} ${-pi/2} ${0}" origin_xyz="${-6.6/1000} ${38/1000} ${30.8/1000}"
                     parent="torso" child="l_shoulder"
-                    effort="100"
-                    velocity="100"
+                    effort="3" velocity="1"
                     damping="1"
                     friction="1"/>
@@ -509,6 +505,5 @@
                     origin_rpy="${-pi/2} ${pi/2} ${0}" origin_xyz="${-5.35/1000} ${0.6/1000} ${12.65/1000}"
                     parent="l_shoulder" child="ls_servo"
-                    effort="100"
-                    velocity="100"
+                    effort="3" velocity="1"
                     damping="1"
                     friction="1"/>
@@ -523,6 +518,5 @@
                     origin_rpy="${-pi/2} ${0} ${pi/2}" origin_xyz="${0/1000} ${0/1000} ${-1.5/1000}"
                     parent="le_servo" child="l_elbow"
-                    effort="100"
-                    velocity="100"
+                    effort="3" velocity="1"
                     damping="1"
                     friction="1"/>
@@ -535,6 +529,5 @@
                     origin_rpy="${pi} 0 ${pi/2}" origin_xyz="${0/1000} ${0/1000} ${14.2/1000}"
                     parent="rb_servo" child="r_hip"
-                    effort="100"
-                    velocity="100"
+                    effort="3" velocity="1"
                     damping="1"
                     friction="1"/>
@@ -543,6 +536,5 @@
                     origin_rpy="${pi} 0 0" origin_xyz="${5.45/1000} ${-2/1000} ${-12.81/1000}"
                     parent="r_hip" child="r_thigh"
-                    effort="100"
-                    velocity="100"
+                    effort="3" velocity="1"
                     damping="1"
                     friction="1"/>
@@ -551,6 +543,5 @@
                     origin_rpy="${pi/2} ${-pi/2} 0" origin_xyz="${-23/1000} ${7.5/1000} ${12.75/1000}"
                     parent="r_thigh" child="r_knee"
-                    effort="100"
-                    velocity="100"
+                    effort="3" velocity="1"
                     damping="1"
                     friction="1"/>
@@ -562,6 +553,5 @@
                     origin_rpy="0 0 0" origin_xyz="${28.1/1000} ${-14.6/1000} ${0.45/1000}"
                     parent="r_knee" child="r_shin"
-                    effort="100"
-                    velocity="100"
+                    effort="3" velocity="1"
                     damping="1"
                     friction="1"/>
@@ -570,6 +560,5 @@
                     origin_rpy="${-pi/2} ${-pi/2} ${pi}" origin_xyz="${33.75/1000} ${-17/1000} ${0/1000}"
                     parent="r_shin" child="r_ankle"
-                    effort="100"
-                    velocity="100"
+                    effort="3" velocity="1"
                     damping="1"
                     friction="1"/>
@@ -578,6 +567,5 @@
                     origin_rpy="${-pi/2} ${-pi/2} 0" origin_xyz="${4.2/1000} ${-12.7/1000} ${-7.4/1000}"
                     parent="r_ankle" child="r_foot"
-                    effort="100"
-                    velocity="100"
+                    effort="3" velocity="1"
                     damping="1"
                     friction="1"/>
@@ -587,6 +575,5 @@
                     origin_rpy="${pi} 0 ${pi/2}" origin_xyz="${0/1000} ${0/1000} ${14.2/1000}"
                     parent="lb_servo" child="l_hip"
-                    effort="100"
-                    velocity="100"
+                    effort="3" velocity="1"
                     damping="1"
                     friction="1"/>
@@ -595,6 +582,5 @@
                     origin_rpy="${pi/2} ${0} ${pi/2}" origin_xyz="${5.5/1000} ${17/1000} ${-12.65/1000}"
                     parent="l_hip" child="l_thigh"
-                    effort="100"
-                    velocity="100"
+                    effort="3" velocity="1"
                     damping="1"
                     friction="1"/>
@@ -603,6 +589,5 @@
                     origin_rpy="${-pi/2} ${0} ${-pi/2}" origin_xyz="${-7.4/1000} ${-12.8/1000} ${-8.6/1000}"
                     parent="l_thigh" child="l_knee"
-                    effort="100"
-                    velocity="100"
+                    effort="3" velocity="1"
                     damping="1"
                     friction="1"/>
@@ -614,6 +599,5 @@
                     origin_rpy="0 ${pi} ${0}" origin_xyz="${28.1/1000} ${-0.2/1000} ${0.45/1000}"
                     parent="l_knee" child="l_shin"
-                    effort="100"
-                    velocity="100"
+                    effort="3" velocity="1"
                     damping="1"
                     friction="1"/>
@@ -622,6 +606,5 @@
                     origin_rpy="${pi} ${pi/2} ${0}" origin_xyz="${-33.75/1000} ${-2/1000} ${0/1000}"
                     parent="l_shin" child="l_ankle"
-                    effort="100"
-                    velocity="100"
+                    effort="3" velocity="1"
                     damping="1"
                     friction="1"/>
@@ -630,7 +613,15 @@
                     origin_rpy="${pi} ${0} ${-pi/2}" origin_xyz="${-4.2/1000} ${7.5/1000} ${12.8/1000}"
                     parent="l_ankle" child="l_foot"
-                    effort="100"
-                    velocity="100"
-                    damping="1"
-                    friction="1"/>
+                    effort="3" velocity="1"
+                    damping="1"
+                    friction="1"/>
+  <!-- <transmission name="tran1">
+    <type>transmission_interface/SimpleTransmission</type>
+    <joint name="rb_servo_r_hip">
+      <hardwareInterface>hardware_interface/EffortJointInterface</hardwareInterface>
+    </joint>
+    <actuator name="motor1">
+      <mechanicalReduction>1</mechanicalReduction>
+    </actuator>
+    </transmission> -->
 </robot>

File: plen_ros/urdf/plen_macro.xacro (robot description, xacro)
@@ -7,5 +7,5 @@
       <parent link="${parent}" />
       <child link="${child}" />
-      <limit effort="${effort}" velocity="${velocity}" lower="-0.001" upper="0.001"/>
+      <limit effort="${effort}" velocity="${velocity}" lower="-1.7" upper="1.7"/>
       <joint_properties damping="${damping}" friction="${friction}" />
     </joint>
@@ -16,5 +16,4 @@
     </joint>
     <actuator name="motor${number}">
-      <hardwareInterface>hardware_interface/EffortJointInterface</hardwareInterface>
       <mechanicalReduction>1</mechanicalReduction>
     </actuator>

Commit message: started buiilding gym environment, and modified urdf for collision sensor, odom publisher and imu sensor

File: plen_ros/urdf/plen.gazebo.xacro (robot description, xacro)
@@ -3,7 +3,34 @@
 <!-- ros_control plugin -->
 <gazebo>
-<plugin name="gazebo_ros_control" filename="libgazebo_ros_control.so">
-  <robotNamespace>/plen</robotNamespace>
-</plugin>
+    <plugin name="gazebo_ros_control" filename="libgazebo_ros_control.so">
+      <robotNamespace>/plen</robotNamespace>
+    </plugin>
+</gazebo>
+<!-- Odometry Publisher plugin -->
+<gazebo>
+    <plugin name="p3d_base_controller" filename="libgazebo_ros_p3d.so">
+        <alwaysOn>true</alwaysOn>
+        <!--<updateRate>50.0</updateRate>--> <!-- Commented so update is as fast as possible - helps with sim reset -->
+        <bodyName>torso</bodyName>
+        <topicName>plen/odom</topicName>
+        <gaussianNoise>0.01</gaussianNoise>
+        <frameName>world</frameName>
+        <xyzOffsets>0 0 0</xyzOffsets>
+        <rpyOffsets>0 0 0</rpyOffsets>
+    </plugin>
+</gazebo>
+<!-- IMU sensor -->
+<gazebo>
+    <plugin name="gazebo_ros_imu_controller" filename="libgazebo_ros_imu.so">
+        <robotNamespace>/plen</robotNamespace>
+        <topicName>imu/data</topicName>
+        <serviceName>imu/service</serviceName>
+        <bodyName>torso</bodyName>
+        <gaussianNoise>0</gaussianNoise>
+        <rpyOffsets>0 0 0</rpyOffsets>
+        <!--<updateRate>50.0</updateRate>-->
+        <alwaysOn>true</alwaysOn>
+        <gaussianNoise>0</gaussianNoise>
+    </plugin>
 </gazebo>
 <gazebo reference="torso">
@@ -267,4 +294,29 @@
     <fdir1>1 1 0</fdir1> <!-- friction direction -->
 </gazebo>
+<!-- Contact Sensor -->
+<gazebo reference="rfs_link">
+    <material>Gazebo/GreyTransparent</material>
+    <mu1>100</mu1> <!-- static -->
+    <mu2>100</mu2> <!-- dynamic -->
+    <dampingFactor>0.001</dampingFactor>
+    <kp>10000000.0</kp> <!-- rigidity (damping) -->
+    <kd>1.0</kd> <!-- rigidity (damping) -->
+    <minDepth>0.001</minDepth>
+    <fdir1>1 1 0</fdir1> <!-- friction direction -->
+    <sensor name="rfs_link_sensor" type="contact">
+      <always_on>true</always_on>
+      <contact>
+        <collision>r_foot_fixed_joint_lump__rfs_link_collision_1</collision>
+        <!-- IMPORTANT!!!!
+        above name is based on bug in SDF parser, must be this format.
+        Figured it out by saving gazebo world as sdf with robot model loaded
+        and then reading the collision name -->
+      </contact>
+      <plugin name="bumper0_plugin" filename="libgazebo_ros_bumper.so">
+        <bumperTopicName>rfoot_rfs_state</bumperTopicName>
+        <frameName>rfs_link</frameName>
+      </plugin>
+    </sensor>
+</gazebo>
 <gazebo reference="l_hip">
     <material>Gazebo/Gray</material>
@@ -337,3 +389,28 @@
     <fdir1>1 1 0</fdir1> <!-- friction direction -->
 </gazebo>
+<!-- Contact Sensor -->
+<gazebo reference="lfs_link">
+    <material>Gazebo/GreyTransparent</material>
+    <mu1>100</mu1> <!-- static -->
+    <mu2>100</mu2> <!-- dynamic -->
+    <dampingFactor>0.001</dampingFactor>
+    <kp>10000000.0</kp> <!-- rigidity (damping) -->
+    <kd>1.0</kd> <!-- rigidity (damping) -->
+    <minDepth>0.001</minDepth>
+    <fdir1>1 1 0</fdir1> <!-- friction direction -->
+    <sensor name="lfs_link_sensor" type="contact">
+      <always_on>true</always_on>
+      <contact>
+        <collision>l_foot_fixed_joint_lump__lfs_link_collision_1</collision>
+        <!-- IMPORTANT!!!!
+        above name is based on bug in SDF parser, must be this format.
+        Figured it out by saving gazebo world as sdf with robot model loaded
+        and then reading the collision name -->
+      </contact>
+      <plugin name="bumper0_plugin" filename="libgazebo_ros_bumper.so">
+        <bumperTopicName>lfoot_lfs_state</bumperTopicName>
+        <frameName>lfs_link</frameName>
+      </plugin>
+    </sensor>
+</gazebo>
 </robot>

File: plen_ros/urdf/plen.urdf.xacro (robot description, xacro)
@@ -348,4 +348,23 @@
               meshfile="package://plen_ros/meshes/rfoot.stl"
               meshscale="0.001 0.001 0.001" />
+  <link name="rfs_link">
+      <inertial >
+            <origin xyz="0 0 0" rpy="0 0 0"/>
+            <mass value="0.000008" />
+            <inertia ixx="1.28e-08" ixy="0.0" ixz="0.0" iyy="1.28e-08" iyz="0.0" izz="1.28e-08"/>
+        </inertial>
+        <collision>
+            <origin xyz="0 0 0" rpy="0 0 0"/>
+            <geometry>
+                <box size="${41/1000} ${62.867/1000} ${2/1000}"/>
+            </geometry>
+        </collision>
+        <visual>
+            <origin rpy="0.0 0 0" xyz="0 0 0"/>
+            <geometry>
+                <box size="${41/1000} ${62.867/1000} ${2/1000}"/>
+            </geometry>
+        </visual>
+  </link>
   <xacro:mesh_link name="l_hip"
               origin_rpy="${0} ${0} ${pi}" origin_xyz="${0/1000} ${0/1000} ${1/1000}"
@@ -439,4 +458,23 @@
               meshfile="package://plen_ros/meshes/lfoot.stl"
               meshscale="0.001 0.001 0.001" />
+  <link name="lfs_link">
+      <inertial >
+            <origin xyz="0 0 0" rpy="0 0 0"/>
+            <mass value="0.000008" />
+            <inertia ixx="1.28e-08" ixy="0.0" ixz="0.0" iyy="1.28e-08" iyz="0.0" izz="1.28e-08"/>
+        </inertial>
+        <collision>
+            <origin xyz="0 0 0" rpy="0 0 0"/>
+            <geometry>
+                <box size="${41/1000} ${62.867/1000} ${2/1000}"/>
+            </geometry>
+        </collision>
+        <visual>
+            <origin rpy="0.0 0 0" xyz="0 0 0"/>
+            <geometry>
+                <box size="${41/1000} ${62.867/1000} ${2/1000}"/>
+            </geometry>
+        </visual>
+  </link>
   <!-- Joints -->
   <!-- TORSO -->
@@ -570,4 +608,9 @@
                     damping="1"
                     friction="1"/>
+  <joint name="r_foot_r_sensor" type="fixed">
+        <parent link="r_foot"/>
+        <child link="rfs_link"/>
+        <origin xyz="${-37/4000} ${0} ${-19/1000}" rpy="0 0 0"/>
+  </joint>
   <!-- LEFT LEG -->
   <xacro:rev_joint name="lb_servo_l_hip" number="7" type="revolute"
@@ -616,4 +659,9 @@
                     damping="1"
                     friction="1"/> <!-- effort and velocity taken from FEETECH FS90-FB datasheet -->
+  <joint name="l_foot_l_sensor" type="fixed">
+        <parent link="l_foot"/>
+        <child link="lfs_link"/>
+        <origin xyz="${37/4000} ${0} ${-19/1000}" rpy="0 0 0"/>
+  </joint>
   <!-- <transmission name="tran1">
     <type>transmission_interface/SimpleTransmission</type>
