Commit message: added inertia

File: plen_ros/urdf/plen.urdf.xacro (robot description, xacro)
@@ -9,8 +9,9 @@
   <mesh_link name="torso"
               origin_rpy="0 0 0" origin_xyz="0 0 0"
-              mass="0"
-              ixx="0" ixy="0" ixz="0"
-              iyy="0" iyz="0"
-              izz="0"
+              i_rpy="0 0 0" i_xyz="${2.641/1000} ${-0.668/1000} ${1.187/1000}"
+              mass="${43.968/1000}"
+              ixx="${4.598e4/1000000000}" ixy="${85.607/1000000000}" ixz="${825.993/1000000000}"
+              iyx="${85.607/1000000000}" iyy="${3.183e4/1000000000}" iyz="${25.76/1000000000}"
+              izx="${825.993/1000000000}" izy="${25.76/1000000000}" izz="${2.994e4/1000000000}"
               matname="red_mat"
               rgba="1 0 0 1"
@@ -19,8 +20,9 @@
   <mesh_link name="head"
               origin_rpy="0 0 0" origin_xyz="0 0 0"
-              mass="0"
-              ixx="0" ixy="0" ixz="0"
-              iyy="0" iyz="0"
-              izz="0"
+              i_rpy="0 0 0" i_xyz="${1.004/1000} ${0.1269/1000} ${1.697/1000}"
+              mass="${19.57/1000}"
+              ixx="${6075.414/1000000000}" ixy="${0.013/1000000000}" ixz="${349.218/1000000000}"
+              iyx="${0.013/1000000000}" iyy="${6582.133/1000000000}" iyz="${-0.022/1000000000}"
+              izx="${349.218/1000000000}" izy="${-0.022/1000000000}" izz="${7690.404/1000000000}"
               matname="green_mat"
               rgba="0 1 0 1"
@@ -29,8 +31,9 @@
   <mesh_link name="rt_servo"
               origin_rpy="0 0 ${pi}" origin_xyz="0 0 0"
-              mass="0"
-              ixx="0" ixy="0" ixz="0"
-              iyy="0" iyz="0"
-              izz="0"
+              i_rpy="0 0 0" i_xyz="${-0.000179884/1000} ${-5.05362/1000} ${-0.931856/1000}"
+              mass="${13/1000}"
+              ixx="${706.436/1000000000}" ixy="${0.008/1000000000}" ixz="${-0.017/1000000000}"
+              iyx="${0.008/1000000000}" iyy="${474.385/1000000000}" iyz="${-26.956/1000000000}"
+              izx="${-0.017/1000000000}" izy="${-26.956/1000000000}" izz="${410.689/1000000000}"
               matname="blue_mat"
               rgba="0 0 1 1"
@@ -39,8 +42,9 @@
   <mesh_link name="lt_servo"
               origin_rpy="0 0 ${pi}" origin_xyz="0 0 0"
-              mass="0"
-              ixx="0" ixy="0" ixz="0"
-              iyy="0" iyz="0"
-              izz="0"
+              i_rpy="0 0 0" i_xyz="${-0.000179884/1000} ${-5.05362/1000} ${-0.931856/1000}"
+              mass="${13/1000}"
+              ixx="${706.436/1000000000}" ixy="${0.008/1000000000}" ixz="${-0.017/1000000000}"
+              iyx="${0.008/1000000000}" iyy="${474.385/1000000000}" iyz="${-26.956/1000000000}"
+              izx="${-0.017/1000000000}" izy="${-26.956/1000000000}" izz="${410.689/1000000000}"
               matname="blue_mat"
               rgba="0 0 1 1"
@@ -49,8 +53,9 @@
   <mesh_link name="rb_servo"
               origin_rpy="0 0 ${pi}" origin_xyz="0 0 0"
-              mass="0"
-              ixx="0" ixy="0" ixz="0"
-              iyy="0" iyz="0"
-              izz="0"
+              i_rpy="0 0 0" i_xyz="${-0.000179884/1000} ${-5.05362/1000} ${-0.931856/1000}"
+              mass="${13/1000}"
+              ixx="${706.436/1000000000}" ixy="${0.008/1000000000}" ixz="${-0.017/1000000000}"
+              iyx="${0.008/1000000000}" iyy="${474.385/1000000000}" iyz="${-26.956/1000000000}"
+              izx="${-0.017/1000000000}" izy="${-26.956/1000000000}" izz="${410.689/1000000000}"
               matname="blue_mat"
               rgba="0 0 1 1"
@@ -59,8 +64,9 @@
   <mesh_link name="lb_servo"
               origin_rpy="0 0 ${pi}" origin_xyz="0 0 0"
-              mass="0"
-              ixx="0" ixy="0" ixz="0"
-              iyy="0" iyz="0"
-              izz="0"
+              i_rpy="0 0 0" i_xyz="${-0.000179884/1000} ${-5.05362/1000} ${-0.931856/1000}"
+              mass="${13/1000}"
+              ixx="${706.436/1000000000}" ixy="${0.008/1000000000}" ixz="${-0.017/1000000000}"
+              iyx="${0.008/1000000000}" iyy="${474.385/1000000000}" iyz="${-26.956/1000000000}"
+              izx="${-0.017/1000000000}" izy="${-26.956/1000000000}" izz="${410.689/1000000000}"
               matname="blue_mat"
               rgba="0 0 1 1"
@@ -69,8 +75,9 @@
   <mesh_link name="r_shoulder"
               origin_rpy="0 0 ${0}" origin_xyz="0 0 0"
-              mass="0"
-              ixx="0" ixy="0" ixz="0"
-              iyy="0" iyz="0"
-              izz="0"
+              i_rpy="0 0 0" i_xyz="${-0.6586/1000} ${-3.013/1000} ${-23.9872/1000}"
+              mass="${2.954/1000}"
+              ixx="${176.048/1000000000}" ixy="${-17.907/1000000000}" ixz="${-3.73/1000000000}"
+              iyx="${-17.907/1000000000}" iyy="${642.45/1000000000}" iyz="${-32.057/1000000000}"
+              izx="${-3.73/1000000000}" izy="${-32.057/1000000000}" izz="${713.005/1000000000}"
               matname="green_mat"
               rgba="0 1 0 1"
@@ -79,8 +86,9 @@
   <mesh_link name="rs_servo"
               origin_rpy="0 0 ${pi}" origin_xyz="0 0 0"
-              mass="0"
-              ixx="0" ixy="0" ixz="0"
-              iyy="0" iyz="0"
-              izz="0"
+              i_rpy="0 0 0" i_xyz="${-0.000179884/1000} ${-5.05362/1000} ${-0.931856/1000}"
+              mass="${13/1000}"
+              ixx="${706.436/1000000000}" ixy="${0.008/1000000000}" ixz="${-0.017/1000000000}"
+              iyx="${0.008/1000000000}" iyy="${474.385/1000000000}" iyz="${-26.956/1000000000}"
+              izx="${-0.017/1000000000}" izy="${-26.956/1000000000}" izz="${410.689/1000000000}"
               matname="blue_mat"
               rgba="0 0 1 1"
@@ -89,8 +97,9 @@
   <mesh_link name="r_arm"
               origin_rpy="0 0 ${0}" origin_xyz="0 0 0"
-              mass="0"
-              ixx="0" ixy="0" ixz="0"
-              iyy="0" iyz="0"
-              izz="0"
+              i_rpy="0 0 0" i_xyz="${-77.4619/1000} ${15.9214/1000} ${-34.001/1000}"
+              mass="${5.091/1000}"
+              ixx="${1485.346/1000000000}" ixy="${242.813/1000000000}" ixz="${3.398/1000000000}"
+              iyx="${242.813/1000000000}" iyy="${858.371/1000000000}" iyz="${-0.939/1000000000}"
+              izx="${3.398/1000000000}" izy="${-0.939/1000000000}" izz="${2003.835/1000000000}"
               matname="red_mat"
               rgba="1 0 0 1"
@@ -99,8 +108,9 @@
   <mesh_link name="re_servo"
               origin_rpy="0 0 ${pi}" origin_xyz="0 0 0"
-              mass="0"
-              ixx="0" ixy="0" ixz="0"
-              iyy="0" iyz="0"
-              izz="0"
+              i_rpy="0 0 0" i_xyz="${-0.000179884/1000} ${-5.05362/1000} ${-0.931856/1000}"
+              mass="${13/1000}"
+              ixx="${706.436/1000000000}" ixy="${0.008/1000000000}" ixz="${-0.017/1000000000}"
+              iyx="${0.008/1000000000}" iyy="${474.385/1000000000}" iyz="${-26.956/1000000000}"
+              izx="${-0.017/1000000000}" izy="${-26.956/1000000000}" izz="${410.689/1000000000}"
               matname="blue_mat"
               rgba="0 0 1 1"
@@ -109,8 +119,9 @@
   <mesh_link name="r_elbow"
               origin_rpy="0 0 ${0}" origin_xyz="${-13.5/1000} 0 0"
-              mass="0"
-              ixx="0" ixy="0" ixz="0"
-              iyy="0" iyz="0"
-              izz="0"
+              i_rpy="0 0 0" i_xyz="${3.8099/1000} ${0.4455/1000} ${-0.0457/1000}"
+              mass="${3.046/1000}"
+              ixx="${717.001/1000000000}" ixy="${-22.513/1000000000}" ixz="${-0.00015/1000000000}"
+              iyx="${-22.513/1000000000}" iyy="${168.898/1000000000}" iyz="${0.0004/1000000000}"
+              izx="${-0.00015/1000000000}" izy="${0.0004/1000000000}" izz="${791.489/1000000000}"
               matname="green_mat"
               rgba="0 1 0 1"
@@ -119,8 +130,9 @@
   <mesh_link name="r_hand"
               origin_rpy="0 0 ${0}" origin_xyz="${0/1000} 0 0"
-              mass="0"
-              ixx="0" ixy="0" ixz="0"
-              iyy="0" iyz="0"
-              izz="0"
+              i_rpy="0 0 0" i_xyz="${-1.228/1000} ${0.00071/1000} ${0.6389/1000}"
+              mass="${8.305/1000}"
+              ixx="${2276.89/1000000000}" ixy="${0.000002/1000000000}" ixz="${-4.196/1000000000}"
+              iyx="${0.000002/1000000000}" iyy="${1619.378/1000000000}" iyz="${0.000004/1000000000}"
+              izx="${-4.196/1000000000}" izy="${0.000004/1000000000}" izz="${1315.428/1000000000}"
               matname="red_mat"
               rgba="1 0 0 1"
@@ -129,8 +141,9 @@
   <mesh_link name="l_shoulder"
               origin_rpy="0 0 ${0}" origin_xyz="0 0 0"
-              mass="0"
-              ixx="0" ixy="0" ixz="0"
-              iyy="0" iyz="0"
-              izz="0"
+              i_rpy="0 0 0" i_xyz="${-0.6586/1000} ${-3.013/1000} ${-23.9872/1000}"
+              mass="${2.954/1000}"
+              ixx="${176.048/1000000000}" ixy="${-17.907/1000000000}" ixz="${-3.73/1000000000}"
+              iyx="${-17.907/1000000000}" iyy="${642.45/1000000000}" iyz="${-32.057/1000000000}"
+              izx="${-3.73/1000000000}" izy="${-32.057/1000000000}" izz="${713.005/1000000000}"
               matname="green_mat"
               rgba="0 1 0 1"
@@ -139,8 +152,9 @@
   <mesh_link name="ls_servo"
               origin_rpy="0 0 ${pi}" origin_xyz="0 0 0"
-              mass="0"
-              ixx="0" ixy="0" ixz="0"
-              iyy="0" iyz="0"
-              izz="0"
+              i_rpy="0 0 0" i_xyz="${-0.000179884/1000} ${-5.05362/1000} ${-0.931856/1000}"
+              mass="${13/1000}"
+              ixx="${706.436/1000000000}" ixy="${0.008/1000000000}" ixz="${-0.017/1000000000}"
+              iyx="${0.008/1000000000}" iyy="${474.385/1000000000}" iyz="${-26.956/1000000000}"
+              izx="${-0.017/1000000000}" izy="${-26.956/1000000000}" izz="${410.689/1000000000}"
               matname="blue_mat"
               rgba="0 0 1 1"
@@ -149,8 +163,9 @@
   <mesh_link name="l_arm"
               origin_rpy="0 0 ${0}" origin_xyz="0 0 0"
-              mass="0"
-              ixx="0" ixy="0" ixz="0"
-              iyy="0" iyz="0"
-              izz="0"
+              i_rpy="0 0 0" i_xyz="${-77.4619/1000} ${15.9214/1000} ${-34.001/1000}"
+              mass="${5.091/1000}"
+              ixx="${1485.346/1000000000}" ixy="${242.813/1000000000}" ixz="${3.398/1000000000}"
+              iyx="${242.813/1000000000}" iyy="${858.371/1000000000}" iyz="${-0.939/1000000000}"
+              izx="${3.398/1000000000}" izy="${-0.939/1000000000}" izz="${2003.835/1000000000}"
               matname="red_mat"
               rgba="1 0 0 1"
@@ -159,8 +174,9 @@
   <mesh_link name="le_servo"
               origin_rpy="0 0 ${pi}" origin_xyz="0 0 0"
-              mass="0"
-              ixx="0" ixy="0" ixz="0"
-              iyy="0" iyz="0"
-              izz="0"
+              i_rpy="0 0 0" i_xyz="${-0.000179884/1000} ${-5.05362/1000} ${-0.931856/1000}"
+              mass="${13/1000}"
+              ixx="${706.436/1000000000}" ixy="${0.008/1000000000}" ixz="${-0.017/1000000000}"
+              iyx="${0.008/1000000000}" iyy="${474.385/1000000000}" iyz="${-26.956/1000000000}"
+              izx="${-0.017/1000000000}" izy="${-26.956/1000000000}" izz="${410.689/1000000000}"
               matname="blue_mat"
               rgba="0 0 1 1"
@@ -169,8 +185,9 @@
   <mesh_link name="l_elbow"
               origin_rpy="0 0 ${0}" origin_xyz="${-13.5/1000} 0 0"
-              mass="0"
-              ixx="0" ixy="0" ixz="0"
-              iyy="0" iyz="0"
-              izz="0"
+              i_rpy="0 0 0" i_xyz="${3.8099/1000} ${0.4455/1000} ${-0.0457/1000}"
+              mass="${3.046/1000}"
+              ixx="${717.001/1000000000}" ixy="${-22.513/1000000000}" ixz="${-0.00015/1000000000}"
+              iyx="${-22.513/1000000000}" iyy="${168.898/1000000000}" iyz="${0.0004/1000000000}"
+              izx="${-0.00015/1000000000}" izy="${0.0004/1000000000}" izz="${791.489/1000000000}"
               matname="green_mat"
               rgba="0 1 0 1"
@@ -179,8 +196,9 @@
   <mesh_link name="l_hand"
               origin_rpy="0 0 ${0}" origin_xyz="${0/1000} 0 0"
-              mass="0"
-              ixx="0" ixy="0" ixz="0"
-              iyy="0" iyz="0"
-              izz="0"
+              i_rpy="0 0 0" i_xyz="${-1.228/1000} ${0.00071/1000} ${0.6389/1000}"
+              mass="${8.305/1000}"
+              ixx="${2276.89/1000000000}" ixy="${0.000002/1000000000}" ixz="${-4.196/1000000000}"
+              iyx="${0.000002/1000000000}" iyy="${1619.378/1000000000}" iyz="${0.000004/1000000000}"
+              izx="${-4.196/1000000000}" izy="${0.000004/1000000000}" izz="${1315.428/1000000000}"
               matname="red_mat"
               rgba="1 0 0 1"
@@ -189,8 +207,9 @@
   <mesh_link name="r_hip"
               origin_rpy="${pi} ${0} ${pi}" origin_xyz="${0/1000} ${0/1000} ${0/1000}"
-              mass="1"
-              ixx="0" ixy="0" ixz="0"
-              iyy="0" iyz="0"
-              izz="0"
+              i_rpy="0 0 0" i_xyz="${-1.14/1000} ${0.586/1000} ${4.525/1000}"
+              mass="${2.568/1000}"
+              ixx="${528.595/1000000000}" ixy="${3.957/1000000000}" ixz="${22.394/1000000000}"
+              iyx="${3.957/1000000000}" iyy="${106.346/1000000000}" iyz="${-13.142/1000000000}"
+              izx="${22.394/1000000000}" izy="${-13.142/1000000000}" izz="${515.988/1000000000}"
               matname="blue_mat"
               rgba="0 0 1 1"
@@ -199,8 +218,9 @@
   <mesh_link name="r_thigh"
               origin_rpy="${0} ${0} ${0}" origin_xyz="${-7.5/1000} ${0} ${-7.5/1000}"
-              mass="1"
-              ixx="0" ixy="0" ixz="0"
-              iyy="0" iyz="0"
-              izz="0"
+              i_rpy="0 0 0" i_xyz="${-0.323/1000} ${-0.327/1000} ${13.86/1000}"
+              mass="${21.617/1000}"
+              ixx="${2815.587/1000000000}" ixy="${116.787/1000000000}" ixz="${69.924/1000000000}"
+              iyx="${116.787/1000000000}" iyy="${2815.587/1000000000}" iyz="${-69.924/1000000000}"
+              izx="${69.924/1000000000}" izy="${-69.924/1000000000}" izz="${2927.98/1000000000}"
               matname="green_mat"
               rgba="0 1 0 1"
@@ -209,8 +229,9 @@
   <mesh_link name="r_knee"
               origin_rpy="${0} ${0} ${0}" origin_xyz="${0/1000} ${0/1000} ${0/1000}"
-              mass="1"
-              ixx="0" ixy="0" ixz="0"
-              iyy="0" iyz="0"
-              izz="0"
+              i_rpy="0 0 0" i_xyz="${3.0845/1000} ${1.595/1000} ${15.504/1000}"
+              mass="${5.004/1000}"
+              ixx="${1381.079/1000000000}" ixy="${5.48/1000000000}" ixz="${66.883/1000000000}"
+              iyx="${5.48/1000000000}" iyy="${656.006/1000000000}" iyz="${87.11/1000000000}"
+              izx="${66.883/1000000000}" izy="${87.11/1000000000}" izz="${923.038/1000000000}"
               matname="red_mat"
               rgba="1 0 0 1"
@@ -219,8 +240,9 @@
   <mesh_link name="r_knee_servo"
               origin_rpy="${0} ${0} ${pi}" origin_xyz="${0/1000} ${0/1000} ${0/1000}"
-              mass="1"
-              ixx="0" ixy="0" ixz="0"
-              iyy="0" iyz="0"
-              izz="0"
+              i_rpy="0 0 0" i_xyz="${-0.000179884/1000} ${-5.05362/1000} ${-0.931856/1000}"
+              mass="${13/1000}"
+              ixx="${706.436/1000000000}" ixy="${0.008/1000000000}" ixz="${-0.017/1000000000}"
+              iyx="${0.008/1000000000}" iyy="${474.385/1000000000}" iyz="${-26.956/1000000000}"
+              izx="${-0.017/1000000000}" izy="${-26.956/1000000000}" izz="${410.689/1000000000}"
               matname="blue_mat"
               rgba="0 0 1 1"
@@ -229,8 +251,9 @@
   <mesh_link name="r_shin"
               origin_rpy="0 ${0} ${0}" origin_xyz="${16.8/1000} ${0} ${-9.1/1000}"
-              mass="1"
-              ixx="0" ixy="0" ixz="0"
-              iyy="0" iyz="0"
-              izz="0"
+              i_rpy="0 0 0" i_xyz="${0.233/1000} ${-1.209/1000} ${8.78/1000}"
+              mass="${6.965/1000}"
+              ixx="${2533.205/1000000000}" ixy="${-1.876/1000000000}" ixz="${11.742/1000000000}"
+              iyx="${-1.876/1000000000}" iyy="${1194.088/1000000000}" iyz="${2.97/1000000000}"
+              izx="${11.724/1000000000}" izy="${2.97/1000000000}" izz="${3147.051/1000000000}"
               matname="blue_mat"
               rgba="0 0 1 1"
@@ -239,8 +262,9 @@
   <mesh_link name="r_ankle"
               origin_rpy="${0} ${0} ${0}" origin_xyz="${0/1000} ${0/1000} ${0/1000}"
-              mass="1"
-              ixx="0" ixy="0" ixz="0"
-              iyy="0" iyz="0"
-              izz="0"
+              i_rpy="0 0 0" i_xyz="${7.859/1000} ${-6.38/1000} ${-15.22/1000}"
+              mass="${21.617/1000}"
+              ixx="${2815.705/1000000000}" ixy="${69.289/1000000000}" ixz="${-116.66/1000000000}"
+              iyx="${69.289/1000000000}" iyy="${2928.22/1000000000}" iyz="${69.297/1000000000}"
+              izx="${-116.66/1000000000}" izy="${69.297/1000000000}" izz="${2815.691/1000000000}"
               matname="green_mat"
               rgba="0 1 0 1"
@@ -249,8 +273,9 @@
   <mesh_link name="r_foot"
               origin_rpy="0 0 ${0}" origin_xyz="${-8.5/1000} 0 ${-19.8/1000}"
-              mass="0"
-              ixx="0" ixy="0" ixz="0"
-              iyy="0" iyz="0"
-              izz="0"
+              i_rpy="0 0 0" i_xyz="${0.961/1000} ${0.257/1000} ${4.745/1000}"
+              mass="${12.396/1000}"
+              ixx="${4031.152/1000000000}" ixy="${-29.757/1000000000}" ixz="${-150.6/1000000000}"
+              iyx="${-29.757/1000000000}" iyy="${1819.588/1000000000}" iyz="${-43.683/1000000000}"
+              izx="${-150.6/1000000000}" izy="${-43.683/1000000000}" izz="${5174.827/1000000000}"
               matname="red_mat"
               rgba="1 0 0 1"
@@ -259,8 +284,9 @@
   <mesh_link name="l_hip"
               origin_rpy="${0} ${0} ${pi}" origin_xyz="${0/1000} ${0/1000} ${1/1000}"
-              mass="1"
-              ixx="0" ixy="0" ixz="0"
-              iyy="0" iyz="0"
-              izz="0"
+              i_rpy="0 0 0" i_xyz="${-1.14/1000} ${0.585/1000} ${-5.325/1000}"
+              mass="${2.568/1000}"
+              ixx="${528.595/1000000000}" ixy="${3.957/1000000000}" ixz="${-22.394/1000000000}"
+              iyx="${3.957/1000000000}" iyy="${106.346/1000000000}" iyz="${13.142/1000000000}"
+              izx="${-22.394/1000000000}" izy="${13.142/1000000000}" izz="${515.988/1000000000}"
               matname="blue_mat"
               rgba="0 0 1 1"
@@ -269,8 +295,9 @@
   <mesh_link name="l_thigh"
               origin_rpy="${0} ${pi/2} ${0}" origin_xyz="${0/1000} ${0} ${0/1000}"
-              mass="1"
-              ixx="0" ixy="0" ixz="0"
-              iyy="0" iyz="0"
-              izz="0"
+              i_rpy="0 0 0" i_xyz="${7.859/1000} ${-6.38/1000} ${-15.22/1000}"
+              mass="${21.617/1000}"
+              ixx="${2815.705/1000000000}" ixy="${69.289/1000000000}" ixz="${-116.66/1000000000}"
+              iyx="${69.289/1000000000}" iyy="${2928.22/1000000000}" iyz="${69.297/1000000000}"
+              izx="${-116.66/1000000000}" izy="${69.297/1000000000}" izz="${2815.691/1000000000}"
               matname="green_mat"
               rgba="0 1 0 1"
@@ -279,8 +306,9 @@
   <mesh_link name="l_knee"
               origin_rpy="${0} ${0} ${0}" origin_xyz="${0/1000} ${0/1000} ${0/1000}"
-              mass="1"
-              ixx="0" ixy="0" ixz="0"
-              iyy="0" iyz="0"
-              izz="0"
+              i_rpy="0 0 0" i_xyz="${20.7147/1000} ${-1.594/1000} ${3.087/1000}"
+              mass="${5.004/1000}"
+              ixx="${923.038/1000000000}" ixy="${87.11/1000000000}" ixz="${-66.883/1000000000}"
+              iyx="${87.11/1000000000}" iyy="${656.006/1000000000}" iyz="${-5.48/1000000000}"
+              izx="${-66.883/1000000000}" izy="${-5.48/1000000000}" izz="${1381.079/1000000000}"
               matname="red_mat"
               rgba="1 0 0 1"
@@ -289,8 +317,9 @@
   <mesh_link name="l_knee_servo"
               origin_rpy="${0} ${0} ${pi}" origin_xyz="${0/1000} ${0/1000} ${0/1000}"
-              mass="1"
-              ixx="0" ixy="0" ixz="0"
-              iyy="0" iyz="0"
-              izz="0"
+              i_rpy="0 0 0" i_xyz="${-0.000179884/1000} ${-5.05362/1000} ${-0.931856/1000}"
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
File: plen_ros/urdf/plen_macro.xacro (robot description, xacro)
@@ -18,5 +18,5 @@
     </joint>
   </xacro:macro>
-  <xacro:macro name="mesh_link" params="name origin_xyz origin_rpy meshfile meshscale matname rgba mass ixx ixy ixz iyy iyz izz">
+  <xacro:macro name="mesh_link" params="name origin_xyz origin_rpy meshfile meshscale matname rgba mass i_xyz i_rpy ixx ixy ixz iyx iyy iyz izx izy izz">
     <link name="${name}">
       <visual>
@@ -37,6 +37,6 @@
       <inertial>
         <mass value="${mass}" />
-        <origin rpy="${origin_rpy}" xyz="${origin_xyz}" />
-        <inertia ixx="${ixx}" ixy="${ixy}" ixz="${ixz}" iyy="${iyy}" iyz="${iyz}" izz="${izz}" />
+        <origin rpy="${i_rpy}" xyz="${i_xyz}" /> <!-- Inertial Axes -->
+        <inertia ixx="${ixx}" ixy="${ixy}" ixz="${ixz}" iyx="${iyx}" iyy="${iyy}" iyz="${iyz}" izx="${izx}" izy="${izy}" izz="${izz}" />
       </inertial>
     </link>
