Commit message: got robot to stand in gazebo! need to add battery pack and simplify collision boxes (very expensive)

File: plen_ros/urdf/plen.urdf.xacro (robot description, xacro)
@@ -3,4 +3,6 @@
   <!-- Include Macros -->
   <xacro:include filename="$(find plen_ros)/urdf/plen_macro.xacro" />
+    <!-- Include Gazebo File -->
+  <xacro:include filename="$(find plen_ros)/urdf/plen.gazebo.xacro" />
   <!-- Robot description -->
   <!-- Links -->
@@ -368,8 +370,8 @@
                     parent="torso" child="head"/>
   <frame_joint name="torso_rt_servo" type="fixed"
-                    origin_rpy="${-pi/2} 0 ${pi}" origin_xyz="${-6.6/1000} ${-19.5/1000} ${30.8/1000}"
+                    origin_rpy="${-pi/2} 0 ${pi}" origin_xyz="${-6.6/1000} ${-22/1000} ${30.8/1000}"
                     parent="torso" child="rt_servo"/>
   <frame_joint name="torso_lt_servo" type="fixed"
-                    origin_rpy="${-pi/2} 0 ${0}" origin_xyz="${-6.6/1000} ${19.5/1000} ${30.8/1000}"
+                    origin_rpy="${-pi/2} 0 ${0}" origin_xyz="${-6.6/1000} ${22/1000} ${30.8/1000}"
                     parent="torso" child="lt_servo"/>
   <frame_joint name="torso_rb_servo" type="fixed"
@@ -380,13 +382,13 @@
                     parent="torso" child="lb_servo"/>
   <!-- RIGHT ARM -->
-  <rev_joint name="torso_r_shoulder" type="continuous"
-                    axis_xyz="0 0 1"
-                    origin_rpy="${pi/2} ${-pi/2} 0" origin_xyz="${-6.6/1000} ${-33.5/1000} ${30.8/1000}"
+  <rev_joint name="torso_r_shoulder" type="revolute"
+                    axis_xyz="0 0 1"
+                    origin_rpy="${pi/2} ${-pi/2} 0" origin_xyz="${-6.6/1000} ${-38/1000} ${30.8/1000}"
                     parent="torso" child="r_shoulder"
                     effort="100"
                     velocity="100"
                     damping="1"
-                    friction="0.1"/>
-  <rev_joint name="r_shoulder_rs_servo" type="continuous"
+                    friction="1"/>
+  <rev_joint name="r_shoulder_rs_servo" type="revolute"
                     axis_xyz="0 0 1"
                     origin_rpy="${-pi/2} ${pi/2} ${0}" origin_xyz="${-5.35/1000} ${0.6/1000} ${12.65/1000}"
@@ -395,5 +397,5 @@
                     velocity="100"
                     damping="1"
-                    friction="0.1"/>
+                    friction="1"/>
   <frame_joint name="rs_servo_r_arm" type="fixed"
                     origin_rpy="${-pi/2} 0 ${0}" origin_xyz="${0/1000} ${19.5/1000} ${-2/1000}"
@@ -402,5 +404,5 @@
                     origin_rpy="${-pi/2} 0 ${0}" origin_xyz="${0/1000} ${2/1000} ${19.5/1000}"
                     parent="r_arm" child="re_servo"/>
-  <rev_joint name="re_servo_r_elbow" type="continuous"
+  <rev_joint name="re_servo_r_elbow" type="revolute"
                     axis_xyz="0 1 0"
                     origin_rpy="${-pi/2} ${0} ${pi/2}" origin_xyz="${0/1000} ${0/1000} ${-1.5/1000}"
@@ -409,18 +411,18 @@
                     velocity="100"
                     damping="1"
-                    friction="0.1"/>
+                    friction="1"/>
   <frame_joint name="r_elbow_r_hand" type="fixed"
                     origin_rpy="${pi} ${pi/2} ${0}" origin_xyz="${-30/1000} ${0/1000} ${0/1000}"
                     parent="r_elbow" child="r_hand"/>
   <!-- LEFT ARM -->
-  <rev_joint name="torso_l_shoulder" type="continuous"
-                    axis_xyz="0 0 1"
-                    origin_rpy="${-pi/2} ${-pi/2} ${0}" origin_xyz="${-6.6/1000} ${33.5/1000} ${30.8/1000}"
+  <rev_joint name="torso_l_shoulder" type="revolute"
+                    axis_xyz="0 0 1"
+                    origin_rpy="${-pi/2} ${-pi/2} ${0}" origin_xyz="${-6.6/1000} ${38/1000} ${30.8/1000}"
                     parent="torso" child="l_shoulder"
                     effort="100"
                     velocity="100"
                     damping="1"
-                    friction="0.1"/>
-  <rev_joint name="l_shoulder_ls_servo" type="continuous"
+                    friction="1"/>
+  <rev_joint name="l_shoulder_ls_servo" type="revolute"
                     axis_xyz="0 0 1"
                     origin_rpy="${-pi/2} ${pi/2} ${0}" origin_xyz="${-5.35/1000} ${0.6/1000} ${12.65/1000}"
@@ -429,5 +431,5 @@
                     velocity="100"
                     damping="1"
-                    friction="0.1"/>
+                    friction="1"/>
   <frame_joint name="ls_servo_l_arm" type="fixed"
                     origin_rpy="${-pi/2} 0 ${0}" origin_xyz="${0/1000} ${19.5/1000} ${-2/1000}"
@@ -436,5 +438,5 @@
                     origin_rpy="${-pi/2} 0 ${0}" origin_xyz="${0/1000} ${2/1000} ${19.5/1000}"
                     parent="l_arm" child="le_servo"/>
-  <rev_joint name="le_servo_l_elbow" type="continuous"
+  <rev_joint name="le_servo_l_elbow" type="revolute"
                     axis_xyz="0 1 0"
                     origin_rpy="${-pi/2} ${0} ${pi/2}" origin_xyz="${0/1000} ${0/1000} ${-1.5/1000}"
@@ -443,10 +445,10 @@
                     velocity="100"
                     damping="1"
-                    friction="0.1"/>
+                    friction="1"/>
   <frame_joint name="l_elbow_l_hand" type="fixed"
                     origin_rpy="${pi} ${pi/2} ${0}" origin_xyz="${-30/1000} ${0/1000} ${0/1000}"
                     parent="l_elbow" child="l_hand"/>
   <!-- RIGHT LEG -->
-  <rev_joint name="rb_servo_r_hip" type="continuous"
+  <rev_joint name="rb_servo_r_hip" type="revolute"
                     axis_xyz="0 0 1"
                     origin_rpy="${pi} 0 ${pi/2}" origin_xyz="${0/1000} ${0/1000} ${14.2/1000}"
@@ -455,6 +457,6 @@
                     velocity="100"
                     damping="1"
-                    friction="0.1"/>
-  <rev_joint name="r_hip_r_thigh" type="continuous"
+                    friction="1"/>
+  <rev_joint name="r_hip_r_thigh" type="revolute"
                     axis_xyz="0 1 0"
                     origin_rpy="${pi} 0 0" origin_xyz="${5.45/1000} ${-2/1000} ${-12.81/1000}"
@@ -463,6 +465,6 @@
                     velocity="100"
                     damping="1"
-                    friction="0.1"/>
-  <rev_joint name="r_thigh_r_knee" type="continuous"
+                    friction="1"/>
+  <rev_joint name="r_thigh_r_knee" type="revolute"
                     axis_xyz="0 1 0"
                     origin_rpy="${pi/2} ${-pi/2} 0" origin_xyz="${-23/1000} ${7.5/1000} ${12.75/1000}"
@@ -471,9 +473,9 @@
                     velocity="100"
                     damping="1"
-                    friction="0.1"/>
+                    friction="1"/>
   <frame_joint name="r_knee_knee_servo" type="fixed"
                     origin_rpy="${-pi/2} 0 0" origin_xyz="${28/1000} ${-12.8/1000} ${0.5/1000}"
                     parent="r_knee" child="r_knee_servo"/>
-  <rev_joint name="r_knee_r_shin" type="continuous"
+  <rev_joint name="r_knee_r_shin" type="revolute"
                     axis_xyz="0 1 0"
                     origin_rpy="0 0 0" origin_xyz="${28.1/1000} ${-14.6/1000} ${0.45/1000}"
@@ -482,6 +484,6 @@
                     velocity="100"
                     damping="1"
-                    friction="0.1"/>
-  <rev_joint name="r_shin_r_ankle" type="continuous"
+                    friction="1"/>
+  <rev_joint name="r_shin_r_ankle" type="revolute"
                     axis_xyz="0 0 1"
                     origin_rpy="${-pi/2} ${-pi/2} ${pi}" origin_xyz="${33.75/1000} ${-17/1000} ${0/1000}"
@@ -490,6 +492,6 @@
                     velocity="100"
                     damping="1"
-                    friction="0.1"/>
-  <rev_joint name="r_ankle_r_foot" type="continuous"
+                    friction="1"/>
+  <rev_joint name="r_ankle_r_foot" type="revolute"
                     axis_xyz="0 1 0"
                     origin_rpy="${-pi/2} ${-pi/2} 0" origin_xyz="${4.2/1000} ${-12.7/1000} ${-7.4/1000}"
@@ -498,7 +500,7 @@
                     velocity="100"
                     damping="1"
-                    friction="0.1"/>
+                    friction="1"/>
   <!-- LEFT LEG -->
-  <rev_joint name="lb_servo_l_hip" type="continuous"
+  <rev_joint name="lb_servo_l_hip" type="revolute"
                     axis_xyz="0 0 1"
                     origin_rpy="${pi} 0 ${pi/2}" origin_xyz="${0/1000} ${0/1000} ${14.2/1000}"
@@ -507,6 +509,6 @@
                     velocity="100"
                     damping="1"
-                    friction="0.1"/>
-  <rev_joint name="l_hip_l_thigh" type="continuous"
+                    friction="1"/>
+  <rev_joint name="l_hip_l_thigh" type="revolute"
                     axis_xyz="1 0 0"
                     origin_rpy="${pi/2} ${0} ${pi/2}" origin_xyz="${5.5/1000} ${17/1000} ${-12.65/1000}"
@@ -515,17 +517,17 @@
                     velocity="100"
                     damping="1"
-                    friction="0.1"/>
-  <rev_joint name="l_thigh_l_knee" type="continuous"
-                    axis_xyz="0 1 0"
-                    origin_rpy="${-pi/2} ${0} ${-pi/2}" origin_xyz="${-7.4/1000} ${-12.8/1000} ${-9.6/1000}"
+                    friction="1"/>
+  <rev_joint name="l_thigh_l_knee" type="revolute"
+                    axis_xyz="0 1 0"
+                    origin_rpy="${-pi/2} ${0} ${-pi/2}" origin_xyz="${-7.4/1000} ${-12.8/1000} ${-8.6/1000}"
                     parent="l_thigh" child="l_knee"
                     effort="100"
                     velocity="100"
                     damping="1"
-                    friction="0.1"/>
+                    friction="1"/>
   <frame_joint name="l_knee_knee_servo" type="fixed"
                     origin_rpy="${-pi/2} ${pi} 0" origin_xyz="${28/1000} ${1.45/1000} ${0/1000}"
                     parent="l_knee" child="l_knee_servo"/>
-  <rev_joint name="l_knee_l_shin" type="continuous"
+  <rev_joint name="l_knee_l_shin" type="revolute"
                     axis_xyz="0 1 0"
                     origin_rpy="0 ${pi} ${0}" origin_xyz="${28.1/1000} ${-0.2/1000} ${0.45/1000}"
@@ -534,6 +536,6 @@
                     velocity="100"
                     damping="1"
-                    friction="0.1"/>
-  <rev_joint name="l_shin_l_ankle" type="continuous"
+                    friction="1"/>
+  <rev_joint name="l_shin_l_ankle" type="revolute"
                     axis_xyz="0 1 0"
                     origin_rpy="${pi} ${pi/2} ${0}" origin_xyz="${-33.75/1000} ${-2/1000} ${0/1000}"
@@ -542,6 +544,6 @@
                     velocity="100"
                     damping="1"
-                    friction="0.1"/>
-  <rev_joint name="l_ankle_l_foot" type="continuous"
+                    friction="1"/>
+  <rev_joint name="l_ankle_l_foot" type="revolute"
                     axis_xyz="0 1 0"
                     origin_rpy="${pi} ${0} ${-pi/2}" origin_xyz="${-4.2/1000} ${7.5/1000} ${12.8/1000}"
@@ -550,4 +552,4 @@
                     velocity="100"
                     damping="1"
-                    friction="0.1"/>
+                    friction="1"/>
 </robot>

File: plen_ros/urdf/plen_macro.xacro (robot description, xacro)
@@ -7,5 +7,5 @@
       <parent link="${parent}" />
       <child link="${child}" />
-      <limit effort="${effort}" velocity="${velocity}" />
+      <limit effort="${effort}" velocity="${velocity}" lower="-0.01" upper="0.01"/>
       <joint_properties damping="${damping}" friction="${friction}" />
     </joint>
@@ -42,81 +42,3 @@
     </link>
   </xacro:macro>
-  <!-- <xacro:macro name="r_box" params="name origin_xyz origin_rpy size matname rgba">
-    <link name="${name}">
-      <visual>
-        <origin rpy="${origin_rpy}" xyz="${origin_xyz}" />
-        <geometry>
-          <box size="${size}" />
-        </geometry>
-        <material name="${matname}">
-         <color rgba="${rgba}" />
-        </material>
-      </visual>
-      <collision>
-        <origin rpy="${origin_rpy}" xyz="${origin_xyz}" />
-        <geometry>
-          <box size="${size}"/>
-        </geometry>
-      </collision>
-      <inertial>
-        <origin rpy="${origin_rpy}" xyz="${origin_xyz}" />
-        <mass value="${mass}"/>
-        <inertia ixx="${ixx}" ixy="${ixy}" ixz="${ixz}"
-                 iyy="${iyy}" iyz="${iyz}"
-                 izz="${izz}" />
-      </inertial>
-    </link>
-  </xacro:macro> -->
-  <!-- <xacro:macro name="r_cyl" params="name origin_xyz origin_rpy length radius matname rgba">
-    <link name="${name}">
-      <visual>
-        <origin rpy="${origin_rpy}" xyz="${origin_xyz}" />
-        <geometry>
-          <cylinder length="${length}" radius="${radius}"/>
-        </geometry>
-        <material name="${matname}">
-         <color rgba="${rgba}" />
-        </material>
-      </visual>
-      <collision>
-        <origin rpy="${origin_rpy}" xyz="${origin_xyz}" />
-        <geometry>
-          <cylinder length="${length}" radius="${radius}"/>
-        </geometry>
-      </collision>
-      <inertial>
-        <origin rpy="${origin_rpy}" xyz="${origin_xyz}" />
-        <mass value="${mass}"/>
-        <inertia ixx="${ixx}" ixy="${ixy}" ixz="${ixz}"
-                 iyy="${iyy}" iyz="${iyz}"
-                 izz="${izz}" />
-      </inertial>
-    </link>
-  </xacro:macro> -->
-  <!-- <xacro:macro name="r_sph" params="name origin_xyz origin_rpy radius matname rgba">
-    <link name="${name}">
-      <visual>
-        <origin rpy="${origin_rpy}" xyz="${origin_xyz}" />
-        <geometry>
-          <sphere radius="${radius}"/>
-        </geometry>
-        <material name="${matname}">
-         <color rgba="${rgba}" />
-        </material>
-      </visual>
-      <collision>
-        <origin rpy="${origin_rpy}" xyz="${origin_xyz}" />
-        <geometry>
-          <sphere radius="${radius}"/>
-        </geometry>
-      </collision>
-      <inertial>
-        <origin rpy="${origin_rpy}" xyz="${origin_xyz}" />
-        <mass value="${mass}"/>
-        <inertia ixx="${ixx}" ixy="${ixy}" ixz="${ixz}"
-                 iyy="${iyy}" iyz="${iyz}"
-                 izz="${izz}" />
-      </inertial>
-    </link>
-  </xacro:macro> -->
 </robot>
