Commit message: added some custom collision boxes, need to adjust some of the origins

File: plen_ros/urdf/plen.urdf.xacro (robot description, xacro)
@@ -16,4 +16,5 @@
               iyx="${85.607/1000000000}" iyy="${3.183e4/1000000000}" iyz="${25.76/1000000000}"
               izx="${825.993/1000000000}" izy="${25.76/1000000000}" izz="${2.994e4/1000000000}"
+              size="${65/1000} ${48/1000} ${75/1000}"
               matname="red_mat"
               rgba="1 0 0 1"
@@ -27,4 +28,5 @@
               iyx="${0.013/1000000000}" iyy="${6582.133/1000000000}" iyz="${-0.022/1000000000}"
               izx="${349.218/1000000000}" izy="${-0.022/1000000000}" izz="${7690.404/1000000000}"
+              size="${40/1000} ${40/1000} ${40/1000}"
               matname="green_mat"
               rgba="0 1 0 1"
@@ -34,30 +36,33 @@
               origin_rpy="0 0 ${pi}" origin_xyz="0 0 0"
               i_rpy="0 0 0" i_xyz="${-0.000179884/1000} ${-5.05362/1000} ${-0.931856/1000}"
+              mass="${15/1000}"
+              ixx="${706.436/1000000000}" ixy="${0.008/1000000000}" ixz="${-0.017/1000000000}"
+              iyx="${0.008/1000000000}" iyy="${474.385/1000000000}" iyz="${-26.956/1000000000}"
+              izx="${-0.017/1000000000}" izy="${-26.956/1000000000}" izz="${410.689/1000000000}"
+              size="${25/1000} ${12/1000} ${28/1000}"
+              matname="blue_mat"
+              rgba="0 0 1 1"
+              meshfile="package://plen_ros/meshes/servo.stl"
+              meshscale="0.001 0.001 0.001" />
+  <mesh_link name="lt_servo"
+              origin_rpy="0 0 ${pi}" origin_xyz="0 0 0"
+              i_rpy="0 0 0" i_xyz="${-0.000179884/1000} ${-5.05362/1000} ${-0.931856/1000}"
+              mass="${15/1000}"
+              ixx="${706.436/1000000000}" ixy="${0.008/1000000000}" ixz="${-0.017/1000000000}"
+              iyx="${0.008/1000000000}" iyy="${474.385/1000000000}" iyz="${-26.956/1000000000}"
+              izx="${-0.017/1000000000}" izy="${-26.956/1000000000}" izz="${410.689/1000000000}"
+              size="${25/1000} ${12/1000} ${28/1000}"
+              matname="blue_mat"
+              rgba="0 0 1 1"
+              meshfile="package://plen_ros/meshes/servo.stl"
+              meshscale="0.001 0.001 0.001" />
+  <mesh_link name="rb_servo"
+              origin_rpy="0 0 ${pi}" origin_xyz="0 0 0"
+              i_rpy="0 0 0" i_xyz="${-0.000179884/1000} ${-5.05362/1000} ${-0.931856/1000}"
               mass="${13/1000}"
               ixx="${706.436/1000000000}" ixy="${0.008/1000000000}" ixz="${-0.017/1000000000}"
               iyx="${0.008/1000000000}" iyy="${474.385/1000000000}" iyz="${-26.956/1000000000}"
               izx="${-0.017/1000000000}" izy="${-26.956/1000000000}" izz="${410.689/1000000000}"
-              matname="blue_mat"
-              rgba="0 0 1 1"
-              meshfile="package://plen_ros/meshes/servo.stl"
-              meshscale="0.001 0.001 0.001" />
-  <mesh_link name="lt_servo"
-              origin_rpy="0 0 ${pi}" origin_xyz="0 0 0"
-              i_rpy="0 0 0" i_xyz="${-0.000179884/1000} ${-5.05362/1000} ${-0.931856/1000}"
-              mass="${13/1000}"
-              ixx="${706.436/1000000000}" ixy="${0.008/1000000000}" ixz="${-0.017/1000000000}"
-              iyx="${0.008/1000000000}" iyy="${474.385/1000000000}" iyz="${-26.956/1000000000}"
-              izx="${-0.017/1000000000}" izy="${-26.956/1000000000}" izz="${410.689/1000000000}"
-              matname="blue_mat"
-              rgba="0 0 1 1"
-              meshfile="package://plen_ros/meshes/servo.stl"
-              meshscale="0.001 0.001 0.001" />
-  <mesh_link name="rb_servo"
-              origin_rpy="0 0 ${pi}" origin_xyz="0 0 0"
-              i_rpy="0 0 0" i_xyz="${-0.000179884/1000} ${-5.05362/1000} ${-0.931856/1000}"
-              mass="${13/1000}"
-              ixx="${706.436/1000000000}" ixy="${0.008/1000000000}" ixz="${-0.017/1000000000}"
-              iyx="${0.008/1000000000}" iyy="${474.385/1000000000}" iyz="${-26.956/1000000000}"
-              izx="${-0.017/1000000000}" izy="${-26.956/1000000000}" izz="${410.689/1000000000}"
+              size="${25/1000} ${12/1000} ${28/1000}"
               matname="blue_mat"
               rgba="0 0 1 1"
@@ -67,8 +72,9 @@
               origin_rpy="0 0 ${pi}" origin_xyz="0 0 0"
               i_rpy="0 0 0" i_xyz="${-0.000179884/1000} ${-5.05362/1000} ${-0.931856/1000}"
-              mass="${13/1000}"
-              ixx="${706.436/1000000000}" ixy="${0.008/1000000000}" ixz="${-0.017/1000000000}"
-              iyx="${0.008/1000000000}" iyy="${474.385/1000000000}" iyz="${-26.956/1000000000}"
-              izx="${-0.017/1000000000}" izy="${-26.956/1000000000}" izz="${410.689/1000000000}"
+              mass="${15/1000}"
+              ixx="${706.436/1000000000}" ixy="${0.008/1000000000}" ixz="${-0.017/1000000000}"
+              iyx="${0.008/1000000000}" iyy="${474.385/1000000000}" iyz="${-26.956/1000000000}"
+              izx="${-0.017/1000000000}" izy="${-26.956/1000000000}" izz="${410.689/1000000000}"
+              size="${25/1000} ${12/1000} ${28/1000}"
               matname="blue_mat"
               rgba="0 0 1 1"
@@ -82,4 +88,5 @@
               iyx="${-17.907/1000000000}" iyy="${642.45/1000000000}" iyz="${-32.057/1000000000}"
               izx="${-3.73/1000000000}" izy="${-32.057/1000000000}" izz="${713.005/1000000000}"
+              size="${25/1000} ${35/1000} ${18/1000}"
               matname="green_mat"
               rgba="0 1 0 1"
@@ -89,8 +96,9 @@
               origin_rpy="0 0 ${pi}" origin_xyz="0 0 0"
               i_rpy="0 0 0" i_xyz="${-0.000179884/1000} ${-5.05362/1000} ${-0.931856/1000}"
-              mass="${13/1000}"
-              ixx="${706.436/1000000000}" ixy="${0.008/1000000000}" ixz="${-0.017/1000000000}"
-              iyx="${0.008/1000000000}" iyy="${474.385/1000000000}" iyz="${-26.956/1000000000}"
-              izx="${-0.017/1000000000}" izy="${-26.956/1000000000}" izz="${410.689/1000000000}"
+              mass="${15/1000}"
+              ixx="${706.436/1000000000}" ixy="${0.008/1000000000}" ixz="${-0.017/1000000000}"
+              iyx="${0.008/1000000000}" iyy="${474.385/1000000000}" iyz="${-26.956/1000000000}"
+              izx="${-0.017/1000000000}" izy="${-26.956/1000000000}" izz="${410.689/1000000000}"
+              size="${25/1000} ${12/1000} ${28/1000}"
               matname="blue_mat"
               rgba="0 0 1 1"
@@ -104,4 +112,5 @@
               iyx="${242.813/1000000000}" iyy="${858.371/1000000000}" iyz="${-0.939/1000000000}"
               izx="${3.398/1000000000}" izy="${-0.939/1000000000}" izz="${2003.835/1000000000}"
+              size="${35/1000} ${15/1000} ${50/1000}"
               matname="red_mat"
               rgba="1 0 0 1"
@@ -111,8 +120,9 @@
               origin_rpy="0 0 ${pi}" origin_xyz="0 0 0"
               i_rpy="0 0 0" i_xyz="${-0.000179884/1000} ${-5.05362/1000} ${-0.931856/1000}"
-              mass="${13/1000}"
-              ixx="${706.436/1000000000}" ixy="${0.008/1000000000}" ixz="${-0.017/1000000000}"
-              iyx="${0.008/1000000000}" iyy="${474.385/1000000000}" iyz="${-26.956/1000000000}"
-              izx="${-0.017/1000000000}" izy="${-26.956/1000000000}" izz="${410.689/1000000000}"
+              mass="${15/1000}"
+              ixx="${706.436/1000000000}" ixy="${0.008/1000000000}" ixz="${-0.017/1000000000}"
+              iyx="${0.008/1000000000}" iyy="${474.385/1000000000}" iyz="${-26.956/1000000000}"
+              izx="${-0.017/1000000000}" izy="${-26.956/1000000000}" izz="${410.689/1000000000}"
+              size="${25/1000} ${12/1000} ${28/1000}"
               matname="blue_mat"
               rgba="0 0 1 1"
@@ -126,4 +136,5 @@
               iyx="${-22.513/1000000000}" iyy="${168.898/1000000000}" iyz="${0.0004/1000000000}"
               izx="${-0.00015/1000000000}" izy="${0.0004/1000000000}" izz="${791.489/1000000000}"
+              size="${14/1000} ${34/1000} ${27/1000}"
               matname="green_mat"
               rgba="0 1 0 1"
@@ -137,4 +148,5 @@
               iyx="${0.000002/1000000000}" iyy="${1619.378/1000000000}" iyz="${0.000004/1000000000}"
               izx="${-4.196/1000000000}" izy="${0.000004/1000000000}" izz="${1315.428/1000000000}"
+              size="${19/1000} ${34/1000} ${35/1000}"
               matname="red_mat"
               rgba="1 0 0 1"
@@ -148,4 +160,5 @@
               iyx="${-17.907/1000000000}" iyy="${642.45/1000000000}" iyz="${-32.057/1000000000}"
               izx="${-3.73/1000000000}" izy="${-32.057/1000000000}" izz="${713.005/1000000000}"
+              size="${25/1000} ${35/1000} ${18/1000}"
               matname="green_mat"
               rgba="0 1 0 1"
@@ -155,8 +168,9 @@
               origin_rpy="0 0 ${pi}" origin_xyz="0 0 0"
               i_rpy="0 0 0" i_xyz="${-0.000179884/1000} ${-5.05362/1000} ${-0.931856/1000}"
-              mass="${13/1000}"
-              ixx="${706.436/1000000000}" ixy="${0.008/1000000000}" ixz="${-0.017/1000000000}"
-              iyx="${0.008/1000000000}" iyy="${474.385/1000000000}" iyz="${-26.956/1000000000}"
-              izx="${-0.017/1000000000}" izy="${-26.956/1000000000}" izz="${410.689/1000000000}"
+              mass="${15/1000}"
+              ixx="${706.436/1000000000}" ixy="${0.008/1000000000}" ixz="${-0.017/1000000000}"
+              iyx="${0.008/1000000000}" iyy="${474.385/1000000000}" iyz="${-26.956/1000000000}"
+              izx="${-0.017/1000000000}" izy="${-26.956/1000000000}" izz="${410.689/1000000000}"
+              size="${25/1000} ${12/1000} ${28/1000}"
               matname="blue_mat"
               rgba="0 0 1 1"
@@ -170,4 +184,5 @@
               iyx="${242.813/1000000000}" iyy="${858.371/1000000000}" iyz="${-0.939/1000000000}"
               izx="${3.398/1000000000}" izy="${-0.939/1000000000}" izz="${2003.835/1000000000}"
+              size="${35/1000} ${15/1000} ${50/1000}"
               matname="red_mat"
               rgba="1 0 0 1"
@@ -177,8 +192,9 @@
               origin_rpy="0 0 ${pi}" origin_xyz="0 0 0"
               i_rpy="0 0 0" i_xyz="${-0.000179884/1000} ${-5.05362/1000} ${-0.931856/1000}"
-              mass="${13/1000}"
-              ixx="${706.436/1000000000}" ixy="${0.008/1000000000}" ixz="${-0.017/1000000000}"
-              iyx="${0.008/1000000000}" iyy="${474.385/1000000000}" iyz="${-26.956/1000000000}"
-              izx="${-0.017/1000000000}" izy="${-26.956/1000000000}" izz="${410.689/1000000000}"
+              mass="${15/1000}"
+              ixx="${706.436/1000000000}" ixy="${0.008/1000000000}" ixz="${-0.017/1000000000}"
+              iyx="${0.008/1000000000}" iyy="${474.385/1000000000}" iyz="${-26.956/1000000000}"
+              izx="${-0.017/1000000000}" izy="${-26.956/1000000000}" izz="${410.689/1000000000}"
+              size="${25/1000} ${12/1000} ${28/1000}"
               matname="blue_mat"
               rgba="0 0 1 1"
@@ -192,4 +208,5 @@
               iyx="${-22.513/1000000000}" iyy="${168.898/1000000000}" iyz="${0.0004/1000000000}"
               izx="${-0.00015/1000000000}" izy="${0.0004/1000000000}" izz="${791.489/1000000000}"
+              size="${14/1000} ${34/1000} ${27/1000}"
               matname="green_mat"
               rgba="0 1 0 1"
@@ -203,4 +220,5 @@
               iyx="${0.000002/1000000000}" iyy="${1619.378/1000000000}" iyz="${0.000004/1000000000}"
               izx="${-4.196/1000000000}" izy="${0.000004/1000000000}" izz="${1315.428/1000000000}"
+              size="${19/1000} ${34/1000} ${35/1000}"
               matname="red_mat"
               rgba="1 0 0 1"
@@ -214,4 +232,5 @@
               iyx="${3.957/1000000000}" iyy="${106.346/1000000000}" iyz="${-13.142/1000000000}"
               izx="${22.394/1000000000}" izy="${-13.142/1000000000}" izz="${515.988/1000000000}"
+              size="${25/1000} ${35/1000} ${18/1000}"
               matname="blue_mat"
               rgba="0 0 1 1"
@@ -221,12 +240,14 @@
               origin_rpy="${0} ${0} ${0}" origin_xyz="${-7.5/1000} ${0} ${-7.5/1000}"
               i_rpy="0 0 0" i_xyz="${-0.323/1000} ${-0.327/1000} ${13.86/1000}"
-              mass="${21.617/1000}"
+              mass="${35/1000}"
               ixx="${2815.587/1000000000}" ixy="${116.787/1000000000}" ixz="${69.924/1000000000}"
               iyx="${116.787/1000000000}" iyy="${2815.587/1000000000}" iyz="${-69.924/1000000000}"
               izx="${69.924/1000000000}" izy="${-69.924/1000000000}" izz="${2927.98/1000000000}"
+              size="${28/1000} ${28/1000} ${28/1000}"
               matname="green_mat"
               rgba="0 1 0 1"
               meshfile="package://plen_ros/meshes/rthigh.stl"
               meshscale="0.001 0.001 0.001" />
+              <!-- og mass: 21.617-->
   <mesh_link name="r_knee"
               origin_rpy="${0} ${0} ${0}" origin_xyz="${0/1000} ${0/1000} ${0/1000}"
@@ -236,4 +257,5 @@
               iyx="${5.48/1000000000}" iyy="${656.006/1000000000}" iyz="${87.11/1000000000}"
               izx="${66.883/1000000000}" izy="${87.11/1000000000}" izz="${923.038/1000000000}"
+              size="${38/1000} ${19/1000} ${40/1000}"
               matname="red_mat"
               rgba="1 0 0 1"
@@ -243,8 +265,9 @@
               origin_rpy="${0} ${0} ${pi}" origin_xyz="${0/1000} ${0/1000} ${0/1000}"
               i_rpy="0 0 0" i_xyz="${-0.000179884/1000} ${-5.05362/1000} ${-0.931856/1000}"
-              mass="${13/1000}"
-              ixx="${706.436/1000000000}" ixy="${0.008/1000000000}" ixz="${-0.017/1000000000}"
-              iyx="${0.008/1000000000}" iyy="${474.385/1000000000}" iyz="${-26.956/1000000000}"
-              izx="${-0.017/1000000000}" izy="${-26.956/1000000000}" izz="${410.689/1000000000}"
+              mass="${15/1000}"
+              ixx="${706.436/1000000000}" ixy="${0.008/1000000000}" ixz="${-0.017/1000000000}"
+              iyx="${0.008/1000000000}" iyy="${474.385/1000000000}" iyz="${-26.956/1000000000}"
+              izx="${-0.017/1000000000}" izy="${-26.956/1000000000}" izz="${410.689/1000000000}"
+              size="${25/1000} ${12/1000} ${28/1000}"
               matname="blue_mat"
               rgba="0 0 1 1"
@@ -258,4 +281,5 @@
               iyx="${-1.876/1000000000}" iyy="${1194.088/1000000000}" iyz="${2.97/1000000000}"
               izx="${11.724/1000000000}" izy="${2.97/1000000000}" izz="${3147.051/1000000000}"
+              size="${40/1000} ${25/1000} ${45/1000}"
               matname="blue_mat"
               rgba="0 0 1 1"
@@ -265,8 +289,9 @@
               origin_rpy="${0} ${0} ${0}" origin_xyz="${0/1000} ${0/1000} ${0/1000}"
               i_rpy="0 0 0" i_xyz="${7.859/1000} ${-6.38/1000} ${-15.22/1000}"
-              mass="${21.617/1000}"
+              mass="${35/1000}"
               ixx="${2815.705/1000000000}" ixy="${69.289/1000000000}" ixz="${-116.66/1000000000}"
               iyx="${69.289/1000000000}" iyy="${2928.22/1000000000}" iyz="${69.297/1000000000}"
               izx="${-116.66/1000000000}" izy="${69.297/1000000000}" izz="${2815.691/1000000000}"
+              size="${28/1000} ${28/1000} ${28/1000}"
               matname="green_mat"
               rgba="0 1 0 1"
@@ -280,4 +305,5 @@
               iyx="${-29.757/1000000000}" iyy="${1819.588/1000000000}" iyz="${-43.683/1000000000}"
               izx="${-150.6/1000000000}" izy="${-43.683/1000000000}" izz="${5174.827/1000000000}"
+              size="${42.360/1000} ${62.867/1000} ${4.8/1000}"
               matname="red_mat"
               rgba="1 0 0 1"
@@ -291,4 +317,5 @@
               iyx="${3.957/1000000000}" iyy="${106.346/1000000000}" iyz="${13.142/1000000000}"
               izx="${-22.394/1000000000}" izy="${13.142/1000000000}" izz="${515.988/1000000000}"
+              size="${25/1000} ${35/1000} ${18/1000}"
               matname="blue_mat"
               rgba="0 0 1 1"
@@ -298,8 +325,9 @@
               origin_rpy="${0} ${pi/2} ${0}" origin_xyz="${0/1000} ${0} ${0/1000}"
               i_rpy="0 0 0" i_xyz="${7.859/1000} ${-6.38/1000} ${-15.22/1000}"
-              mass="${21.617/1000}"
+              mass="${35/1000}"
               ixx="${2815.705/1000000000}" ixy="${69.289/1000000000}" ixz="${-116.66/1000000000}"
               iyx="${69.289/1000000000}" iyy="${2928.22/1000000000}" iyz="${69.297/1000000000}"
               izx="${-116.66/1000000000}" izy="${69.297/1000000000}" izz="${2815.691/1000000000}"
+              size="${28/1000} ${28/1000} ${28/1000}"
               matname="green_mat"
               rgba="0 1 0 1"
@@ -313,4 +341,5 @@
               iyx="${87.11/1000000000}" iyy="${656.006/1000000000}" iyz="${-5.48/1000000000}"
               izx="${-66.883/1000000000}" izy="${-5.48/1000000000}" izz="${1381.079/1000000000}"
+              size="${38/1000} ${19/1000} ${40/1000}"
               matname="red_mat"
               rgba="1 0 0 1"
@@ -320,8 +349,9 @@
               origin_rpy="${0} ${0} ${pi}" origin_xyz="${0/1000} ${0/1000} ${0/1000}"
               i_rpy="0 0 0" i_xyz="${-0.000179884/1000} ${-5.05362/1000} ${-0.931856/1000}"
-              mass="${13/1000}"
-              ixx="${706.436/1000000000}" ixy="${0.008/1000000000}" ixz="${-0.017/1000000000}"
-              iyx="${0.008/1000000000}" iyy="${474.385/1000000000}" iyz="${-26.956/1000000000}"
-              izx="${-0.017/1000000000}" izy="${-26.956/1000000000}" izz="${410.689/1000000000}"
+              mass="${15/1000}"
+              ixx="${706.436/1000000000}" ixy="${0.008/1000000000}" ixz="${-0.017/1000000000}"
+              iyx="${0.008/1000000000}" iyy="${474.385/1000000000}" iyz="${-26.956/1000000000}"
+              izx="${-0.017/1000000000}" izy="${-26.956/1000000000}" izz="${410.689/1000000000}"
+              size="${25/1000} ${12/1000} ${28/1000}"
               matname="blue_mat"
               rgba="0 0 1 1"
@@ -335,4 +365,5 @@
               iyx="${-1.876/1000000000}" iyy="${1194.088/1000000000}" iyz="${2.97/1000000000}"
               izx="${11.724/1000000000}" izy="${2.97/1000000000}" izz="${3147.051/1000000000}"
+              size="${40/1000} ${25/1000} ${45/1000}"
               matname="blue_mat"
               rgba="0 0 1 1"
@@ -342,8 +373,9 @@
               origin_rpy="${0} ${0} ${0}" origin_xyz="${-7.5/1000} ${0/1000} ${-7.5/1000}"
               i_rpy="0 0 0" i_xyz="${-0.323/1000} ${-0.327/1000} ${13.86/1000}"
-              mass="${21.617/1000}"
+              mass="${35/1000}"
               ixx="${2815.587/1000000000}" ixy="${116.787/1000000000}" ixz="${69.924/1000000000}"
               iyx="${116.787/1000000000}" iyy="${2815.587/1000000000}" iyz="${-69.924/1000000000}"
               izx="${69.924/1000000000}" izy="${-69.924/1000000000}" izz="${2927.98/1000000000}"
+              size="${28/1000} ${28/1000} ${28/1000}"
               matname="green_mat"
               rgba="0 1 0 1"
@@ -357,4 +389,5 @@
               iyx="${29.757/1000000000}" iyy="${1819.588/1000000000}" iyz="${-43.683/1000000000}"
               izx="${150.6/1000000000}" izy="${-43.683/1000000000}" izz="${5174.827/1000000000}"
+              size="${42.360/1000} ${62.867/1000} ${4.8/1000}"
               matname="red_mat"
               rgba="1 0 0 1"

File: plen_ros/urdf/plen_macro.xacro (robot description, xacro)
@@ -18,5 +18,5 @@
     </joint>
   </xacro:macro>
-  <xacro:macro name="mesh_link" params="name origin_xyz origin_rpy meshfile meshscale matname rgba mass i_xyz i_rpy ixx ixy ixz iyx iyy iyz izx izy izz">
+  <xacro:macro name="mesh_link" params="name origin_xyz origin_rpy meshfile meshscale size matname rgba mass i_xyz i_rpy ixx ixy ixz iyx iyy iyz izx izy izz">
     <link name="${name}">
       <visual>
@@ -32,5 +32,5 @@
         <origin rpy="${origin_rpy}" xyz="${origin_xyz}" />
         <geometry>
-          <mesh filename="${meshfile}" scale="${meshscale}"/>
+          <box size="${size}" />
         </geometry>
       </collision>
