Commit message: hip boxes successfully placed. will now repeat method for all links. may need to adjust box sizes

File: plen_ros/urdf/plen.urdf.xacro (robot description, xacro)
@@ -16,4 +16,5 @@
               iyx="${85.607/1000000000}" iyy="${3.183e4/1000000000}" iyz="${25.76/1000000000}"
               izx="${825.993/1000000000}" izy="${25.76/1000000000}" izz="${2.994e4/1000000000}"
+              c_xyz="${0} ${0} ${0/2000}"
               size="${65/1000} ${48/1000} ${75/1000}"
               matname="red_mat"
@@ -28,4 +29,5 @@
               iyx="${0.013/1000000000}" iyy="${6582.133/1000000000}" iyz="${-0.022/1000000000}"
               izx="${349.218/1000000000}" izy="${-0.022/1000000000}" izz="${7690.404/1000000000}"
+              c_xyz="${0} ${0} ${0/2000}"
               size="${40/1000} ${40/1000} ${40/1000}"
               matname="green_mat"
@@ -40,4 +42,5 @@
               iyx="${0.008/1000000000}" iyy="${474.385/1000000000}" iyz="${-26.956/1000000000}"
               izx="${-0.017/1000000000}" izy="${-26.956/1000000000}" izz="${410.689/1000000000}"
+              c_xyz="${0} ${0} ${0/2000}"
               size="${25/1000} ${12/1000} ${28/1000}"
               matname="blue_mat"
@@ -52,4 +55,5 @@
               iyx="${0.008/1000000000}" iyy="${474.385/1000000000}" iyz="${-26.956/1000000000}"
               izx="${-0.017/1000000000}" izy="${-26.956/1000000000}" izz="${410.689/1000000000}"
+              c_xyz="${0} ${0} ${0/2000}"
               size="${25/1000} ${12/1000} ${28/1000}"
               matname="blue_mat"
@@ -64,4 +68,5 @@
               iyx="${0.008/1000000000}" iyy="${474.385/1000000000}" iyz="${-26.956/1000000000}"
               izx="${-0.017/1000000000}" izy="${-26.956/1000000000}" izz="${410.689/1000000000}"
+              c_xyz="${0} ${0} ${0/2000}"
               size="${25/1000} ${12/1000} ${28/1000}"
               matname="blue_mat"
@@ -76,4 +81,5 @@
               iyx="${0.008/1000000000}" iyy="${474.385/1000000000}" iyz="${-26.956/1000000000}"
               izx="${-0.017/1000000000}" izy="${-26.956/1000000000}" izz="${410.689/1000000000}"
+              c_xyz="${0} ${0} ${0/2000}"
               size="${25/1000} ${12/1000} ${28/1000}"
               matname="blue_mat"
@@ -88,5 +94,6 @@
               iyx="${-17.907/1000000000}" iyy="${642.45/1000000000}" iyz="${-32.057/1000000000}"
               izx="${-3.73/1000000000}" izy="${-32.057/1000000000}" izz="${713.005/1000000000}"
-              size="${25/1000} ${35/1000} ${18/1000}"
+             c_xyz="${0} ${0} ${0/2000}"
+             size="${25/1000} ${35/1000} ${18/1000}"
               matname="green_mat"
               rgba="0 1 0 1"
@@ -100,4 +107,5 @@
               iyx="${0.008/1000000000}" iyy="${474.385/1000000000}" iyz="${-26.956/1000000000}"
               izx="${-0.017/1000000000}" izy="${-26.956/1000000000}" izz="${410.689/1000000000}"
+              c_xyz="${0} ${0} ${0/2000}"
               size="${25/1000} ${12/1000} ${28/1000}"
               matname="blue_mat"
@@ -112,4 +120,5 @@
               iyx="${242.813/1000000000}" iyy="${858.371/1000000000}" iyz="${-0.939/1000000000}"
               izx="${3.398/1000000000}" izy="${-0.939/1000000000}" izz="${2003.835/1000000000}"
+              c_xyz="${0} ${0} ${0/2000}"
               size="${35/1000} ${15/1000} ${50/1000}"
               matname="red_mat"
@@ -124,4 +133,5 @@
               iyx="${0.008/1000000000}" iyy="${474.385/1000000000}" iyz="${-26.956/1000000000}"
               izx="${-0.017/1000000000}" izy="${-26.956/1000000000}" izz="${410.689/1000000000}"
+              c_xyz="${0} ${0} ${0/2000}"
               size="${25/1000} ${12/1000} ${28/1000}"
               matname="blue_mat"
@@ -136,4 +146,5 @@
               iyx="${-22.513/1000000000}" iyy="${168.898/1000000000}" iyz="${0.0004/1000000000}"
               izx="${-0.00015/1000000000}" izy="${0.0004/1000000000}" izz="${791.489/1000000000}"
+              c_xyz="${0} ${0} ${0/2000}"
               size="${14/1000} ${34/1000} ${27/1000}"
               matname="green_mat"
@@ -148,4 +159,5 @@
               iyx="${0.000002/1000000000}" iyy="${1619.378/1000000000}" iyz="${0.000004/1000000000}"
               izx="${-4.196/1000000000}" izy="${0.000004/1000000000}" izz="${1315.428/1000000000}"
+              c_xyz="${0} ${0} ${0/2000}"
               size="${19/1000} ${34/1000} ${35/1000}"
               matname="red_mat"
@@ -160,4 +172,5 @@
               iyx="${-17.907/1000000000}" iyy="${642.45/1000000000}" iyz="${-32.057/1000000000}"
               izx="${-3.73/1000000000}" izy="${-32.057/1000000000}" izz="${713.005/1000000000}"
+              c_xyz="${0} ${0} ${0/2000}"
               size="${25/1000} ${35/1000} ${18/1000}"
               matname="green_mat"
@@ -172,4 +185,5 @@
               iyx="${0.008/1000000000}" iyy="${474.385/1000000000}" iyz="${-26.956/1000000000}"
               izx="${-0.017/1000000000}" izy="${-26.956/1000000000}" izz="${410.689/1000000000}"
+              c_xyz="${0} ${0} ${0/2000}"
               size="${25/1000} ${12/1000} ${28/1000}"
               matname="blue_mat"
@@ -184,4 +198,5 @@
               iyx="${242.813/1000000000}" iyy="${858.371/1000000000}" iyz="${-0.939/1000000000}"
               izx="${3.398/1000000000}" izy="${-0.939/1000000000}" izz="${2003.835/1000000000}"
+              c_xyz="${0} ${0} ${0/2000}"
               size="${35/1000} ${15/1000} ${50/1000}"
               matname="red_mat"
@@ -196,4 +211,5 @@
               iyx="${0.008/1000000000}" iyy="${474.385/1000000000}" iyz="${-26.956/1000000000}"
               izx="${-0.017/1000000000}" izy="${-26.956/1000000000}" izz="${410.689/1000000000}"
+              c_xyz="${0} ${0} ${0/2000}"
               size="${25/1000} ${12/1000} ${28/1000}"
               matname="blue_mat"
@@ -208,4 +224,5 @@
               iyx="${-22.513/1000000000}" iyy="${168.898/1000000000}" iyz="${0.0004/1000000000}"
               izx="${-0.00015/1000000000}" izy="${0.0004/1000000000}" izz="${791.489/1000000000}"
+              c_xyz="${0} ${0} ${0/2000}"
               size="${14/1000} ${34/1000} ${27/1000}"
               matname="green_mat"
@@ -220,4 +237,5 @@
               iyx="${0.000002/1000000000}" iyy="${1619.378/1000000000}" iyz="${0.000004/1000000000}"
               izx="${-4.196/1000000000}" izy="${0.000004/1000000000}" izz="${1315.428/1000000000}"
+              c_xyz="${0} ${0} ${0/2000}"
               size="${19/1000} ${34/1000} ${35/1000}"
               matname="red_mat"
@@ -232,4 +250,5 @@
               iyx="${3.957/1000000000}" iyy="${106.346/1000000000}" iyz="${-13.142/1000000000}"
               izx="${22.394/1000000000}" izy="${-13.142/1000000000}" izz="${515.988/1000000000}"
+              c_xyz="${0} ${0} ${-18/2000}"
               size="${25/1000} ${35/1000} ${18/1000}"
               matname="blue_mat"
@@ -244,4 +263,5 @@
               iyx="${116.787/1000000000}" iyy="${2815.587/1000000000}" iyz="${-69.924/1000000000}"
               izx="${69.924/1000000000}" izy="${-69.924/1000000000}" izz="${2927.98/1000000000}"
+              c_xyz="${0} ${0} ${0/2000}"
               size="${28/1000} ${28/1000} ${28/1000}"
               matname="green_mat"
@@ -257,4 +277,5 @@
               iyx="${5.48/1000000000}" iyy="${656.006/1000000000}" iyz="${87.11/1000000000}"
               izx="${66.883/1000000000}" izy="${87.11/1000000000}" izz="${923.038/1000000000}"
+              c_xyz="${0} ${0} ${0/2000}"
               size="${38/1000} ${19/1000} ${40/1000}"
               matname="red_mat"
@@ -269,4 +290,5 @@
               iyx="${0.008/1000000000}" iyy="${474.385/1000000000}" iyz="${-26.956/1000000000}"
               izx="${-0.017/1000000000}" izy="${-26.956/1000000000}" izz="${410.689/1000000000}"
+              c_xyz="${0} ${0} ${0/2000}"
               size="${25/1000} ${12/1000} ${28/1000}"
               matname="blue_mat"
@@ -281,4 +303,5 @@
               iyx="${-1.876/1000000000}" iyy="${1194.088/1000000000}" iyz="${2.97/1000000000}"
               izx="${11.724/1000000000}" izy="${2.97/1000000000}" izz="${3147.051/1000000000}"
+              c_xyz="${0} ${0} ${0/2000}"
               size="${40/1000} ${25/1000} ${45/1000}"
               matname="blue_mat"
@@ -293,4 +316,5 @@
               iyx="${69.289/1000000000}" iyy="${2928.22/1000000000}" iyz="${69.297/1000000000}"
               izx="${-116.66/1000000000}" izy="${69.297/1000000000}" izz="${2815.691/1000000000}"
+              c_xyz="${0} ${0} ${0/2000}"
               size="${28/1000} ${28/1000} ${28/1000}"
               matname="green_mat"
@@ -305,4 +329,5 @@
               iyx="${-29.757/1000000000}" iyy="${1819.588/1000000000}" iyz="${-43.683/1000000000}"
               izx="${-150.6/1000000000}" izy="${-43.683/1000000000}" izz="${5174.827/1000000000}"
+              c_xyz="${0} ${0} ${0/2000}"
               size="${42.360/1000} ${62.867/1000} ${4.8/1000}"
               matname="red_mat"
@@ -317,4 +342,5 @@
               iyx="${3.957/1000000000}" iyy="${106.346/1000000000}" iyz="${13.142/1000000000}"
               izx="${-22.394/1000000000}" izy="${13.142/1000000000}" izz="${515.988/1000000000}"
+              c_xyz="${0} ${0} ${-18/2000}"
               size="${25/1000} ${35/1000} ${18/1000}"
               matname="blue_mat"
@@ -329,4 +355,5 @@
               iyx="${69.289/1000000000}" iyy="${2928.22/1000000000}" iyz="${69.297/1000000000}"
               izx="${-116.66/1000000000}" izy="${69.297/1000000000}" izz="${2815.691/1000000000}"
+              c_xyz="${0} ${0} ${0/2000}"
               size="${28/1000} ${28/1000} ${28/1000}"
               matname="green_mat"
@@ -341,4 +368,5 @@
               iyx="${87.11/1000000000}" iyy="${656.006/1000000000}" iyz="${-5.48/1000000000}"
               izx="${-66.883/1000000000}" izy="${-5.48/1000000000}" izz="${1381.079/1000000000}"
+              c_xyz="${0} ${0} ${0/2000}"
               size="${38/1000} ${19/1000} ${40/1000}"
               matname="red_mat"
@@ -353,4 +381,5 @@
               iyx="${0.008/1000000000}" iyy="${474.385/1000000000}" iyz="${-26.956/1000000000}"
               izx="${-0.017/1000000000}" izy="${-26.956/1000000000}" izz="${410.689/1000000000}"
+              c_xyz="${0} ${0} ${0/2000}"
               size="${25/1000} ${12/1000} ${28/1000}"
               matname="blue_mat"
@@ -365,4 +394,5 @@
               iyx="${-1.876/1000000000}" iyy="${1194.088/1000000000}" iyz="${2.97/1000000000}"
               izx="${11.724/1000000000}" izy="${2.97/1000000000}" izz="${3147.051/1000000000}"
+              c_xyz="${0} ${0} ${0/2000}"
               size="${40/1000} ${25/1000} ${45/1000}"
               matname="blue_mat"
@@ -377,4 +407,5 @@
               iyx="${116.787/1000000000}" iyy="${2815.587/1000000000}" iyz="${-69.924/1000000000}"
               izx="${69.924/1000000000}" izy="${-69.924/1000000000}" izz="${2927.98/1000000000}"
+              c_xyz="${0} ${0} ${0/2000}"
               size="${28/1000} ${28/1000} ${28/1000}"
               matname="green_mat"
@@ -389,4 +420,5 @@
               iyx="${29.757/1000000000}" iyy="${1819.588/1000000000}" iyz="${-43.683/1000000000}"
               izx="${150.6/1000000000}" izy="${-43.683/1000000000}" izz="${5174.827/1000000000}"
+              c_xyz="${0} ${0} ${0/2000}"
               size="${42.360/1000} ${62.867/1000} ${4.8/1000}"
               matname="red_mat"

File: plen_ros/urdf/plen_macro.xacro (robot description, xacro)
@@ -18,5 +18,5 @@
     </joint>
   </xacro:macro>
-  <xacro:macro name="mesh_link" params="name origin_xyz origin_rpy meshfile meshscale size matname rgba mass i_xyz i_rpy ixx ixy ixz iyx iyy iyz izx izy izz">
+  <xacro:macro name="mesh_link" params="name origin_xyz origin_rpy meshfile meshscale size c_xyz matname rgba mass i_xyz i_rpy ixx ixy ixz iyx iyy iyz izx izy izz">
     <link name="${name}">
       <visual>
@@ -30,5 +30,5 @@
       </visual>
       <collision>
-        <origin rpy="${origin_rpy}" xyz="${origin_xyz}" />
+        <origin rpy="${origin_rpy}" xyz="${c_xyz}" />
         <geometry>
           <box size="${size}" />
