Commit message: used collision box dimensions for inertia. works nicely. May need to alter component masses after 3D print. still need to add battery.

File: plen_ros/urdf/plen.urdf.xacro (robot description, xacro)
@@ -11,9 +11,9 @@
   <mesh_link name="torso"
               origin_rpy="0 0 0" origin_xyz="0 0 0"
-              i_rpy="0 0 0" i_xyz="${2.641/1000} ${-0.668/1000} ${1.187/1000}"
+              i_rpy="0 0 0" i_xyz="${0/8000} ${0} ${0/2000}"
               mass="${43.968/1000}"
-              ixx="${4.598*10000/1000000000}" ixy="${85.607/1000000000}" ixz="${825.993/1000000000}"
-              iyx="${85.607/1000000000}" iyy="${3.183*10000/1000000000}" iyz="${25.76/1000000000}"
-              izx="${825.993/1000000000}" izy="${25.76/1000000000}" izz="${2.994*10000/1000000000}"
+              ixx="${43.968*(45*45+75*75)/(12*1000000000)}" ixy="${0}" ixz="${0}"
+              iyy="${43.968*(45*45+75*75)/(12*1000000000)}" iyz="${0}"
+              izz="${43.968*(45*45+48*48)/(12*1000000000)}"
               c_xyz="${0/8000} ${0} ${0/2000}"
               size="${45/1000} ${48/1000} ${75/1000}"
@@ -24,9 +24,9 @@
   <mesh_link name="head"
               origin_rpy="0 0 0" origin_xyz="0 0 0"
-              i_rpy="0 0 0" i_xyz="${1.004/1000} ${0.1269/1000} ${1.697/1000}"
-              mass="${19.57/1000}"
-              ixx="${6075.414/1000000000}" ixy="${0.013/1000000000}" ixz="${349.218/1000000000}"
-              iyx="${0.013/1000000000}" iyy="${6582.133/1000000000}" iyz="${-0.022/1000000000}"
-              izx="${349.218/1000000000}" izy="${-0.022/1000000000}" izz="${7690.404/1000000000}"
+              i_rpy="0 0 0" i_xyz="${0/8000} ${0} ${0/2000}"
+              mass="${10/1000}"
+              ixx="${10*(40*40+40*40)/(12*1000000000)}" ixy="${0}" ixz="${0}"
+              iyy="${10*(40*40+40*40)/(12*1000000000)}" iyz="${0}"
+              izz="${10*(40*40+40*40)/(12*1000000000)}"
               c_xyz="${0} ${0} ${0/2000}"
               size="${40/1000} ${40/1000} ${40/1000}"
@@ -37,9 +37,9 @@
   <mesh_link name="rt_servo"
               origin_rpy="0 0 ${pi}" origin_xyz="0 0 0"
-              i_rpy="0 0 0" i_xyz="${-0.000179884/1000} ${-5.05362/1000} ${-0.931856/1000}"
-              mass="${15/1000}"
-              ixx="${706.436/1000000000}" ixy="${0.008/1000000000}" ixz="${-0.017/1000000000}"
-              iyx="${0.008/1000000000}" iyy="${474.385/1000000000}" iyz="${-26.956/1000000000}"
-              izx="${-0.017/1000000000}" izy="${-26.956/1000000000}" izz="${410.689/1000000000}"
+              i_rpy="0 0 0" i_xyz="${0} ${25/4000} ${0/2000}"
+              mass="${12/1000}"
+              ixx="${12*(12*12+25*25)/(12*1000000000)}" ixy="${0}" ixz="${0}"
+              iyy="${12*(12*12+25*25)/(12*1000000000)}" iyz="${0}"
+              izz="${12*(12*12+25*25)/(12*1000000000)}"
               c_xyz="${0} ${25/4000} ${0/2000}"
               size="${12/1000} ${25/1000} ${25/1000}"
@@ -50,9 +50,9 @@
   <mesh_link name="lt_servo"
               origin_rpy="0 0 ${pi}" origin_xyz="0 0 0"
-              i_rpy="0 0 0" i_xyz="${-0.000179884/1000} ${-5.05362/1000} ${-0.931856/1000}"
-              mass="${15/1000}"
-              ixx="${706.436/1000000000}" ixy="${0.008/1000000000}" ixz="${-0.017/1000000000}"
-              iyx="${0.008/1000000000}" iyy="${474.385/1000000000}" iyz="${-26.956/1000000000}"
-              izx="${-0.017/1000000000}" izy="${-26.956/1000000000}" izz="${410.689/1000000000}"
+              i_rpy="0 0 0" i_xyz="${0} ${25/4000} ${0/2000}"
+              mass="${12/1000}"
+              ixx="${12*(12*12+25*25)/(12*1000000000)}" ixy="${0}" ixz="${0}"
+              iyy="${12*(12*12+25*25)/(12*1000000000)}" iyz="${0}"
+              izz="${12*(12*12+25*25)/(12*1000000000)}"
               c_xyz="${0} ${25/4000} ${0/2000}"
               size="${12/1000} ${25/1000} ${25/1000}"
@@ -63,9 +63,9 @@
   <mesh_link name="rb_servo"
               origin_rpy="0 0 ${pi}" origin_xyz="0 0 0"
-              i_rpy="0 0 0" i_xyz="${-0.000179884/1000} ${-5.05362/1000} ${-0.931856/1000}"
-              mass="${13/1000}"
-              ixx="${706.436/1000000000}" ixy="${0.008/1000000000}" ixz="${-0.017/1000000000}"
-              iyx="${0.008/1000000000}" iyy="${474.385/1000000000}" iyz="${-26.956/1000000000}"
-              izx="${-0.017/1000000000}" izy="${-26.956/1000000000}" izz="${410.689/1000000000}"
+              i_rpy="0 0 0" i_xyz="${0} ${25/4000} ${0/2000}"
+              mass="${12/1000}"
+              ixx="${12*(12*12+25*25)/(12*1000000000)}" ixy="${0}" ixz="${0}"
+              iyy="${12*(12*12+25*25)/(12*1000000000)}" iyz="${0}"
+              izz="${12*(12*12+25*25)/(12*1000000000)}"
               c_xyz="${0} ${25/4000} ${0/2000}"
               size="${12/1000} ${25/1000} ${25/1000}"
@@ -76,9 +76,9 @@
   <mesh_link name="lb_servo"
               origin_rpy="0 0 ${pi}" origin_xyz="0 0 0"
-              i_rpy="0 0 0" i_xyz="${-0.000179884/1000} ${-5.05362/1000} ${-0.931856/1000}"
-              mass="${15/1000}"
-              ixx="${706.436/1000000000}" ixy="${0.008/1000000000}" ixz="${-0.017/1000000000}"
-              iyx="${0.008/1000000000}" iyy="${474.385/1000000000}" iyz="${-26.956/1000000000}"
-              izx="${-0.017/1000000000}" izy="${-26.956/1000000000}" izz="${410.689/1000000000}"
+              i_rpy="0 0 0" i_xyz="${0} ${25/4000} ${0/2000}"
+              mass="${12/1000}"
+              ixx="${12*(12*12+25*25)/(12*1000000000)}" ixy="${0}" ixz="${0}"
+              iyy="${12*(12*12+25*25)/(12*1000000000)}" iyz="${0}"
+              izz="${12*(12*12+25*25)/(12*1000000000)}"
               c_xyz="${0} ${25/4000} ${0/2000}"
               size="${12/1000} ${25/1000} ${25/1000}"
@@ -89,9 +89,9 @@
   <mesh_link name="r_shoulder"
               origin_rpy="0 0 ${0}" origin_xyz="0 0 0"
-              i_rpy="0 0 0" i_xyz="${-0.6586/1000} ${-3.013/1000} ${-23.9872/1000}"
+              i_rpy="0 0 0" i_xyz="${0} ${0} ${25/2000}"
               mass="${2.954/1000}"
-              ixx="${176.048/1000000000}" ixy="${-17.907/1000000000}" ixz="${-3.73/1000000000}"
-              iyx="${-17.907/1000000000}" iyy="${642.45/1000000000}" iyz="${-32.057/1000000000}"
-              izx="${-3.73/1000000000}" izy="${-32.057/1000000000}" izz="${713.005/1000000000}"
+              ixx="${2.954*(18*18+25*25)/(12*1000000000)}" ixy="${0}" ixz="${0}"
+              iyy="${2.954*(18*18+25*25)/(12*1000000000)}" iyz="${0}"
+              izz="${2.954*(18*18+35*35)/(12*1000000000)}"
               c_xyz="${0} ${0} ${25/2000}"
               size="${18/1000} ${35/1000} ${25/1000}"
@@ -102,9 +102,9 @@
   <mesh_link name="rs_servo"
               origin_rpy="0 0 ${pi}" origin_xyz="0 0 0"
-              i_rpy="0 0 0" i_xyz="${-0.000179884/1000} ${-5.05362/1000} ${-0.931856/1000}"
-              mass="${15/1000}"
-              ixx="${706.436/1000000000}" ixy="${0.008/1000000000}" ixz="${-0.017/1000000000}"
-              iyx="${0.008/1000000000}" iyy="${474.385/1000000000}" iyz="${-26.956/1000000000}"
-              izx="${-0.017/1000000000}" izy="${-26.956/1000000000}" izz="${410.689/1000000000}"
+              i_rpy="0 0 0" i_xyz="${0} ${25/4000} ${0/2000}"
+              mass="${12/1000}"
+              ixx="${12*(12*12+25*25)/(12*1000000000)}" ixy="${0}" ixz="${0}"
+              iyy="${12*(12*12+25*25)/(12*1000000000)}" iyz="${0}"
+              izz="${12*(12*12+25*25)/(12*1000000000)}"
               c_xyz="${0} ${25/4000} ${0/2000}"
               size="${12/1000} ${25/1000} ${25/1000}"
@@ -115,9 +115,9 @@
   <mesh_link name="r_arm"
               origin_rpy="0 0 ${0}" origin_xyz="0 0 0"
-              i_rpy="0 0 0" i_xyz="${-77.4619/1000} ${15.9214/1000} ${-34.001/1000}"
+              i_rpy="0 0 0" i_xyz="${0} ${0} ${0/2000}"
               mass="${5.091/1000}"
-              ixx="${1485.346/1000000000}" ixy="${242.813/1000000000}" ixz="${3.398/1000000000}"
-              iyx="${242.813/1000000000}" iyy="${858.371/1000000000}" iyz="${-0.939/1000000000}"
-              izx="${3.398/1000000000}" izy="${-0.939/1000000000}" izz="${2003.835/1000000000}"
+              ixx="${5.091*(15*15+50*50)/(12*1000000000)}" ixy="${0}" ixz="${0}"
+              iyy="${5.091*(15*15+50*50)/(12*1000000000)}" iyz="${0}"
+              izz="${5.091*(15*15+35*35)/(12*1000000000)}"
               c_xyz="${0} ${0} ${0/2000}"
               size="${15/1000} ${35/1000} ${50/1000}"
@@ -128,9 +128,9 @@
   <mesh_link name="re_servo"
               origin_rpy="0 0 ${pi}" origin_xyz="0 0 0"
-              i_rpy="0 0 0" i_xyz="${-0.000179884/1000} ${-5.05362/1000} ${-0.931856/1000}"
-              mass="${15/1000}"
-              ixx="${706.436/1000000000}" ixy="${0.008/1000000000}" ixz="${-0.017/1000000000}"
-              iyx="${0.008/1000000000}" iyy="${474.385/1000000000}" iyz="${-26.956/1000000000}"
-              izx="${-0.017/1000000000}" izy="${-26.956/1000000000}" izz="${410.689/1000000000}"
+              i_rpy="0 0 0" i_xyz="${0} ${25/4000} ${0/2000}"
+              mass="${12/1000}"
+              ixx="${12*(12*12+25*25)/(12*1000000000)}" ixy="${0}" ixz="${0}"
+              iyy="${12*(12*12+25*25)/(12*1000000000)}" iyz="${0}"
+              izz="${12*(12*12+25*25)/(12*1000000000)}"
               c_xyz="${0} ${25/4000} ${0/2000}"
               size="${12/1000} ${25/1000} ${25/1000}"
@@ -141,9 +141,9 @@
   <mesh_link name="r_elbow"
               origin_rpy="0 0 ${0}" origin_xyz="${-13.5/1000} 0 0"
-              i_rpy="0 0 0" i_xyz="${3.8099/1000} ${0.4455/1000} ${-0.0457/1000}"
+              i_rpy="0 0 0" i_xyz="${-27/4000} ${0} ${0/2000}"
               mass="${3.046/1000}"
-              ixx="${717.001/1000000000}" ixy="${-22.513/1000000000}" ixz="${-0.00015/1000000000}"
-              iyx="${-22.513/1000000000}" iyy="${168.898/1000000000}" iyz="${0.0004/1000000000}"
-              izx="${-0.00015/1000000000}" izy="${0.0004/1000000000}" izz="${791.489/1000000000}"
+              ixx="${3.046*(27*27+14*14)/(12*1000000000)}" ixy="${0}" ixz="${0}"
+              iyy="${3.046*(27*27+14*14)/(12*1000000000)}" iyz="${0}"
+              izz="${3.046*(27*27+34*34)/(12*1000000000)}"
               c_xyz="${-27/4000} ${0} ${0/2000}"
               size="${27/1000} ${34/1000} ${14/1000}"
@@ -154,9 +154,9 @@
   <mesh_link name="r_hand"
               origin_rpy="0 0 ${0}" origin_xyz="${0/1000} 0 0"
-              i_rpy="0 0 0" i_xyz="${-1.228/1000} ${0.00071/1000} ${0.6389/1000}"
+              i_rpy="0 0 0" i_xyz="${0} ${0} ${0/2000}"
               mass="${8.305/1000}"
-              ixx="${2276.89/1000000000}" ixy="${0.000002/1000000000}" ixz="${-4.196/1000000000}"
-              iyx="${0.000002/1000000000}" iyy="${1619.378/1000000000}" iyz="${0.000004/1000000000}"
-              izx="${-4.196/1000000000}" izy="${0.000004/1000000000}" izz="${1315.428/1000000000}"
+              ixx="${8.305*(19*19+35*35)/(12*1000000000)}" ixy="${0}" ixz="${0}"
+              iyy="${8.305*(19*19+35*35)/(12*1000000000)}" iyz="${0}"
+              izz="${8.305*(19*19+34*34)/(12*1000000000)}"
               c_xyz="${0} ${0} ${0/2000}"
               size="${19/1000} ${34/1000} ${35/1000}"
@@ -167,9 +167,9 @@
   <mesh_link name="l_shoulder"
               origin_rpy="0 0 ${0}" origin_xyz="0 0 0"
-              i_rpy="0 0 0" i_xyz="${-0.6586/1000} ${-3.013/1000} ${-23.9872/1000}"
+              i_rpy="0 0 0" i_xyz="${0} ${0} ${25/2000}"
               mass="${2.954/1000}"
-              ixx="${176.048/1000000000}" ixy="${-17.907/1000000000}" ixz="${-3.73/1000000000}"
-              iyx="${-17.907/1000000000}" iyy="${642.45/1000000000}" iyz="${-32.057/1000000000}"
-              izx="${-3.73/1000000000}" izy="${-32.057/1000000000}" izz="${713.005/1000000000}"
+              ixx="${2.954*(18*18+25*25)/(12*1000000000)}" ixy="${0}" ixz="${0}"
+              iyy="${2.954*(18*18+25*25)/(12*1000000000)}" iyz="${0}"
+              izz="${2.954*(18*18+35*35)/(12*1000000000)}"
               c_xyz="${0} ${0} ${25/2000}"
               size="${18/1000} ${35/1000} ${25/1000}"
@@ -180,9 +180,9 @@
   <mesh_link name="ls_servo"
               origin_rpy="0 0 ${pi}" origin_xyz="0 0 0"
-              i_rpy="0 0 0" i_xyz="${-0.000179884/1000} ${-5.05362/1000} ${-0.931856/1000}"
-              mass="${15/1000}"
-              ixx="${706.436/1000000000}" ixy="${0.008/1000000000}" ixz="${-0.017/1000000000}"
-              iyx="${0.008/1000000000}" iyy="${474.385/1000000000}" iyz="${-26.956/1000000000}"
-              izx="${-0.017/1000000000}" izy="${-26.956/1000000000}" izz="${410.689/1000000000}"
+              i_rpy="0 0 0" i_xyz="${0} ${25/4000} ${0/2000}"
+              mass="${12/1000}"
+              ixx="${12*(12*12+25*25)/(12*1000000000)}" ixy="${0}" ixz="${0}"
+              iyy="${12*(12*12+25*25)/(12*1000000000)}" iyz="${0}"
+              izz="${12*(12*12+25*25)/(12*1000000000)}"
               c_xyz="${0} ${25/4000} ${0/2000}"
               size="${12/1000} ${25/1000} ${25/1000}"
@@ -193,9 +193,9 @@
   <mesh_link name="l_arm"
               origin_rpy="0 0 ${0}" origin_xyz="0 0 0"
-              i_rpy="0 0 0" i_xyz="${-77.4619/1000} ${15.9214/1000} ${-34.001/1000}"
+              i_rpy="0 0 0" i_xyz="${0} ${0} ${0/2000}"
               mass="${5.091/1000}"
-              ixx="${1485.346/1000000000}" ixy="${242.813/1000000000}" ixz="${3.398/1000000000}"
-              iyx="${242.813/1000000000}" iyy="${858.371/1000000000}" iyz="${-0.939/1000000000}"
-              izx="${3.398/1000000000}" izy="${-0.939/1000000000}" izz="${2003.835/1000000000}"
+              ixx="${5.091*(15*15+50*50)/(12*1000000000)}" ixy="${0}" ixz="${0}"
+              iyy="${5.091*(15*15+50*50)/(12*1000000000)}" iyz="${0}"
+              izz="${5.091*(15*15+35*35)/(12*1000000000)}"
               c_xyz="${0} ${0} ${0/2000}"
               size="${15/1000} ${35/1000} ${50/1000}"
@@ -206,9 +206,9 @@
   <mesh_link name="le_servo"
               origin_rpy="0 0 ${pi}" origin_xyz="0 0 0"
-              i_rpy="0 0 0" i_xyz="${-0.000179884/1000} ${-5.05362/1000} ${-0.931856/1000}"
-              mass="${15/1000}"
-              ixx="${706.436/1000000000}" ixy="${0.008/1000000000}" ixz="${-0.017/1000000000}"
-              iyx="${0.008/1000000000}" iyy="${474.385/1000000000}" iyz="${-26.956/1000000000}"
-              izx="${-0.017/1000000000}" izy="${-26.956/1000000000}" izz="${410.689/1000000000}"
+              i_rpy="0 0 0" i_xyz="${0} ${25/4000} ${0/2000}"
+              mass="${12/1000}"
+              ixx="${12*(12*12+25*25)/(12*1000000000)}" ixy="${0}" ixz="${0}"
+              iyy="${12*(12*12+25*25)/(12*1000000000)}" iyz="${0}"
+              izz="${12*(12*12+25*25)/(12*1000000000)}"
               c_xyz="${0} ${25/4000} ${0/2000}"
               size="${12/1000} ${25/1000} ${25/1000}"
@@ -219,9 +219,9 @@
   <mesh_link name="l_elbow"
               origin_rpy="0 0 ${0}" origin_xyz="${-13.5/1000} 0 0"
-              i_rpy="0 0 0" i_xyz="${3.8099/1000} ${0.4455/1000} ${-0.0457/1000}"
+              i_rpy="0 0 0" i_xyz="${-27/4000} ${0} ${0/2000}"
               mass="${3.046/1000}"
-              ixx="${717.001/1000000000}" ixy="${-22.513/1000000000}" ixz="${-0.00015/1000000000}"
-              iyx="${-22.513/1000000000}" iyy="${168.898/1000000000}" iyz="${0.0004/1000000000}"
-              izx="${-0.00015/1000000000}" izy="${0.0004/1000000000}" izz="${791.489/1000000000}"
+              ixx="${3.046*(27*27+14*14)/(12*1000000000)}" ixy="${0}" ixz="${0}"
+              iyy="${3.046*(27*27+14*14)/(12*1000000000)}" iyz="${0}"
+              izz="${3.046*(27*27+34*34)/(12*1000000000)}"
               c_xyz="${-27/4000} ${0} ${0/2000}"
               size="${27/1000} ${34/1000} ${14/1000}"
@@ -232,9 +232,9 @@
   <mesh_link name="l_hand"
               origin_rpy="0 0 ${0}" origin_xyz="${0/1000} 0 0"
-              i_rpy="0 0 0" i_xyz="${-1.228/1000} ${0.00071/1000} ${0.6389/1000}"
+              i_rpy="0 0 0" i_xyz="${0} ${0} ${0/2000}"
               mass="${8.305/1000}"
-              ixx="${2276.89/1000000000}" ixy="${0.000002/1000000000}" ixz="${-4.196/1000000000}"
-              iyx="${0.000002/1000000000}" iyy="${1619.378/1000000000}" iyz="${0.000004/1000000000}"
-              izx="${-4.196/1000000000}" izy="${0.000004/1000000000}" izz="${1315.428/1000000000}"
+              ixx="${8.305*(19*19+35*35)/(12*1000000000)}" ixy="${0}" ixz="${0}"
+              iyy="${8.305*(19*19+35*35)/(12*1000000000)}" iyz="${0}"
+              izz="${8.305*(19*19+34*34)/(12*1000000000)}"
               c_xyz="${0} ${0} ${0/2000}"
               size="${19/1000} ${34/1000} ${35/1000}"
@@ -245,9 +245,9 @@
   <mesh_link name="r_hip"
               origin_rpy="${pi} ${0} ${pi}" origin_xyz="${0/1000} ${0/1000} ${0/1000}"
-              i_rpy="0 0 0" i_xyz="${-1.14/1000} ${0.586/1000} ${4.525/1000}"
+              i_rpy="0 0 0" i_xyz="${0} ${0} ${-18/2000}"
               mass="${2.568/1000}"
-              ixx="${528.595/1000000000}" ixy="${3.957/1000000000}" ixz="${22.394/1000000000}"
-              iyx="${3.957/1000000000}" iyy="${106.346/1000000000}" iyz="${-13.142/1000000000}"
-              izx="${22.394/1000000000}" izy="${-13.142/1000000000}" izz="${515.988/1000000000}"
+              ixx="${2.568*(25*25+18*18)/(12*1000000000)}" ixy="${0}" ixz="${0}"
+              iyy="${2.568*(25*25+18*18)/(12*1000000000)}" iyz="${0}"
+              izz="${2.568*(25*25+35*35)/(12*1000000000)}"
               c_xyz="${0} ${0} ${-18/2000}"
               size="${25/1000} ${35/1000} ${18/1000}"
@@ -258,9 +258,9 @@
   <mesh_link name="r_thigh"
               origin_rpy="${0} ${0} ${0}" origin_xyz="${-7.5/1000} ${0} ${-7.5/1000}"
-              i_rpy="0 0 0" i_xyz="${-0.323/1000} ${-0.327/1000} ${13.86/1000}"
-              mass="${35/1000}"
-              ixx="${2815.587/1000000000}" ixy="${116.787/1000000000}" ixz="${69.924/1000000000}"
-              iyx="${116.787/1000000000}" iyy="${2815.587/1000000000}" iyz="${-69.924/1000000000}"
-              izx="${69.924/1000000000}" izy="${-69.924/1000000000}" izz="${2927.98/1000000000}"
+              i_rpy="0 0 0" i_xyz="${-14/2000} ${0} ${14/2000}"
+              mass="${40/1000}"
+              ixx="${40*(28*28+28*28)/(12*1000000000)}" ixy="${0}" ixz="${0}"
+              iyy="${40*(28*28+28*28)/(12*1000000000)}" iyz="${0}"
+              izz="${40*(28*28+28*28)/(12*1000000000)}"
               c_xyz="${-14/2000} ${0} ${14/2000}"
               size="${28/1000} ${28/1000} ${28/1000}"
@@ -272,9 +272,9 @@
   <mesh_link name="r_knee"
               origin_rpy="${0} ${0} ${0}" origin_xyz="${0/1000} ${0/1000} ${0/1000}"
-              i_rpy="0 0 0" i_xyz="${3.0845/1000} ${1.595/1000} ${15.504/1000}"
+              i_rpy="0 0 0" i_xyz="${35/2000} ${-30/2000} ${0/2000}"
               mass="${5.004/1000}"
-              ixx="${1381.079/1000000000}" ixy="${5.48/1000000000}" ixz="${66.883/1000000000}"
-              iyx="${5.48/1000000000}" iyy="${656.006/1000000000}" iyz="${87.11/1000000000}"
-              izx="${66.883/1000000000}" izy="${87.11/1000000000}" izz="${923.038/1000000000}"
+              ixx="${5.004*(38*38+24*24)/(12*1000000000)}" ixy="${0}" ixz="${0}"
+              iyy="${5.004*(38*38+24*24)/(12*1000000000)}" iyz="${0}"
+              izz="${5.004*(38*38+30*30)/(12*1000000000)}"
               c_xyz="${35/2000} ${-30/2000} ${0/2000}"
               size="${38/1000} ${30/1000} ${24/1000}"
@@ -284,10 +284,10 @@
               meshscale="0.001 0.001 0.001" />
   <mesh_link name="r_knee_servo"
-              origin_rpy="${0} ${0} ${pi}" origin_xyz="${0/1000} ${0/1000} ${0/1000}"
-              i_rpy="0 0 0" i_xyz="${-0.000179884/1000} ${-5.05362/1000} ${-0.931856/1000}"
-              mass="${15/1000}"
-              ixx="${706.436/1000000000}" ixy="${0.008/1000000000}" ixz="${-0.017/1000000000}"
-              iyx="${0.008/1000000000}" iyy="${474.385/1000000000}" iyz="${-26.956/1000000000}"
-              izx="${-0.017/1000000000}" izy="${-26.956/1000000000}" izz="${410.689/1000000000}"
+              origin_rpy="0 0 ${pi}" origin_xyz="0 0 0"
+              i_rpy="0 0 0" i_xyz="${0} ${25/4000} ${0/2000}"
+              mass="${12/1000}"
+              ixx="${12*(12*12+25*25)/(12*1000000000)}" ixy="${0}" ixz="${0}"
+              iyy="${12*(12*12+25*25)/(12*1000000000)}" iyz="${0}"
+              izz="${12*(12*12+25*25)/(12*1000000000)}"
               c_xyz="${0} ${25/4000} ${0/2000}"
               size="${12/1000} ${25/1000} ${25/1000}"
@@ -298,9 +298,9 @@
   <mesh_link name="r_shin"
               origin_rpy="0 ${0} ${0}" origin_xyz="${16.8/1000} ${0} ${-9.1/1000}"
-              i_rpy="0 0 0" i_xyz="${0.233/1000} ${-1.209/1000} ${8.78/1000}"
+              i_rpy="0 0 0" i_xyz="${36/2000} ${0} ${8/2000}"
               mass="${6.965/1000}"
-              ixx="${2533.205/1000000000}" ixy="${-1.876/1000000000}" ixz="${11.742/1000000000}"
-              iyx="${-1.876/1000000000}" iyy="${1194.088/1000000000}" iyz="${2.97/1000000000}"
-              izx="${11.724/1000000000}" izy="${2.97/1000000000}" izz="${3147.051/1000000000}"
+              ixx="${6.965*(45*45+23*23)/(12*1000000000)}" ixy="${0}" ixz="${0}"
+              iyy="${6.965*(45*45+23*23)/(12*1000000000)}" iyz="${0}"
+              izz="${6.965*(45*45+40*40)/(12*1000000000)}"
               c_xyz="${36/2000} ${0} ${8/2000}"
               size="${45/1000} ${40/1000} ${23/1000}"
@@ -311,9 +311,9 @@
   <mesh_link name="r_ankle"
               origin_rpy="${0} ${0} ${0}" origin_xyz="${0/1000} ${0/1000} ${0/1000}"
-              i_rpy="0 0 0" i_xyz="${7.859/1000} ${-6.38/1000} ${-15.22/1000}"
-              mass="${35/1000}"
-              ixx="${2815.705/1000000000}" ixy="${69.289/1000000000}" ixz="${-116.66/1000000000}"
-              iyx="${69.289/1000000000}" iyy="${2928.22/1000000000}" iyz="${69.297/1000000000}"
-              izx="${-116.66/1000000000}" izy="${69.297/1000000000}" izz="${2815.691/1000000000}"
+              i_rpy="0 0 0" i_xyz="${14/2000} ${-14/2000} ${-28/2000}"
+              mass="${40/1000}"
+              ixx="${40*(28*28+28*28)/(12*1000000000)}" ixy="${0}" ixz="${0}"
+              iyy="${40*(28*28+28*28)/(12*1000000000)}" iyz="${0}"
+              izz="${40*(28*28+28*28)/(12*1000000000)}"
               c_xyz="${14/2000} ${-14/2000} ${-28/2000}"
               size="${28/1000} ${28/1000} ${28/1000}"
@@ -324,9 +324,9 @@
   <mesh_link name="r_foot"
               origin_rpy="0 0 ${0}" origin_xyz="${-8.5/1000} 0 ${-19.8/1000}"
-              i_rpy="0 0 0" i_xyz="${0.961/1000} ${0.257/1000} ${4.745/1000}"
-              mass="${12.396/1000}"
-              ixx="${4031.152/1000000000}" ixy="${-29.757/1000000000}" ixz="${-150.6/1000000000}"
-              iyx="${-29.757/1000000000}" iyy="${1819.588/1000000000}" iyz="${-43.683/1000000000}"
-              izx="${-150.6/1000000000}" izy="${-43.683/1000000000}" izz="${5174.827/1000000000}"
+              i_rpy="0 0 0" i_xyz="${-37/4000} ${0} ${-9/1000}"
+              mass="${15/1000}"
+              ixx="${15*(41*41+4*4)/(12*1000000000)}" ixy="${0}" ixz="${0}"
+              iyy="${15*(41*41+4*4)/(12*1000000000)}" iyz="${0}"
+              izz="${15*(41*41+62.867*62.867)/(12*1000000000)}"
               c_xyz="${-37/4000} ${0} ${-17/1000}"
               size="${41/1000} ${62.867/1000} ${4/1000}"
@@ -337,9 +337,9 @@
   <mesh_link name="l_hip"
               origin_rpy="${0} ${0} ${pi}" origin_xyz="${0/1000} ${0/1000} ${1/1000}"
-              i_rpy="0 0 0" i_xyz="${-1.14/1000} ${0.585/1000} ${-5.325/1000}"
+              i_rpy="0 0 0" i_xyz="${0} ${0} ${-18/2000}"
               mass="${2.568/1000}"
-              ixx="${528.595/1000000000}" ixy="${3.957/1000000000}" ixz="${-22.394/1000000000}"
-              iyx="${3.957/1000000000}" iyy="${106.346/1000000000}" iyz="${13.142/1000000000}"
-              izx="${-22.394/1000000000}" izy="${13.142/1000000000}" izz="${515.988/1000000000}"
+              ixx="${2.568*(25*25+18*18)/(12*1000000000)}" ixy="${0}" ixz="${0}"
+              iyy="${2.568*(25*25+18*18)/(12*1000000000)}" iyz="${0}"
+              izz="${2.568*(25*25+35*35)/(12*1000000000)}"
               c_xyz="${0} ${0} ${-18/2000}"
               size="${25/1000} ${35/1000} ${18/1000}"
@@ -350,9 +350,9 @@
   <mesh_link name="l_thigh"
               origin_rpy="${0} ${pi/2} ${0}" origin_xyz="${0/1000} ${0} ${0/1000}"
-              i_rpy="0 0 0" i_xyz="${7.859/1000} ${-6.38/1000} ${-15.22/1000}"
-              mass="${35/1000}"
-              ixx="${2815.705/1000000000}" ixy="${69.289/1000000000}" ixz="${-116.66/1000000000}"
-              iyx="${69.289/1000000000}" iyy="${2928.22/1000000000}" iyz="${69.297/1000000000}"
-              izx="${-116.66/1000000000}" izy="${69.297/1000000000}" izz="${2815.691/1000000000}"
+              i_rpy="0 0 0" i_xyz="${-28/2000} ${-14/2000} ${-14/2000}"
+              mass="${40/1000}"
+              ixx="${40*(28*28+28*28)/(12*1000000000)}" ixy="${0}" ixz="${0}"
+              iyy="${40*(28*28+28*28)/(12*1000000000)}" iyz="${0}"
+              izz="${40*(28*28+28*28)/(12*1000000000)}"
               c_xyz="${-28/2000} ${-14/2000} ${-14/2000}"
               size="${28/1000} ${28/1000} ${28/1000}"
@@ -363,9 +363,9 @@
   <mesh_link name="l_knee"
               origin_rpy="${0} ${0} ${0}" origin_xyz="${0/1000} ${0/1000} ${0/1000}"
-              i_rpy="0 0 0" i_xyz="${20.7147/1000} ${-1.594/1000} ${3.087/1000}"
+              i_rpy="0 0 0" i_xyz="${35/2000} ${-2/2000} ${0/2000}"
               mass="${5.004/1000}"
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