Commit message: used collision box dimensions for inertia. works nicely. May need to alter component masses after 3D print. still need to add battery.

File: plen_ros/urdf/plen_macro.xacro (robot description, xacro)
@@ -7,5 +7,5 @@
       <parent link="${parent}" />
       <child link="${child}" />
-      <limit effort="${effort}" velocity="${velocity}" lower="-0.01" upper="0.01"/>
+      <limit effort="${effort}" velocity="${velocity}" lower="-0.001" upper="0.001"/>
       <joint_properties damping="${damping}" friction="${friction}" />
     </joint>
@@ -18,5 +18,5 @@
     </joint>
   </xacro:macro>
-  <xacro:macro name="mesh_link" params="name origin_xyz origin_rpy meshfile meshscale size c_xyz matname rgba mass i_xyz i_rpy ixx ixy ixz iyx iyy iyz izx izy izz">
+  <xacro:macro name="mesh_link" params="name origin_xyz origin_rpy meshfile meshscale size c_xyz matname rgba mass i_xyz i_rpy ixx ixy ixz iyy iyz izz">
     <link name="${name}">
       <visual>
@@ -38,5 +38,5 @@
         <mass value="${mass}" />
         <origin rpy="${i_rpy}" xyz="${i_xyz}" /> <!-- Inertial Axes -->
-        <inertia ixx="${ixx}" ixy="${ixy}" ixz="${ixz}" iyx="${iyx}" iyy="${iyy}" iyz="${iyz}" izx="${izx}" izy="${izy}" izz="${izz}" />
+        <inertia ixx="${ixx}" ixy="${ixy}" ixz="${ixz}" iyx="${ixy}" iyy="${iyy}" iyz="${iyz}" izx="${ixz}" izy="${iyz}" izz="${izz}" />
       </inertial>
     </link>

Commit message: fixed urdf contact sensor and td3 typo (tested on bipedal walker)

File: plen_ros/urdf/plen.urdf.xacro (robot description, xacro)
@@ -365,4 +365,7 @@
                 <box size="${41/1000} ${62.867/1000} ${2/1000}"/>
             </geometry>
+            <material name="blue_mat">
+              <color rgba="0 0 1 1" />
+            </material>
         </visual>
   </link>
@@ -475,4 +478,7 @@
                 <box size="${41/1000} ${62.867/1000} ${2/1000}"/>
             </geometry>
+            <material name="blue_mat">
+              <color rgba="0 0 1 1" />
+            </material>
         </visual>
   </link>
@@ -611,5 +617,5 @@
         <parent link="r_foot"/>
         <child link="rfs_link"/>
-        <origin xyz="${-37/4000} ${0} ${-19/1000}" rpy="0 0 0"/>
+        <origin xyz="${-37/4000} ${0} ${-18/1000}" rpy="0 0 0"/>
   </joint>
   <!-- LEFT LEG -->
@@ -662,5 +668,5 @@
         <parent link="l_foot"/>
         <child link="lfs_link"/>
-        <origin xyz="${37/4000} ${0} ${-19/1000}" rpy="0 0 0"/>
+        <origin xyz="${37/4000} ${0} ${-18/1000}" rpy="0 0 0"/>
   </joint>
   <!-- <transmission name="tran1">

Commit message: added hard joint limits to urdf and modified reset for higher fidelity. May need to add rate.sleep if fidelity still not high enough. Also increased batch size of replay buffer.

File: plen_ros/urdf/plen.urdf.xacro (robot description, xacro)
@@ -513,5 +513,7 @@
                     effort="0.15" velocity="8"
                     damping="1"
-                    friction="1"/>
+                    friction="1"
+                    lower="-1.7"
+                    upper="1.7"/>
   <xacro:rev_joint name="r_shoulder_rs_servo" number="14" type="revolute"
                     axis_xyz="0 0 1"
@@ -520,5 +522,7 @@
                     effort="0.15" velocity="8"
                     damping="1"
-                    friction="1"/>
+                    friction="1"
+                    lower="-0.15"
+                    upper="1.7"/>
   <xacro:frame_joint name="rs_servo_r_arm" type="fixed"
                     origin_rpy="${-pi/2} 0 ${0}" origin_xyz="${0/1000} ${19.5/1000} ${-2/1000}"
@@ -533,5 +537,7 @@
                     effort="0.15" velocity="8"
                     damping="1"
-                    friction="1"/>
+                    friction="1"
+                    lower="-0.2"
+                    upper="0.5"/>
   <xacro:frame_joint name="r_elbow_r_hand" type="fixed"
                     origin_rpy="${pi} ${pi/2} ${0}" origin_xyz="${-30/1000} ${0/1000} ${0/1000}"
@@ -544,5 +550,7 @@
                     effort="0.15" velocity="8"
                     damping="1"
-                    friction="1"/>
+                    friction="1"
+                    lower="-1.7"
+                    upper="1.7"/>
   <xacro:rev_joint name="l_shoulder_ls_servo" number="17" type="revolute"
                     axis_xyz="0 0 1"
@@ -551,5 +559,7 @@
                     effort="0.15" velocity="8"
                     damping="1"
-                    friction="1"/>
+                    friction="1"
+                    lower="-0.15"
+                    upper="1.7"/>
   <xacro:frame_joint name="ls_servo_l_arm" type="fixed"
                     origin_rpy="${-pi/2} 0 ${0}" origin_xyz="${0/1000} ${19.5/1000} ${-2/1000}"
@@ -564,5 +574,7 @@
                     effort="0.15" velocity="8"
                     damping="1"
-                    friction="1"/>
+                    friction="1"
+                    lower="-0.2"
+                    upper="0.5"/>
   <xacro:frame_joint name="l_elbow_l_hand" type="fixed"
                     origin_rpy="${pi} ${pi/2} ${0}" origin_xyz="${-30/1000} ${0/1000} ${0/1000}"
@@ -575,5 +587,7 @@
                     effort="0.15" velocity="8"
                     damping="1"
-                    friction="1"/>
+                    friction="1"
+                    lower="-1.7"
+                    upper="1.7"/>
   <xacro:rev_joint name="r_hip_r_thigh" number="2" type="revolute"
                     axis_xyz="0 1 0"
@@ -582,5 +596,7 @@
                     effort="0.15" velocity="8"
                     damping="1"
-                    friction="1"/>
+                    friction="1"
+                    lower="-1.54"
+                    upper="0.12"/>
   <xacro:rev_joint name="r_thigh_r_knee" number="3" type="revolute"
                     axis_xyz="0 1 0"
@@ -589,5 +605,7 @@
                     effort="0.15" velocity="8"
                     damping="1"
-                    friction="1"/>
+                    friction="1"
+                    lower="-1.7"
+                    upper="0.75"/>
   <xacro:frame_joint name="r_knee_knee_servo" type="fixed"
                     origin_rpy="${-pi/2} 0 0" origin_xyz="${28/1000} ${-12.8/1000} ${0.5/1000}"
@@ -599,5 +617,7 @@
                     effort="0.15" velocity="8"
                     damping="1"
-                    friction="1"/>
+                    friction="1"
+                    lower="-0.2"
+                    upper="0.95"/>
   <xacro:rev_joint name="r_shin_r_ankle" number="5" type="revolute"
                     axis_xyz="0 0 1"
@@ -606,5 +626,7 @@
                     effort="0.15" velocity="8"
                     damping="1"
-                    friction="1"/>
+                    friction="1"
+                    lower="-0.95"
+                    upper="1.54"/>
   <xacro:rev_joint name="r_ankle_r_foot" number="6" type="revolute"
                     axis_xyz="0 1 0"
@@ -613,5 +635,7 @@
                     effort="0.15" velocity="8"
                     damping="1"
-                    friction="1"/>
+                    friction="1"
+                    lower="-0.45"
+                    upper="0.8"/>
   <joint name="r_foot_r_sensor" type="fixed">
         <parent link="r_foot"/>
@@ -626,5 +650,7 @@
                     effort="0.15" velocity="8"
                     damping="1"
-                    friction="1"/>
+                    friction="1"
+                    lower="-1.7"
+                    upper="1.7"/>
   <xacro:rev_joint name="l_hip_l_thigh" number="8" type="revolute"
                     axis_xyz="1 0 0"
@@ -633,5 +659,7 @@
                     effort="0.15" velocity="8"
                     damping="1"
-                    friction="1"/>
+                    friction="1"
+                    lower="-0.12"
+                    upper="1.54"/>
   <xacro:rev_joint name="l_thigh_l_knee" number="9" type="revolute"
                     axis_xyz="0 1 0"
@@ -640,5 +668,7 @@
                     effort="0.15" velocity="8"
                     damping="1"
-                    friction="1"/>
+                    friction="1"
+                    lower="-0.75"
+                    upper="1.7"/>
   <xacro:frame_joint name="l_knee_knee_servo" type="fixed"
                     origin_rpy="${-pi/2} ${pi} 0" origin_xyz="${28/1000} ${1.45/1000} ${0/1000}"
@@ -650,5 +680,7 @@
                     effort="0.15" velocity="8"
                     damping="1"
-                    friction="1"/>
+                    friction="1"
+                    lower="-0.95"
+                    upper="0.2"/>
   <xacro:rev_joint name="l_shin_l_ankle" number="11" type="revolute"
                     axis_xyz="0 1 0"
@@ -657,5 +689,7 @@
                     effort="0.15" velocity="8"
                     damping="1"
-                    friction="1"/>
+                    friction="1"
+                    lower="-1.54"
+                    upper="0.95"/>
   <xacro:rev_joint name="l_ankle_l_foot" number="12" type="revolute"
                     axis_xyz="0 1 0"
@@ -664,5 +698,7 @@
                     effort="0.15" velocity="8"
                     damping="1"
-                    friction="1"/> <!-- effort and velocity taken from FEETECH FS90-FB datasheet -->
+                    friction="1"
+                    lower="-0.8"
+                    upper="0.45"/> <!-- effort and velocity taken from FEETECH FS90-FB datasheet -->
   <joint name="l_foot_l_sensor" type="fixed">
         <parent link="l_foot"/>

File: plen_ros/urdf/plen_macro.xacro (robot description, xacro)
@@ -1,5 +1,5 @@
 <?xml version="1.0" ?>
 <robot xmlns:xacro="http://www.ros.org/wiki/xacro">
-  <xacro:macro name="rev_joint" params="name number type axis_xyz origin_rpy origin_xyz parent child effort velocity damping friction">
+  <xacro:macro name="rev_joint" params="name number type axis_xyz origin_rpy origin_xyz parent child effort velocity damping friction upper lower">
     <joint name="${name}" type="${type}">
       <axis xyz="${axis_xyz}" />
@@ -7,5 +7,5 @@
       <parent link="${parent}" />
       <child link="${child}" />
-      <limit effort="${effort}" velocity="${velocity}" lower="-1.7" upper="1.7"/>
+      <limit effort="${effort}" velocity="${velocity}" lower="${lower}" upper="${upper}"/>
       <joint_properties damping="${damping}" friction="${friction}" />
     </joint>
