Commit message: modified joint limits for urdf and gazebo

File: plen_ros/urdf/plen.urdf.xacro (robot description, xacro)
@@ -19,5 +19,5 @@
               size="${45/1000} ${48/1000} ${75/1000}"
               matname="red_mat"
-              rgba="1 0 0 1"
+              rgba="0 0 0 1"
               meshfile="package://plen_ros/meshes/torso.stl"
               meshscale="0.001 0.001 0.001" /> <!-- m to mm -->
@@ -31,6 +31,6 @@
               c_xyz="${15/2000} ${0} ${46/4000}"
               size="${11/1000} ${51/1000} ${46/1000}"
-              matname="green_mat"
-              rgba="0 1 0 1"
+              matname="purple_mat"
+              rgba="0.42 0.05 0.68 1"
               meshfile="package://plen_ros/meshes/battery.stl"
               meshscale="0.001 0.001 0.001" />
@@ -44,6 +44,6 @@
               c_xyz="${0} ${0} ${0/2000}"
               size="${40/1000} ${40/1000} ${40/1000}"
-              matname="green_mat"
-              rgba="0 1 0 1"
+              matname="purple_mat"
+              rgba="0.42 0.05 0.68 1"
               meshfile="package://plen_ros/meshes/head.stl"
               meshscale="0.001 0.001 0.001" />
@@ -57,6 +57,6 @@
               c_xyz="${0} ${25/4000} ${0/2000}"
               size="${12/1000} ${25/1000} ${25/1000}"
-              matname="blue_mat"
-              rgba="0 0 1 1"
+              matname="orange_mat"
+              rgba="1 0.49 0 1"
               meshfile="package://plen_ros/meshes/servo.stl"
               meshscale="0.001 0.001 0.001" />
@@ -70,6 +70,6 @@
               c_xyz="${0} ${25/4000} ${0/2000}"
               size="${12/1000} ${25/1000} ${25/1000}"
-              matname="blue_mat"
-              rgba="0 0 1 1"
+              matname="orange_mat"
+              rgba="1 0.49 0 1"
               meshfile="package://plen_ros/meshes/servo.stl"
               meshscale="0.001 0.001 0.001" />
@@ -83,6 +83,6 @@
               c_xyz="${0} ${25/4000} ${0/2000}"
               size="${12/1000} ${25/1000} ${25/1000}"
-              matname="blue_mat"
-              rgba="0 0 1 1"
+              matname="orange_mat"
+              rgba="1 0.49 0 1"
               meshfile="package://plen_ros/meshes/servo.stl"
               meshscale="0.001 0.001 0.001" />
@@ -96,6 +96,6 @@
               c_xyz="${0} ${25/4000} ${0/2000}"
               size="${12/1000} ${25/1000} ${25/1000}"
-              matname="blue_mat"
-              rgba="0 0 1 1"
+              matname="orange_mat"
+              rgba="1 0.49 0 1"
               meshfile="package://plen_ros/meshes/servo.stl"
               meshscale="0.001 0.001 0.001" />
@@ -109,6 +109,6 @@
               c_xyz="${0} ${0} ${25/2000}"
               size="${18/1000} ${35/1000} ${25/1000}"
-              matname="green_mat"
-              rgba="0 1 0 1"
+              matname="purple_mat"
+              rgba="0.42 0.05 0.68 1"
               meshfile="package://plen_ros/meshes/shoulder.stl"
               meshscale="0.001 0.001 0.001" />
@@ -122,6 +122,6 @@
               c_xyz="${0} ${25/4000} ${0/2000}"
               size="${12/1000} ${25/1000} ${25/1000}"
-              matname="blue_mat"
-              rgba="0 0 1 1"
+              matname="orange_mat"
+              rgba="1 0.49 0 1"
               meshfile="package://plen_ros/meshes/servo.stl"
               meshscale="0.001 0.001 0.001" />
@@ -136,5 +136,5 @@
               size="${15/1000} ${35/1000} ${50/1000}"
               matname="red_mat"
-              rgba="1 0 0 1"
+              rgba="0 0 0 1"
               meshfile="package://plen_ros/meshes/arm.stl"
               meshscale="0.001 0.001 0.001" />
@@ -148,6 +148,6 @@
               c_xyz="${0} ${25/4000} ${0/2000}"
               size="${12/1000} ${25/1000} ${25/1000}"
-              matname="blue_mat"
-              rgba="0 0 1 1"
+              matname="orange_mat"
+              rgba="1 0.49 0 1"
               meshfile="package://plen_ros/meshes/servo.stl"
               meshscale="0.001 0.001 0.001" />
@@ -161,6 +161,6 @@
               c_xyz="${-27/4000} ${0} ${0/2000}"
               size="${27/1000} ${34/1000} ${14/1000}"
-              matname="green_mat"
-              rgba="0 1 0 1"
+              matname="purple_mat"
+              rgba="0.42 0.05 0.68 1"
               meshfile="package://plen_ros/meshes/elbow.stl"
               meshscale="0.001 0.001 0.001" />
@@ -175,5 +175,5 @@
               size="${19/1000} ${34/1000} ${35/1000}"
               matname="red_mat"
-              rgba="1 0 0 1"
+              rgba="0 0 0 1"
               meshfile="package://plen_ros/meshes/hand.stl"
               meshscale="0.001 0.001 0.001" />
@@ -187,6 +187,6 @@
               c_xyz="${0} ${0} ${25/2000}"
               size="${18/1000} ${35/1000} ${25/1000}"
-              matname="green_mat"
-              rgba="0 1 0 1"
+              matname="purple_mat"
+              rgba="0.42 0.05 0.68 1"
               meshfile="package://plen_ros/meshes/shoulder.stl"
               meshscale="0.001 0.001 0.001" />
@@ -200,6 +200,6 @@
               c_xyz="${0} ${25/4000} ${0/2000}"
               size="${12/1000} ${25/1000} ${25/1000}"
-              matname="blue_mat"
-              rgba="0 0 1 1"
+              matname="orange_mat"
+              rgba="1 0.49 0 1"
               meshfile="package://plen_ros/meshes/servo.stl"
               meshscale="0.001 0.001 0.001" />
@@ -214,5 +214,5 @@
               size="${15/1000} ${35/1000} ${50/1000}"
               matname="red_mat"
-              rgba="1 0 0 1"
+              rgba="0 0 0 1"
               meshfile="package://plen_ros/meshes/arm.stl"
               meshscale="0.001 0.001 0.001" />
@@ -226,6 +226,6 @@
               c_xyz="${0} ${25/4000} ${0/2000}"
               size="${12/1000} ${25/1000} ${25/1000}"
-              matname="blue_mat"
-              rgba="0 0 1 1"
+              matname="orange_mat"
+              rgba="1 0.49 0 1"
               meshfile="package://plen_ros/meshes/servo.stl"
               meshscale="0.001 0.001 0.001" />
@@ -239,6 +239,6 @@
               c_xyz="${-27/4000} ${0} ${0/2000}"
               size="${27/1000} ${34/1000} ${14/1000}"
-              matname="green_mat"
-              rgba="0 1 0 1"
+              matname="purple_mat"
+              rgba="0.42 0.05 0.68 1"
               meshfile="package://plen_ros/meshes/elbow.stl"
               meshscale="0.001 0.001 0.001" />
@@ -253,5 +253,5 @@
               size="${19/1000} ${34/1000} ${35/1000}"
               matname="red_mat"
-              rgba="1 0 0 1"
+              rgba="0 0 0 1"
               meshfile="package://plen_ros/meshes/hand.stl"
               meshscale="0.001 0.001 0.001" />
@@ -265,6 +265,6 @@
               c_xyz="${0} ${0} ${-18/2000}"
               size="${25/1000} ${35/1000} ${18/1000}"
-              matname="blue_mat"
-              rgba="0 0 1 1"
+              matname="orange_mat"
+              rgba="1 0.49 0 1"
               meshfile="package://plen_ros/meshes/rhip.stl"
               meshscale="0.001 0.001 0.001" />
@@ -278,6 +278,6 @@
               c_xyz="${-14/2000} ${0} ${14/2000}"
               size="${28/1000} ${28/1000} ${28/1000}"
-              matname="green_mat"
-              rgba="0 1 0 1"
+              matname="purple_mat"
+              rgba="0.42 0.05 0.68 1"
               meshfile="package://plen_ros/meshes/rthigh.stl"
               meshscale="0.001 0.001 0.001" />
@@ -293,5 +293,5 @@
               size="${38/1000} ${30/1000} ${24/1000}"
               matname="red_mat"
-              rgba="1 0 0 1"
+              rgba="0 0 0 1"
               meshfile="package://plen_ros/meshes/rknee.stl"
               meshscale="0.001 0.001 0.001" />
@@ -305,6 +305,6 @@
               c_xyz="${0} ${25/4000} ${0/2000}"
               size="${12/1000} ${25/1000} ${25/1000}"
-              matname="blue_mat"
-              rgba="0 0 1 1"
+              matname="orange_mat"
+              rgba="1 0.49 0 1"
               meshfile="package://plen_ros/meshes/servo.stl"
               meshscale="0.001 0.001 0.001" />
@@ -318,6 +318,6 @@
               c_xyz="${36/2000} ${0} ${8/2000}"
               size="${45/1000} ${40/1000} ${23/1000}"
-              matname="blue_mat"
-              rgba="0 0 1 1"
+              matname="orange_mat"
+              rgba="1 0.49 0 1"
               meshfile="package://plen_ros/meshes/rshin.stl"
               meshscale="0.001 0.001 0.001" />
@@ -331,6 +331,6 @@
               c_xyz="${14/2000} ${-14/2000} ${-28/2000}"
               size="${28/1000} ${28/1000} ${28/1000}"
-              matname="green_mat"
-              rgba="0 1 0 1"
+              matname="purple_mat"
+              rgba="0.42 0.05 0.68 1"
               meshfile="package://plen_ros/meshes/rankle.stl"
               meshscale="0.001 0.001 0.001" />
@@ -345,5 +345,5 @@
               size="${41/1000} ${62.867/1000} ${4/1000}"
               matname="red_mat"
-              rgba="1 0 0 1"
+              rgba="0 0 0 1"
               meshfile="package://plen_ros/meshes/rfoot.stl"
               meshscale="0.001 0.001 0.001" />
@@ -365,6 +365,6 @@
                 <box size="${41/1000} ${62.867/1000} ${2/1000}"/>
             </geometry>
-            <material name="blue_mat">
-              <color rgba="0 0 1 1" />
+            <material name="orange_mat">
+              <color rgba="1 0.49 0 1" />
             </material>
         </visual>
@@ -379,6 +379,6 @@
               c_xyz="${0} ${0} ${-18/2000}"
               size="${25/1000} ${35/1000} ${18/1000}"
-              matname="blue_mat"
-              rgba="0 0 1 1"
+              matname="orange_mat"
+              rgba="1 0.49 0 1"
               meshfile="package://plen_ros/meshes/lhip.stl"
               meshscale="0.001 0.001 0.001" />
@@ -392,6 +392,6 @@
               c_xyz="${-28/2000} ${-14/2000} ${-14/2000}"
               size="${28/1000} ${28/1000} ${28/1000}"
-              matname="green_mat"
-              rgba="0 1 0 1"
+              matname="purple_mat"
+              rgba="0.42 0.05 0.68 1"
               meshfile="package://plen_ros/meshes/rankle.stl"
               meshscale="0.001 0.001 0.001" />
@@ -406,5 +406,5 @@
               size="${38/1000} ${30/1000} ${24/1000}"
               matname="red_mat"
-              rgba="1 0 0 1"
+              rgba="0 0 0 1"
               meshfile="package://plen_ros/meshes/lknee.stl"
               meshscale="0.001 0.001 0.001" />
@@ -418,6 +418,6 @@
               c_xyz="${0} ${25/4000} ${0/2000}"
               size="${12/1000} ${25/1000} ${25/1000}"
-              matname="blue_mat"
-              rgba="0 0 1 1"
+              matname="orange_mat"
+              rgba="1 0.49 0 1"
               meshfile="package://plen_ros/meshes/servo.stl"
               meshscale="0.001 0.001 0.001" />
@@ -431,6 +431,6 @@
               c_xyz="${-36/2000} ${0} ${8/2000}"
               size="${45/1000} ${40/1000} ${23/1000}"
-              matname="blue_mat"
-              rgba="0 0 1 1"
+              matname="orange_mat"
+              rgba="1 0.49 0 1"
               meshfile="package://plen_ros/meshes/rshin.stl"
               meshscale="0.001 0.001 0.001" />
@@ -444,6 +444,6 @@
               c_xyz="${-14/2000} ${0/2000} ${14/2000}"
               size="${28/1000} ${28/1000} ${28/1000}"
-              matname="green_mat"
-              rgba="0 1 0 1"
+              matname="purple_mat"
+              rgba="0.42 0.05 0.68 1"
               meshfile="package://plen_ros/meshes/rthigh.stl"
               meshscale="0.001 0.001 0.001" />
@@ -458,5 +458,5 @@
               size="${41/1000} ${62.867/1000} ${4/1000}"
               matname="red_mat"
-              rgba="1 0 0 1"
+              rgba="0 0 0 1"
               meshfile="package://plen_ros/meshes/lfoot.stl"
               meshscale="0.001 0.001 0.001" />
@@ -478,6 +478,6 @@
                 <box size="${41/1000} ${62.867/1000} ${2/1000}"/>
             </geometry>
-            <material name="blue_mat">
-              <color rgba="0 0 1 1" />
+            <material name="orange_mat">
+              <color rgba="1 0.49 0 1" />
             </material>
         </visual>
@@ -514,6 +514,6 @@
                     damping="1"
                     friction="1"
-                    lower="-1.7"
-                    upper="1.7"/>
+                    lower="-1.57"
+                    upper="1.57"/>
   <xacro:rev_joint name="r_shoulder_rs_servo" number="14" type="revolute"
                     axis_xyz="0 0 1"
@@ -524,5 +524,5 @@
                     friction="1"
                     lower="-0.15"
-                    upper="1.7"/>
+                    upper="1.57"/>
   <xacro:frame_joint name="rs_servo_r_arm" type="fixed"
                     origin_rpy="${-pi/2} 0 ${0}" origin_xyz="${0/1000} ${19.5/1000} ${-2/1000}"
@@ -539,5 +539,5 @@
                     friction="1"
                     lower="-0.2"
-                    upper="0.5"/>
+                    upper="0.35"/>
   <xacro:frame_joint name="r_elbow_r_hand" type="fixed"
                     origin_rpy="${pi} ${pi/2} ${0}" origin_xyz="${-30/1000} ${0/1000} ${0/1000}"
@@ -551,6 +551,6 @@
                     damping="1"
                     friction="1"
-                    lower="-1.7"
-                    upper="1.7"/>
+                    lower="-1.57"
+                    upper="1.57"/>
   <xacro:rev_joint name="l_shoulder_ls_servo" number="17" type="revolute"
                     axis_xyz="0 0 1"
@@ -561,5 +561,5 @@
                     friction="1"
                     lower="-0.15"
-                    upper="1.7"/>
+                    upper="1.57"/>
   <xacro:frame_joint name="ls_servo_l_arm" type="fixed"
                     origin_rpy="${-pi/2} 0 ${0}" origin_xyz="${0/1000} ${19.5/1000} ${-2/1000}"
@@ -576,5 +576,5 @@
                     friction="1"
                     lower="-0.2"
-                    upper="0.5"/>
+                    upper="0.35"/>
   <xacro:frame_joint name="l_elbow_l_hand" type="fixed"
                     origin_rpy="${pi} ${pi/2} ${0}" origin_xyz="${-30/1000} ${0/1000} ${0/1000}"
@@ -588,6 +588,6 @@
                     damping="1"
                     friction="1"
-                    lower="-1.7"
-                    upper="1.7"/>
+                    lower="-1.57"
+                    upper="1.57"/>
   <xacro:rev_joint name="r_hip_r_thigh" number="2" type="revolute"
                     axis_xyz="0 1 0"
@@ -597,6 +597,6 @@
                     damping="1"
                     friction="1"
-                    lower="-1.54"
-                    upper="0.12"/>
+                    lower="-0.15"
+                    upper="1.5"/>
   <xacro:rev_joint name="r_thigh_r_knee" number="3" type="revolute"
                     axis_xyz="0 1 0"
@@ -606,5 +606,5 @@
                     damping="1"
                     friction="1"
-                    lower="-1.7"
+                    lower="-0.95"
                     upper="0.75"/>
   <xacro:frame_joint name="r_knee_knee_servo" type="fixed"
@@ -618,6 +618,6 @@
                     damping="1"
                     friction="1"
-                    lower="-0.2"
-                    upper="0.95"/>
+                    lower="-0.9"
+                    upper="0.3"/>
   <xacro:rev_joint name="r_shin_r_ankle" number="5" type="revolute"
                     axis_xyz="0 0 1"
@@ -628,5 +628,5 @@
                     friction="1"
                     lower="-0.95"
-                    upper="1.54"/>
+                    upper="1.2"/>
   <xacro:rev_joint name="r_ankle_r_foot" number="6" type="revolute"
                     axis_xyz="0 1 0"
@@ -636,6 +636,6 @@
                     damping="1"
                     friction="1"
-                    lower="-0.45"
-                    upper="0.8"/>
+                    lower="-0.8"
+                    upper="0.4"/>
   <joint name="r_foot_r_sensor" type="fixed">
         <parent link="r_foot"/>
@@ -651,6 +651,6 @@
                     damping="1"
                     friction="1"
-                    lower="-1.7"
-                    upper="1.7"/>
+                    lower="-1.57"
+                    upper="1.57"/>
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