Commit message: modified urdf to sim joint control. Position-based control with max velocity seems like a good method... compare to real servo and use time attribute to record how long reach took. recorded joint names as well.

File: plen_bullet/plen.urdf (robot description, URDF)
Before this commit: robot plen, 33 links, 32 joints
Joints:
- joint r_shoulder_rs_servo: limit lower=-0.001 upper=0.001 effort=100 velocity=100 -> lower=-3.14 upper=3.14 effort=100 velocity=100

Commit message: added option to load prior policy in td3.
Converted meshes to binary for bullet

File: plen_bullet/plen.urdf (robot description, URDF)
Before this commit: robot plen, 33 links, 32 joints
Links:
- link battery: geometry collision box size=0.011 0.051 0.046; visual mesh filename=package://plen_ros/meshes_bin/battery.stl scale=0.001 0.001 0.001
- link head: geometry collision box size=0.04 0.04 0.04; visual mesh filename=package://plen_ros/meshes_bin/head.stl scale=0.001 0.001 0.001
- link l_ankle: geometry collision box size=0.028 0.028 0.028; visual mesh filename=package://plen_ros/meshes_bin/rthigh.stl scale=0.001 0.001 0.001
- link l_arm: geometry collision box size=0.015 0.035 0.05; visual mesh filename=package://plen_ros/meshes_bin/arm.stl scale=0.001 0.001 0.001
- link l_elbow: geometry collision box size=0.027 0.034 0.014; visual mesh filename=package://plen_ros/meshes_bin/elbow.stl scale=0.001 0.001 0.001
- link l_foot: geometry collision box size=0.041 0.062867 0.004; visual mesh filename=package://plen_ros/meshes_bin/lfoot.stl scale=0.001 0.001 0.001
- link l_hand: geometry collision box size=0.019 0.034 0.035; visual mesh filename=package://plen_ros/meshes_bin/hand.stl scale=0.001 0.001 0.001
- link l_hip: geometry collision box size=0.025 0.035 0.018; visual mesh filename=package://plen_ros/meshes_bin/lhip.stl scale=0.001 0.001 0.001
- link l_knee: geometry collision box size=0.038 0.03 0.024; visual mesh filename=package://plen_ros/meshes_bin/lknee.stl scale=0.001 0.001 0.001
- link l_knee_servo: geometry collision box size=0.012 0.025 0.025; visual mesh filename=package://plen_ros/meshes_bin/servo.stl scale=0.001 0.001 0.001
- link l_shin: geometry collision box size=0.045 0.04 0.023; visual mesh filename=package://plen_ros/meshes_bin/rshin.stl scale=0.001 0.001 0.001
- link l_shoulder: geometry collision box size=0.018 0.035 0.025; visual mesh filename=package://plen_ros/meshes_bin/shoulder.stl scale=0.001 0.001 0.001
- link l_thigh: geometry collision box size=0.028 0.028 0.028; visual mesh filename=package://plen_ros/meshes_bin/rankle.stl scale=0.001 0.001 0.001
- link lb_servo: geometry collision box size=0.012 0.025 0.025; visual mesh filename=package://plen_ros/meshes_bin/servo.stl scale=0.001 0.001 0.001
- link le_servo: geometry collision box size=0.012 0.025 0.025; visual mesh filename=package://plen_ros/meshes_bin/servo.stl scale=0.001 0.001 0.001
- link ls_servo: geometry collision box size=0.012 0.025 0.025; visual mesh filename=package://plen_ros/meshes_bin/servo.stl scale=0.001 0.001 0.001
- link lt_servo: geometry collision box size=0.012 0.025 0.025; visual mesh filename=package://plen_ros/meshes_bin/servo.stl scale=0.001 0.001 0.001
- link r_ankle: geometry collision box size=0.028 0.028 0.028; visual mesh filename=package://plen_ros/meshes_bin/rankle.stl scale=0.001 0.001 0.001
- link r_arm: geometry collision box size=0.015 0.035 0.05; visual mesh filename=package://plen_ros/meshes_bin/arm.stl scale=0.001 0.001 0.001
- link r_elbow: geometry collision box size=0.027 0.034 0.014; visual mesh filename=package://plen_ros/meshes_bin/elbow.stl scale=0.001 0.001 0.001
- link r_foot: geometry collision box size=0.041 0.062867 0.004; visual mesh filename=package://plen_ros/meshes_bin/rfoot.stl scale=0.001 0.001 0.001
- link r_hand: geometry collision box size=0.019 0.034 0.035; visual mesh filename=package://plen_ros/meshes_bin/hand.stl scale=0.001 0.001 0.001
- link r_hip: geometry collision box size=0.025 0.035 0.018; visual mesh filename=package://plen_ros/meshes_bin/rhip.stl scale=0.001 0.001 0.001
- link r_knee: geometry collision box size=0.038 0.03 0.024; visual mesh filename=package://plen_ros/meshes_bin/rknee.stl scale=0.001 0.001 0.001
- link r_knee_servo: geometry collision box size=0.012 0.025 0.025; visual mesh filename=package://plen_ros/meshes_bin/servo.stl scale=0.001 0.001 0.001
- link r_shin: geometry collision box size=0.045 0.04 0.023; visual mesh filename=package://plen_ros/meshes_bin/rshin.stl scale=0.001 0.001 0.001
- link r_shoulder: geometry collision box size=0.018 0.035 0.025; visual mesh filename=package://plen_ros/meshes_bin/shoulder.stl scale=0.001 0.001 0.001
- link r_thigh: geometry collision box size=0.028 0.028 0.028; visual mesh filename=package://plen_ros/meshes_bin/rthigh.stl scale=0.001 0.001 0.001
- link rb_servo: geometry collision box size=0.012 0.025 0.025; visual mesh filename=package://plen_ros/meshes_bin/servo.stl scale=0.001 0.001 0.001
- link re_servo: geometry collision box size=0.012 0.025 0.025; visual mesh filename=package://plen_ros/meshes_bin/servo.stl scale=0.001 0.001 0.001
- link rs_servo: geometry collision box size=0.012 0.025 0.025; visual mesh filename=package://plen_ros/meshes_bin/servo.stl scale=0.001 0.001 0.001
- link rt_servo: geometry collision box size=0.012 0.025 0.025; visual mesh filename=package://plen_ros/meshes_bin/servo.stl scale=0.001 0.001 0.001
- link torso: geometry collision box size=0.045 0.048 0.075; visual mesh filename=package://plen_ros/meshes_bin/torso.stl scale=0.001 0.001 0.001
