Commit message: found issue with bullet; urdf had joint limits

File: plen_bullet/src/plen.urdf (robot description, URDF)
Before this commit: robot plen, 33 links, 32 joints
Joints:
- joint l_ankle_l_foot: limit lower=-0.001 upper=0.001 effort=100 velocity=100 -> lower=-1.7 upper=1.7 effort=0.15 velocity=8.0
- joint l_hip_l_thigh: limit lower=-0.001 upper=0.001 effort=100 velocity=100 -> lower=-1.7 upper=1.7 effort=0.15 velocity=8.0
- joint l_knee_l_shin: limit lower=-0.001 upper=0.001 effort=100 velocity=100 -> lower=-1.7 upper=1.7 effort=0.15 velocity=8.0
- joint l_shin_l_ankle: limit lower=-0.001 upper=0.001 effort=100 velocity=100 -> lower=-1.7 upper=1.7 effort=0.15 velocity=8.0
- joint l_shoulder_ls_servo: limit lower=-0.001 upper=0.001 effort=100 velocity=100 -> lower=-1.7 upper=1.7 effort=0.15 velocity=8.0
- joint l_thigh_l_knee: limit lower=-0.001 upper=0.001 effort=100 velocity=100 -> lower=-1.7 upper=1.7 effort=0.15 velocity=8.0
- joint lb_servo_l_hip: limit lower=-0.001 upper=0.001 effort=100 velocity=100 -> lower=-1.7 upper=1.7 effort=0.15 velocity=8.0
- joint le_servo_l_elbow: limit lower=-0.001 upper=0.001 effort=100 velocity=100 -> lower=-1.7 upper=1.7 effort=0.15 velocity=8.0
- joint r_ankle_r_foot: limit lower=-0.001 upper=0.001 effort=100 velocity=100 -> lower=-1.7 upper=1.7 effort=0.15 velocity=8.0
- joint r_hip_r_thigh: limit lower=-0.001 upper=0.001 effort=100 velocity=100 -> lower=-1.7 upper=1.7 effort=0.15 velocity=8.0
- joint r_knee_r_shin: limit lower=-0.001 upper=0.001 effort=100 velocity=100 -> lower=-1.7 upper=1.7 effort=0.15 velocity=8.0
- joint r_shin_r_ankle: limit lower=-0.001 upper=0.001 effort=100 velocity=100 -> lower=-1.7 upper=1.7 effort=0.15 velocity=8.0
- joint r_shoulder_rs_servo: limit lower=-3.14 upper=3.14 effort=100 velocity=100 -> lower=-3.14 upper=3.14 effort=0.15 velocity=8.0
- joint r_thigh_r_knee: limit lower=-0.001 upper=0.001 effort=100 velocity=100 -> lower=-1.7 upper=1.7 effort=0.15 velocity=8.0
- joint rb_servo_r_hip: limit lower=-0.001 upper=0.001 effort=100 velocity=100 -> lower=-1.7 upper=1.7 effort=0.15 velocity=8.0
- joint re_servo_r_elbow: limit lower=-0.001 upper=0.001 effort=100 velocity=100 -> lower=-1.7 upper=1.7 effort=0.15 velocity=8.0
- joint torso_l_shoulder: limit lower=-0.001 upper=0.001 effort=100 velocity=100 -> lower=-1.7 upper=1.7 effort=0.15 velocity=8.0
- joint torso_r_shoulder: limit lower=-0.001 upper=0.001 effort=100 velocity=100 -> lower=-1.7 upper=1.7 effort=0.15 velocity=8.0

Commit message: bullet sim now works great, fixed contact leg ID issue

File: plen_bullet/src/plen.urdf (robot description, URDF)
Before this commit: robot plen, 33 links, 32 joints
Joints:
- joint r_shoulder_rs_servo: limit lower=-3.14 upper=3.14 effort=0.15 velocity=8.0 -> lower=-1.7 upper=1.7 effort=0.15 velocity=8.0

Commit message: improved model behavior and added foot mesh as collision object (tiny loss of performance for much higher accuracy!). All other collision objects left as basic geometry

File: plen_bullet/src/plen.urdf (robot description, URDF)
Before this commit: robot plen, 33 links, 32 joints
Links:
- link l_foot: geometry collision mesh filename=package://plen_ros/meshes_bin/lfoot.stl scale=0.001 0.001 0.001; visual mesh filename=package://plen_ros/meshes_bin/lfoot.stl scale=0.001 0.001 0.001
- link r_foot: geometry collision mesh filename=package://plen_ros/meshes_bin/rfoot.stl scale=0.001 0.001 0.001; visual mesh filename=package://plen_ros/meshes_bin/rfoot.stl scale=0.001 0.001 0.001
